File: nestbox_power.sch (KiCad schematic (older format))
At the start: 9 parts, among them P4 NFC_PWR_SEL, U3 TPS630250RNC

Commit message: pcb file components clustering
pcb file components were clustered according to the Eeschema -
currently everything is on one layer, F.Cu
Parts:
- BT1: symbol Battery -> Battery-RESCUE-Nestbox_v1
Changed lines of the file:
@@
 EESchema Schematic File Version 2
+LIBS:Nestbox_v1-rescue
 LIBS:power
 LIBS:device
@@
 LIBS:contrib
 LIBS:valves
-LIBS:octanis3
 LIBS:SeeedOPL-Capacitor-2016
 LIBS:SeeedOPL-Connector-2016
@@
 LIBS:SeeedOPL-Switch-2016
 LIBS:SeeedOPL-Transistor-2016
-LIBS:crystal_4pin
 LIBS:Nestbox_v1-cache
 EELAYER 25 0
@@
 $EndComp
 $Comp
-L Battery BT1
+L Battery-RESCUE-Nestbox_v1 BT1
 U 1 1 587BD6BC
 P 3650 3650
+AR Path="/587BD6BC" Ref="BT1"  Part="1"
+AR Path="/587910A2/587BD6BC" Ref="BT1"  Part="1"
 F 0 "BT1" H 3750 3700 50  0000 L CNN
 F 1 "Battery" H 3750 3600 50  0000 L CNN

Commit message: NFC & power placed
Parts:
- R25: value R -> 180k
Changed lines of the file:
@@
 P 6750 3850
 F 0 "R25" V 6830 3850 50  0000 C CNN
-F 1 "R" V 6750 3850 50  0000 C CNN
+F 1 "180k" V 6750 3850 50  0000 C CNN
 F 2 "Resistors_SMD:R_0603" V 6680 3850 50  0001 C CNN
 F 3 "" H 6750 3850 50  0000 C CNN

Commit message: corrected phototransistor pins, added power jumpers & testpoints and light barrier signal access
Parts:
- added JP1, JP2: JUMPER, Socket_Strips:Socket_Strip_Straight_1x02, symbol JUMPER
- L7: value XFL4020 -> XFL4020-102ME
Connections:
- net +3V3: now also JP2.2; no longer C27.1, C28.1, R24.2, U3.12 (VOUT_2), U3.13 (VOUT_3), U3.14 (VOUT)
- net +BATT: now also JP1.1; no longer C26.1, U3.4 (VIN_2), U3.5 (VIN_3), U3.6 (VIN), U3.7 (VINA), U3.8 (EN)
- new net: C27.1, C28.1, JP2.1, R24.2, U3.12 (VOUT_2), U3.13 (VOUT_3), U3.14 (VOUT)
- new net: C26.1, JP1.2, U3.4 (VIN_2), U3.5 (VIN_3), U3.6 (VIN), U3.7 (VINA), U3.8 (EN)
Changed lines of the file:
@@
 P 5650 2650
 F 0 "L7" V 5600 2650 50  0000 C CNN
-F 1 "XFL4020" V 5750 2650 50  0000 C CNN
+F 1 "XFL4020-102ME" V 5750 2650 50  0000 C CNN
 F 2 "Octanis3:XFL4020" H 5650 2650 50  0001 C CNN
 F 3 "" H 5650 2650 50  0000 C CNN
@@
 	6450 3950 6250 3950
 $Comp
-L GNDPWR #PWR052
+L GNDPWR #PWR053
 U 1 1 5879F49C
 P 6450 4200
-F 0 "#PWR052" H 6450 4000 50  0001 C CNN
+F 0 "#PWR053" H 6450 4000 50  0001 C CNN
 F 1 "GNDPWR" H 6450 4070 50  0000 C CNN
 F 2 "" H 6450 4150 50  0000 C CNN
@@
 Connection ~ 4850 3450
 Wire Wire Line
-	3650 3300 5050 3300
+	4300 3300 5050 3300
 Wire Wire Line
 	4300 3450 4300 3300
@@
 Connection ~ 4850 4150
 $Comp
-L +BATT #PWR053
+L +BATT #PWR054
 U 1 1 587A0223
 P 3650 3200
-F 0 "#PWR053" H 3650 3050 50  0001 C CNN
+F 0 "#PWR054" H 3650 3050 50  0001 C CNN
 F 1 "+BATT" H 3650 3340 50  0000 C CNN
 F 2 "" H 3650 3200 50  0000 C CNN
@@
 Connection ~ 7050 4150
 Wire Wire Line
-	7650 3300 7650 3200
+	8600 3300 8600 3150
 Connection ~ 7450 3300
 $Comp
-L +BATT #PWR054
+L +BATT #PWR055
 U 1 1 587A067D
 P 1450 2850
-F 0 "#PWR054" H 1450 2700 50  0001 C CNN
+F 0 "#PWR055" H 1450 2700 50  0001 C CNN
 F 1 "+BATT" H 1450 2990 50  0000 C CNN
 F 2 "" H 1450 2850 50  0000 C CNN
@@
 $EndComp
 $Comp
-L +3.3V #PWR055
+L +3.3V #PWR056
 U 1 1 587A294F
 P 2150 2850
-F 0 "#PWR055" H 2150 2700 50  0001 C CNN
+F 0 "#PWR056" H 2150 2700 50  0001 C CNN
 F 1 "+3.3V" H 2150 2990 50  0000 C CNN
 F 2 "" H 2150 2850 50  0000 C CNN
@@
 	1450 3100 1450 2850
 $Comp
-L +3.3V #PWR056
+L +3.3V #PWR057
 U 1 1 587BA5E2
-P 7650 3200
-F 0 "#PWR056" H 7650 3050 50  0001 C CNN
-F 1 "+3.3V" H 7650 3340 50  0000 C CNN
-F 2 "" H 7650 3200 50  0000 C CNN
-F 3 "" H 7650 3200 50  0000 C CNN
-	1    7650 3200
-	1    0    0    -1
-$EndComp
-$Comp
-L VDDA #PWR057
+P 8600 3150
+F 0 "#PWR057" H 8600 3000 50  0001 C CNN
+F 1 "+3.3V" H 8600 3290 50  0000 C CNN
+F 2 "" H 8600 3150 50  0000 C CNN
+F 3 "" H 8600 3150 50  0000 C CNN
+	1    8600 3150
+	1    0    0    -1
+$EndComp
+$Comp
+L VDDA #PWR058
 U 1 1 587A2978
 P 1850 3000
-F 0 "#PWR057" H 1850 2850 50  0001 C CNN
+F 0 "#PWR058" H 1850 2850 50  0001 C CNN
 F 1 "VDDA" H 1850 3150 50  0000 C CNN
 F 2 "" H 1850 3000 50  0000 C CNN
@@
 	6400 3200 6400 3300
 Connection ~ 6400 3300
+$Comp
+L JUMPER JP1
+U 1 1 58BC8F5E
+P 4000 3300
+F 0 "JP1" H 4000 3450 50  0000 C CNN
+F 1 "JUMPER" H 4000 3220 50  0000 C CNN
+F 2 "Socket_Strips:Socket_Strip_Straight_1x02" H 4000 3300 50  0001 C CNN
+F 3 "" H 4000 3300 50  0000 C CNN
+	1    4000 3300
+	1    0    0    -1
+$EndComp
+Wire Wire Line
+	3700 3300 3650 3300
+$Comp
+L JUMPER JP2
+U 1 1 58BC90EE
+P 7950 3300
+F 0 "JP2" H 7950 3450 50  0000 C CNN
+F 1 "JUMPER" H 7950 3220 50  0000 C CNN
+F 2 "Socket_Strips:Socket_Strip_Straight_1x02" H 7950 3300 50  0001 C CNN
+F 3 "" H 7950 3300 50  0000 C CNN
+	1    7950 3300
+	1    0    0    -1
+$EndComp
+Wire Wire Line
+	8250 3300 8600 3300
 $EndSCHEMATC

Commit message: updated schematics and BOM with MPN
Parts:
- JP1, JP2: MPN (none) -> 969102-0000-DA
- L7: MPN (none) -> XFL4020-102MEC
- R25: MPN (none) -> RR0816P-184-D
- U3: MPN (none) -> TPS630250RNCT
Changed lines of the file:
@@
 F 2 "Octanis3:XFL4020" H 5650 2650 50  0001 C CNN
 F 3 "" H 5650 2650 50  0000 C CNN
+F 4 "XFL4020-102MEC" H 5650 2650 50  0001 C CNN "MPN"
+F 5 "" H 5650 2650 50  0001 C CNN "SKU"
+F 6 "" H 5650 2650 50  0001 C CNN "MouserLink"
 	1    5650 2650
 	0    -1   -1   0
@@
 F 4 "CC0805KKX5R8BB106" H 4330 3750 20  0001 C CNN "MPN"
 F 5 "302010178" H 4330 3750 20  0001 C CNN "SKU"
+F 6 "" H 4330 3750 20  0001 C CNN "" "MouserLink"
 	1    4300 3600
 	0    1    1    0
@@
 F 4 "CC0805MKX5R5BB226" H 7080 3800 20  0001 C CNN "MPN"
 F 5 "302010171" H 7080 3800 20  0001 C CNN "SKU"
+F 6 "" H 7080 3800 20  0001 C CNN "" "MouserLink"
 	1    7050 3650
 	0    1    1    0
@@
 F 4 "CC0805MKX5R5BB226" H 7480 3800 20  0001 C CNN "MPN"
 F 5 "302010171" H 7480 3800 20  0001 C CNN "SKU"
+F 6 "" H 7480 3800 20  0001 C CNN "" "MouserLink"
 	1    7450 3650
 	0    1    1    0
@@
 F 4 "RC0603JR-07560KL" H 6780 3600 20  0001 C CNN "MPN"
 F 5 "301010230" H 6780 3600 20  0001 C CNN "SKU"
+F 6 "" H 6780 3600 20  0001 C CNN "" "MouserLink"
 	1    6750 3450
 	0    -1   -1   0
@@
 F 2 "Resistors_SMD:R_0603" V 6680 3850 50  0001 C CNN
 F 3 "" H 6750 3850 50  0000 C CNN
+F 4 "RR0816P-184-D" H 6750 3850 50  0001 C CNN "MPN"
+F 5 "" H 6750 3850 50  0001 C CNN "SKU"
+F 6 "" H 6750 3850 50  0001 C CNN "MouserLink"
 	1    6750 3850
 	1    0    0    -1
@@
 F 2 "Octanis3:RNC0014A" H 5700 3550 60  0001 C CNN
 F 3 "" H 5700 3550 60  0001 C CNN
+F 4 "TPS630250RNCT" H 5700 3550 60  0001 C CNN "MPN"
+F 5 "" H 5700 3550 60  0001 C CNN "SKU"
+F 6 "" H 5700 3550 60  0001 C CNN "MouserLink"
 	1    5650 3550
 	1    0    0    -1
@@
 F 2 "Socket_Strips:Socket_Strip_Straight_1x03" H 1850 3300 50  0001 C CNN
 F 3 "" H 1850 3300 50  0000 C CNN
+F 4 "" H 1850 3300 50  0001 C CNN "MPN"
+F 5 "" H 1850 3300 50  0001 C CNN "SKU"
+F 6 "" H 1850 3300 50  0001 C CNN "MouserLink"
 	1    1850 3300
 	0    1    1    0
@@
 F 2 "Connectors_Molex:Molex_KK-6410-02_02x2.54mm_Straight" V 3650 3690 50  0001 C CNN
 F 3 "" V 3650 3690 50  0000 C CNN
+F 4 "" V 3650 3690 50  0001 C CNN "MPN"
+F 5 "" V 3650 3690 50  0001 C CNN "SKU"
+F 6 "" V 3650 3690 50  0001 C CNN "MouserLink"
 	1    3650 3650
 	1    0    0    -1
@@
 F 2 "Socket_Strips:Socket_Strip_Straight_1x02" H 4000 3300 50  0001 C CNN
 F 3 "" H 4000 3300 50  0000 C CNN
+F 4 "969102-0000-DA" H 4000 3300 50  0001 C CNN "MPN"
+F 5 "" H 4000 3300 50  0001 C CNN "SKU"
+F 6 "" H 4000 3300 50  0001 C CNN "MouserLink"
 	1    4000 3300
 	1    0    0    -1
@@
 F 2 "Socket_Strips:Socket_Strip_Straight_1x02" H 7950 3300 50  0001 C CNN
 F 3 "" H 7950 3300 50  0000 C CNN
+F 4 "969102-0000-DA" H 7950 3300 50  0001 C CNN "MPN"
+F 5 "" H 7950 3300 50  0001 C CNN "SKU"
+F 6 "" H 7950 3300 50  0001 C CNN "MouserLink"
 	1    7950 3300
 	1    0    0    -1
