File: nestbox_lora.sch (KiCad schematic (older format))
At the start: 1 part, among them U4 RN2483

Commit message: finished component placement incl. LoRa
Parts:
- added ANT_UHF1: ANTENNA-CONN-U-FL_3P_, SeeedOPL-Connector-2016:U-FL3P-SMD-2.6X2.6X1.0MM, symbol ANTENNA-CONN-U-FL_3P_
- added R26: SMD-RES-10K-1%-1_10W_0603_, SeeedOPL-Resistor-2016:R0603, symbol SMD-RES-10K-1%-1_10W_0603_
Connections:
- net +3V3: now also R26.2
- net GND: now also ANT_UHF1.GND1, ANT_UHF1.GND2
- net at U4.23 (RFH): now also ANT_UHF1.D
- net LORA_RST_N: now reaches U4.32 (RESET_N)
- net LORA_RST_N: now also R26.1
Changed lines of the file:
@@
 Wire Wire Line
 	4600 3350 4200 3350
+Wire Wire Line
+	4600 3100 3900 3100
+Text GLabel 3900 3100 0    60   Input ~ 0
+LORA_RST_N
+Wire Wire Line
+	4050 3100 4050 2900
+Connection ~ 4050 3100
+$Comp
+L SMD-RES-10K-1%-1_10W_0603_ R26
+U 1 1 58B96CE5
+P 4050 2750
+F 0 "R26" H 3900 2800 45  0000 L BNN
+F 1 "SMD-RES-10K-1%-1_10W_0603_" H 3900 2650 45  0000 L BNN
+F 2 "SeeedOPL-Resistor-2016:R0603" H 4050 2750 40  0001 C CNN
+F 3 "" H 4050 2750 40  0001 C CNN
+F 4 "RC0603FR-0710KL" H 4080 2900 20  0001 C CNN "MPN"
+F 5 "301010299" H 4080 2900 20  0001 C CNN "SKU"
+	1    4050 2750
+	0    -1   -1   0
+$EndComp
+$Comp
+L +3V3 #PWR073
+U 1 1 58B96D33
+P 4050 2600
+F 0 "#PWR073" H 4050 2450 50  0001 C CNN
+F 1 "+3V3" H 4050 2740 50  0000 C CNN
+F 2 "" H 4050 2600 50  0000 C CNN
+F 3 "" H 4050 2600 50  0000 C CNN
+	1    4050 2600
+	1    0    0    -1
+$EndComp
+$Comp
+L ANTENNA-CONN-U-FL_3P_ ANT_UHF1
+U 1 1 58B96D5F
+P 5550 1750
+F 0 "ANT_UHF1" H 5400 2000 45  0000 L BNN
+F 1 "ANTENNA-CONN-U-FL_3P_" H 5400 1450 45  0000 L BNN
+F 2 "SeeedOPL-Connector-2016:U-FL3P-SMD-2.6X2.6X1.0MM" H 5550 1750 60  0001 C CNN
+F 3 "" H 5550 1750 60  0001 C CNN
+F 4 "320110048" H 5580 1900 20  0001 C CNN "SKU"
+	1    5550 1750
+	0    -1   -1   0
+$EndComp
+Wire Wire Line
+	5550 2050 5550 2350
+$Comp
+L GND #PWR074
+U 1 1 58B96E06
+P 5450 1450
+F 0 "#PWR074" H 5450 1200 50  0001 C CNN
+F 1 "GND" H 5450 1300 50  0000 C CNN
+F 2 "" H 5450 1450 50  0000 C CNN
+F 3 "" H 5450 1450 50  0000 C CNN
+	1    5450 1450
+	-1   0    0    1
+$EndComp
+$Comp
+L GND #PWR075
+U 1 1 58B96E56
+P 5650 1450
+F 0 "#PWR075" H 5650 1200 50  0001 C CNN
+F 1 "GND" H 5650 1300 50  0000 C CNN
+F 2 "" H 5650 1450 50  0000 C CNN
+F 3 "" H 5650 1450 50  0000 C CNN
+	1    5650 1450
+	-1   0    0    1
+$EndComp
 $EndSCHEMATC

Commit message: added additional connector for light barrier
Changed lines of the file:
@@
 	-1   0    0    1
-$EndComp
-$Comp
-L +3V3 #PWR071
-U 1 1 58B953E0
-P 6600 3150
-F 0 "#PWR071" H 6600 3000 50  0001 C CNN
-F 1 "+3V3" H 6600 3290 50  0000 C CNN
-F 2 "" H 6600 3150 50  0000 C CNN
-F 3 "" H 6600 3150 50  0000 C CNN
-	1    6600 3150
-	1    0    0    -1
-$EndComp
-Wire Wire Line
-	6600 3150 6300 3150
-$Comp
-L +3V3 #PWR072
-U 1 1 58B9540E
-P 4200 3350
-F 0 "#PWR072" H 4200 3200 50  0001 C CNN
-F 1 "+3V3" H 4200 3490 50  0000 C CNN
-F 2 "" H 4200 3350 50  0000 C CNN
-F 3 "" H 4200 3350 50  0000 C CNN
-	1    4200 3350
-	1    0    0    -1
 $EndComp
 Wire Wire Line
 	4600 3350 4200 3350
 Wire Wire Line
-	4600 3100 3900 3100
+	3900 3100 4600 3100
 Text GLabel 3900 3100 0    60   Input ~ 0
 LORA_RST_N
@@
 $EndComp
 $Comp
-L +3V3 #PWR073
-U 1 1 58B96D33
-P 4050 2600
-F 0 "#PWR073" H 4050 2450 50  0001 C CNN
-F 1 "+3V3" H 4050 2740 50  0000 C CNN
-F 2 "" H 4050 2600 50  0000 C CNN
-F 3 "" H 4050 2600 50  0000 C CNN
-	1    4050 2600
-	1    0    0    -1
-$EndComp
-$Comp
 L ANTENNA-CONN-U-FL_3P_ ANT_UHF1
 U 1 1 58B96D5F
@@
 	5550 2050 5550 2350
 $Comp
-L GND #PWR074
+L GND #PWR071
 U 1 1 58B96E06
 P 5450 1450
-F 0 "#PWR074" H 5450 1200 50  0001 C CNN
+F 0 "#PWR071" H 5450 1200 50  0001 C CNN
 F 1 "GND" H 5450 1300 50  0000 C CNN
 F 2 "" H 5450 1450 50  0000 C CNN
@@
 $EndComp
 $Comp
-L GND #PWR075
+L GND #PWR072
 U 1 1 58B96E56
 P 5650 1450
-F 0 "#PWR075" H 5650 1200 50  0001 C CNN
+F 0 "#PWR072" H 5650 1200 50  0001 C CNN
 F 1 "GND" H 5650 1300 50  0000 C CNN
 F 2 "" H 5650 1450 50  0000 C CNN
@@
 	-1   0    0    1
 $EndComp
+Wire Wire Line
+	6600 3150 6300 3150
+$Comp
+L +3.3V #PWR073
+U 1 1 58BA812D
+P 4050 2600
+F 0 "#PWR073" H 4050 2450 50  0001 C CNN
+F 1 "+3.3V" H 4050 2740 50  0000 C CNN
+F 2 "" H 4050 2600 50  0000 C CNN
+F 3 "" H 4050 2600 50  0000 C CNN
+	1    4050 2600
+	1    0    0    -1
+$EndComp
+$Comp
+L +3.3V #PWR074
+U 1 1 58BA814A
+P 4200 3350
+F 0 "#PWR074" H 4200 3200 50  0001 C CNN
+F 1 "+3.3V" H 4200 3490 50  0000 C CNN
+F 2 "" H 4200 3350 50  0000 C CNN
+F 3 "" H 4200 3350 50  0000 C CNN
+	1    4200 3350
+	1    0    0    -1
+$EndComp
+$Comp
+L +3.3V #PWR075
+U 1 1 58BA8167
+P 6600 3150
+F 0 "#PWR075" H 6600 3000 50  0001 C CNN
+F 1 "+3.3V" H 6600 3290 50  0000 C CNN
+F 2 "" H 6600 3150 50  0000 C CNN
+F 3 "" H 6600 3150 50  0000 C CNN
+	1    6600 3150
+	1    0    0    -1
+$EndComp
 $EndSCHEMATC

Commit message: updated schematics and BOM with MPN
Parts:
- U4: MPN (none) -> RN2483-I/RM101
Changed lines of the file:
@@
 F 2 "Octanis3:RN2483" H 5450 3350 60  0001 C CNN
 F 3 "" H 5450 3350 60  0001 C CNN
+F 4 "RN2483-I/RM101" H 5450 3350 60  0001 C CNN "MPN"
+F 5 "" H 5450 3350 60  0001 C CNN "SKU"
+F 6 "" H 5450 3350 60  0001 C CNN "MouserLink"
 	1    5450 3400
 	1    0    0    -1
@@
 F 4 "RC0603FR-0710KL" H 4080 2900 20  0001 C CNN "MPN"
 F 5 "301010299" H 4080 2900 20  0001 C CNN "SKU"
+F 6 "" H 4080 2900 20  0001 C CNN "" "MouserLink"
 	1    4050 2750
 	0    -1   -1   0
@@
 F 3 "" H 5550 1750 60  0001 C CNN
 F 4 "320110048" H 5580 1900 20  0001 C CNN "SKU"
+F 6 "" H 5580 1900 20  0001 C CNN "" "MouserLink"
 	1    5550 1750
 	0    -1   -1   0
