File: Nestbox_v2/Nestbox_v2_Comm.sch (KiCad schematic (older format))
At the start: 7 parts

Commit message: Annotated entire schematic
Parts:
- gave numbers to parts that had none: 7
Changed lines of the file:
@@
 $EndDescr
 $Comp
-L RN2483 U?
+L RN2483 U602
 U 1 1 59F64206
 P 8300 4200
-F 0 "U?" H 7750 5150 60  0000 C CNN
+F 0 "U602" H 7750 5150 60  0000 C CNN
 F 1 "RN2483" H 8300 4150 60  0000 C CNN
 F 2 "Octanis3:RN2483" H 8300 4150 60  0001 C CNN
@@
 LORA_TX
 $Comp
-L GND #PWR?
+L GND #PWR0620
 U 1 1 59F64207
 P 9150 4850
-F 0 "#PWR?" H 9150 4600 50  0001 C CNN
+F 0 "#PWR0620" H 9150 4600 50  0001 C CNN
 F 1 "GND" H 9150 4700 50  0000 C CNN
 F 2 "" H 9150 4850 50  0000 C CNN
@@
 $EndComp
 $Comp
-L GND #PWR?
+L GND #PWR0619
 U 1 1 59F64208
 P 7450 4850
-F 0 "#PWR?" H 7450 4600 50  0001 C CNN
+F 0 "#PWR0619" H 7450 4600 50  0001 C CNN
 F 1 "GND" H 7450 4700 50  0000 C CNN
 F 2 "" H 7450 4850 50  0000 C CNN
@@
 $EndComp
 $Comp
-L GND #PWR?
+L GND #PWR0618
 U 1 1 59F64209
 P 7450 4550
-F 0 "#PWR?" H 7450 4300 50  0001 C CNN
+F 0 "#PWR0618" H 7450 4300 50  0001 C CNN
 F 1 "GND" H 7450 4400 50  0000 C CNN
 F 2 "" H 7450 4550 50  0000 C CNN
@@
 $EndComp
 $Comp
-L GND #PWR?
+L GND #PWR0614
 U 1 1 59F6420A
 P 7450 4050
-F 0 "#PWR?" H 7450 3800 50  0001 C CNN
+F 0 "#PWR0614" H 7450 3800 50  0001 C CNN
 F 1 "GND" H 7450 3900 50  0000 C CNN
 F 2 "" H 7450 4050 50  0000 C CNN
@@
 $EndComp
 $Comp
-L GND #PWR?
+L GND #PWR0611
 U 1 1 59F6420B
 P 7450 3700
-F 0 "#PWR?" H 7450 3450 50  0001 C CNN
+F 0 "#PWR0611" H 7450 3450 50  0001 C CNN
 F 1 "GND" H 7450 3550 50  0000 C CNN
 F 2 "" H 7450 3700 50  0000 C CNN
@@
 $EndComp
 $Comp
-L GND #PWR?
+L GND #PWR0612
 U 1 1 59F6420C
 P 9150 3700
-F 0 "#PWR?" H 9150 3450 50  0001 C CNN
+F 0 "#PWR0612" H 9150 3450 50  0001 C CNN
 F 1 "GND" H 9150 3550 50  0000 C CNN
 F 2 "" H 9150 3700 50  0000 C CNN
@@
 $EndComp
 $Comp
-L GND #PWR?
+L GND #PWR0615
 U 1 1 59F6420D
 P 9150 4100
-F 0 "#PWR?" H 9150 3850 50  0001 C CNN
+F 0 "#PWR0615" H 9150 3850 50  0001 C CNN
 F 1 "GND" H 9150 3950 50  0000 C CNN
 F 2 "" H 9150 4100 50  0000 C CNN
@@
 $EndComp
 $Comp
-L GND #PWR?
+L GND #PWR0617
 U 1 1 59F6420E
 P 9150 4250
-F 0 "#PWR?" H 9150 4000 50  0001 C CNN
+F 0 "#PWR0617" H 9150 4000 50  0001 C CNN
 F 1 "GND" H 9150 4100 50  0000 C CNN
 F 2 "" H 9150 4250 50  0000 C CNN
@@
 $EndComp
 $Comp
-L GND #PWR?
+L GND #PWR0609
 U 1 1 59F6420F
 P 8600 3150
-F 0 "#PWR?" H 8600 2900 50  0001 C CNN
+F 0 "#PWR0609" H 8600 2900 50  0001 C CNN
 F 1 "GND" H 8600 3000 50  0000 C CNN
 F 2 "" H 8600 3150 50  0000 C CNN
@@
 $EndComp
 $Comp
-L GND #PWR?
+L GND #PWR0608
 U 1 1 59F64210
 P 8500 3150
-F 0 "#PWR?" H 8500 2900 50  0001 C CNN
+F 0 "#PWR0608" H 8500 2900 50  0001 C CNN
 F 1 "GND" H 8500 3000 50  0000 C CNN
 F 2 "" H 8500 3150 50  0000 C CNN
@@
 $EndComp
 $Comp
-L GND #PWR?
+L GND #PWR0607
 U 1 1 59F64211
 P 8300 3150
-F 0 "#PWR?" H 8300 2900 50  0001 C CNN
+F 0 "#PWR0607" H 8300 2900 50  0001 C CNN
 F 1 "GND" H 8300 3000 50  0000 C CNN
 F 2 "" H 8300 3150 50  0000 C CNN
@@
 $EndComp
 $Comp
-L GND #PWR?
+L GND #PWR0606
 U 1 1 59F64212
 P 8100 3150
-F 0 "#PWR?" H 8100 2900 50  0001 C CNN
+F 0 "#PWR0606" H 8100 2900 50  0001 C CNN
 F 1 "GND" H 8100 3000 50  0000 C CNN
 F 2 "" H 8100 3150 50  0000 C CNN
@@
 $EndComp
 $Comp
-L GND #PWR?
+L GND #PWR0605
 U 1 1 59F64213
 P 8000 3150
-F 0 "#PWR?" H 8000 2900 50  0001 C CNN
+F 0 "#PWR0605" H 8000 2900 50  0001 C CNN
 F 1 "GND" H 8000 3000 50  0000 C CNN
 F 2 "" H 8000 3150 50  0000 C CNN
@@
 Connection ~ 6900 3900
 $Comp
-L ANTENNA-CONN-U-FL_3P_ ANT_UHF?
+L ANTENNA-CONN-U-FL_3P_ ANT_UHF601
 U 1 1 59F64215
 P 8400 2550
-F 0 "ANT_UHF?" H 8250 2800 45  0000 L BNN
+F 0 "ANT_UHF601" H 8250 2800 45  0000 L BNN
 F 1 "ANTENNA-CONN-U-FL_3P_" H 8250 2250 45  0000 L BNN
 F 2 "SeeedOPL-Connector-2016:U-FL3P-SMD-2.6X2.6X1.0MM" H 8400 2550 60  0001 C CNN
@@
 	8400 2850 8400 3150
 $Comp
-L GND #PWR?
+L GND #PWR0603
 U 1 1 59F64216
 P 8300 2250
-F 0 "#PWR?" H 8300 2000 50  0001 C CNN
+F 0 "#PWR0603" H 8300 2000 50  0001 C CNN
 F 1 "GND" H 8300 2100 50  0000 C CNN
 F 2 "" H 8300 2250 50  0000 C CNN
@@
 $EndComp
 $Comp
-L GND #PWR?
+L GND #PWR0604
 U 1 1 59F64217
 P 8500 2250
-F 0 "#PWR?" H 8500 2000 50  0001 C CNN
+F 0 "#PWR0604" H 8500 2000 50  0001 C CNN
 F 1 "GND" H 8500 2100 50  0000 C CNN
 F 2 "" H 8500 2250 50  0000 C CNN
@@
 	9450 3950 9150 3950
 $Comp
-L +3.3V #PWR?
+L +3.3V #PWR0610
 U 1 1 59F64218
 P 6900 3400
-F 0 "#PWR?" H 6900 3250 50  0001 C CNN
+F 0 "#PWR0610" H 6900 3250 50  0001 C CNN
 F 1 "+3.3V" H 6900 3540 50  0000 C CNN
 F 2 "" H 6900 3400 50  0000 C CNN
@@
 $EndComp
 $Comp
-L +3.3V #PWR?
+L +3.3V #PWR0616
 U 1 1 59F64219
 P 7050 4150
-F 0 "#PWR?" H 7050 4000 50  0001 C CNN
+F 0 "#PWR0616" H 7050 4000 50  0001 C CNN
 F 1 "+3.3V" H 7050 4290 50  0000 C CNN
 F 2 "" H 7050 4150 50  0000 C CNN
@@
 $EndComp
 $Comp
-L +3.3V #PWR?
+L +3.3V #PWR0613
 U 1 1 59F6421A
 P 9450 3950
-F 0 "#PWR?" H 9450 3800 50  0001 C CNN
+F 0 "#PWR0613" H 9450 3800 50  0001 C CNN
 F 1 "+3.3V" H 9450 4090 50  0000 C CNN
 F 2 "" H 9450 3950 50  0000 C CNN
@@
 Connection ~ 3200 1550
 $Comp
-L GND #PWR?
+L GND #PWR0602
 U 1 1 59FDFCD3
 P 3200 1750
-F 0 "#PWR?" H 3200 1500 50  0001 C CNN
+F 0 "#PWR0602" H 3200 1500 50  0001 C CNN
 F 1 "GND" H 3205 1577 50  0000 C CNN
 F 2 "" H 3200 1750 50  0000 C CNN
@@
 DATA_TX
 $Comp
-L XBee-S2C-802.15.4_SMT U?
+L XBee-S2C-802.15.4_SMT U601
 U 1 1 59FE0508
 P 3950 1050
-F 0 "U?" H 4325 1197 60  0000 C CNN
+F 0 "U601" H 4325 1197 60  0000 C CNN
 F 1 "XBee-S2C-802.15.4_SMT" H 4325 1091 60  0000 C CNN
 F 2 "" H 3950 1050 60  0001 C CNN
@@
 $EndComp
 $Comp
-L Q_PMOS_DGS Q?
+L Q_PMOS_DGS Q601
 U 1 1 59FE0AF1
 P 1750 1450
-F 0 "Q?" H 1956 1496 50  0000 L CNN
+F 0 "Q601" H 1956 1496 50  0000 L CNN
 F 1 "Q_PMOS_DGS" H 1956 1405 50  0000 L CNN
 F 2 "" H 1950 1550 50  0000 C CNN
@@
 $EndComp
 $Comp
-L +3.3V #PWR?
+L +3.3V #PWR0601
 U 1 1 59FE0C6C
 P 1850 1200
-F 0 "#PWR?" H 1850 1050 50  0001 C CNN
+F 0 "#PWR0601" H 1850 1050 50  0001 C CNN
 F 1 "+3.3V" H 1865 1373 50  0000 C CNN
 F 2 "" H 1850 1200 50  0000 C CNN
@@
 DATA_Enable_N
 $Comp
-L R R?
+L R R601
 U 1 1 59FF56E8
 P 6900 3550
-F 0 "R?" H 6970 3596 50  0000 L CNN
+F 0 "R601" H 6970 3596 50  0000 L CNN
 F 1 "10K" H 6970 3505 50  0000 L CNN
 F 2 "" V 6830 3550 50  0000 C CNN
@@
 $EndComp
 $Comp
-L ESP-12S U?
+L ESP-12S U603
 U 1 1 59FF5CBB
 P 2800 5050
-F 0 "U?" H 3200 5237 60  0000 C CNN
+F 0 "U603" H 3200 5237 60  0000 C CNN
 F 1 "ESP-12S" H 3200 5131 60  0000 C CNN
 F 2 "" H 2800 5050 60  0001 C CNN
@@
 NoConn ~ 3700 5700
 $Comp
-L R R?
+L R R602
 U 1 1 59FF5E36
 P 2550 5300
-F 0 "R?" H 2620 5346 50  0000 L CNN
+F 0 "R602" H 2620 5346 50  0000 L CNN
 F 1 "10K" H 2620 5255 50  0000 L CNN
 F 2 "" V 2480 5300 50  0000 C CNN
@@
 $EndComp
 $Comp
-L +3.3V #PWR?
+L +3.3V #PWR0621
 U 1 1 59FF5EE6
 P 2550 5100
-F 0 "#PWR?" H 2550 4950 50  0001 C CNN
+F 0 "#PWR0621" H 2550 4950 50  0001 C CNN
 F 1 "+3.3V" H 2565 5273 50  0000 C CNN
 F 2 "" H 2550 5100 50  0000 C CNN
@@
 	2550 5500 2700 5500
 $Comp
-L +3.3V #PWR?
+L +3.3V #PWR0622
 U 1 1 59FF5FCD
 P 2550 6200
-F 0 "#PWR?" H 2550 6050 50  0001 C CNN
+F 0 "#PWR0622" H 2550 6050 50  0001 C CNN
 F 1 "+3.3V" V 2565 6328 50  0000 L CNN
 F 2 "" H 2550 6200 50  0000 C CNN
@@
 	2550 6200 2700 6200
 $Comp
-L GND #PWR?
+L GND #PWR0623
 U 1 1 59FF60B0
 P 3900 6200
-F 0 "#PWR?" H 3900 5950 50  0001 C CNN
+F 0 "#PWR0623" H 3900 5950 50  0001 C CNN
 F 1 "GND" V 3905 6072 50  0000 R CNN
 F 2 "" H 3900 6200 50  0000 C CNN
