File: Nestbox_v2/Nestbox_v2_Comm.sch (KiCad schematic (older format))
At the start: 11 parts, among them J501 CONN_01X01, J502 CONN_01X06, Q501 NTR3A052PZT1G, U501 ESP-12S

Commit message: corrected transistor pins
Parts:
- removed Q501: NTR3A052PZT1G, TO_SOT_Packages_SMD:SOT-23, symbol Q_PMOS_DGS
- added Q501: NTR3A052PZT1G, TO_SOT_Packages_SMD:TSOT-23, symbol Q_PMOS_GSD
Connections:
- net +3V3: now also Q501.3 (D)
- net ESP12_ENABLE: now also Q501.1 (G)
- net ESP12_VCC: now also Q501.2 (S)
Changed lines of the file:
@@
 $EndComp
 $Comp
-L GND #PWR048
+L GND #PWR502
 U 1 1 59FF60B0
 P 4300 6250
-F 0 "#PWR048" H 4300 6000 50  0001 C CNN
+F 0 "#PWR502" H 4300 6000 50  0001 C CNN
 F 1 "GND" V 4305 6122 50  0000 R CNN
 F 2 "" H 4300 6250 50  0000 C CNN
@@
 $EndComp
 $Comp
-L +3.3V #PWR049
+L +3.3V #PWR503
 U 1 1 59F64218
 P 6900 3400
-F 0 "#PWR049" H 6900 3250 50  0001 C CNN
+F 0 "#PWR503" H 6900 3250 50  0001 C CNN
 F 1 "+3.3V" H 6900 3540 50  0000 C CNN
 F 2 "" H 6900 3400 50  0000 C CNN
@@
 $EndComp
 $Comp
-L +3.3V #PWR050
+L +3.3V #PWR501
 U 1 1 5B158F7F
 P 3300 2650
-F 0 "#PWR050" H 3300 2500 50  0001 C CNN
+F 0 "#PWR501" H 3300 2500 50  0001 C CNN
 F 1 "+3.3V" H 3315 2823 50  0000 C CNN
 F 2 "" H 3300 2650 50  0000 C CNN
@@
 Text Label 4000 5900 0    60   ~ 0
 DTR
-$Comp
-L Q_PMOS_DGS Q501
-U 1 1 5B1510D8
-P 3200 2950
-F 0 "Q501" H 3400 3000 50  0000 L CNN
-F 1 "NTR3A052PZT1G" H 3400 2900 50  0000 L CNN
-F 2 "TO_SOT_Packages_SMD:SOT-23" H 3400 3050 50  0001 C CNN
-F 3 "" H 3200 2950 50  0001 C CNN
-	1    3200 2950
-	1    0    0    -1
-$EndComp
 Text Label 3300 3300 3    60   ~ 0
 ESP12_VCC
@@
 Text Label 2550 6200 2    60   ~ 0
 ESP12_VCC
+$Comp
+L Q_PMOS_GSD Q501
+U 1 1 5B18B1E8
+P 3200 2950
+F 0 "Q501" H 3400 3000 50  0000 L CNN
+F 1 "NTR3A052PZT1G" H 3400 2900 50  0000 L CNN
+F 2 "TO_SOT_Packages_SMD:TSOT-23" H 3400 3050 50  0001 C CNN
+F 3 "" H 3200 2950 50  0001 C CNN
+	1    3200 2950
+	1    0    0    -1
+$EndComp
 $EndSCHEMATC

Commit message: annotated schematic with necessary changes to load cell circuit. added pull-ups for enable PMOSes
Parts:
- added R?: 82k, Resistors_SMD:R_0603, symbol R
Connections:
- net +3V3: now also R?.1
- net ESP12_ENABLE: now also R?.2
Changed lines of the file:
@@
+	1    0    0    -1
+$EndComp
+$Comp
+L R R?
+U 1 1 5B28C223
+P 2950 2750
+F 0 "R?" H 3020 2796 50  0000 L CNN
+F 1 "82k" H 3020 2705 50  0000 L CNN
+F 2 "Resistors_SMD:R_0603" V 2880 2750 50  0001 C CNN
+F 3 "" H 2950 2750 50  0000 C CNN
+	1    2950 2750
+	1    0    0    -1
+$EndComp
+Wire Wire Line
+	2950 2900 2950 2950
+Connection ~ 2950 2950
+$Comp
+L +3.3V #PWR?
+U 1 1 5B28C2B7
+P 2950 2600
+F 0 "#PWR?" H 2950 2450 50  0001 C CNN
+F 1 "+3.3V" H 2965 2773 50  0000 C CNN
+F 2 "" H 2950 2600 50  0000 C CNN
+F 3 "" H 2950 2600 50  0000 C CNN
+	1    2950 2600
 	1    0    0    -1
 $EndComp

Commit message: TAPEOUT second batch nestbox main + EM pcb. added pull-ups, corrected pmos of load cell, WIFI AND SDCARD ENABLE PMOS ARE STILL WRONGLY ORIENTED
Parts:
- R502: value 10K -> 82k
- gave numbers to parts that had none: 1
Changed lines of the file:
@@
 $EndComp
 $Comp
-L GND #PWR502
+L GND #PWR503
 U 1 1 59FF60B0
 P 4300 6250
-F 0 "#PWR502" H 4300 6000 50  0001 C CNN
+F 0 "#PWR503" H 4300 6000 50  0001 C CNN
 F 1 "GND" V 4305 6122 50  0000 R CNN
 F 2 "" H 4300 6250 50  0000 C CNN
@@
 P 6900 3550
 F 0 "R502" H 6970 3596 50  0000 L CNN
-F 1 "10K" H 6970 3505 50  0000 L CNN
+F 1 "82k" H 6970 3505 50  0000 L CNN
 F 2 "Resistors_SMD:R_0603" V 6830 3550 50  0001 C CNN
 F 3 "" H 6900 3550 50  0000 C CNN
@@
 $EndComp
 $Comp
-L +3.3V #PWR503
+L +3.3V #PWR504
 U 1 1 59F64218
 P 6900 3400
-F 0 "#PWR503" H 6900 3250 50  0001 C CNN
+F 0 "#PWR504" H 6900 3250 50  0001 C CNN
 F 1 "+3.3V" H 6900 3540 50  0000 C CNN
 F 2 "" H 6900 3400 50  0000 C CNN
@@
 $EndComp
 $Comp
-L +3.3V #PWR501
+L +3.3V #PWR502
 U 1 1 5B158F7F
 P 3300 2650
-F 0 "#PWR501" H 3300 2500 50  0001 C CNN
+F 0 "#PWR502" H 3300 2500 50  0001 C CNN
 F 1 "+3.3V" H 3315 2823 50  0000 C CNN
 F 2 "" H 3300 2650 50  0000 C CNN
@@
 $EndComp
 $Comp
-L R R?
+L R R507
 U 1 1 5B28C223
 P 2950 2750
-F 0 "R?" H 3020 2796 50  0000 L CNN
+F 0 "R507" H 3020 2796 50  0000 L CNN
 F 1 "82k" H 3020 2705 50  0000 L CNN
 F 2 "Resistors_SMD:R_0603" V 2880 2750 50  0001 C CNN
@@
 Connection ~ 2950 2950
 $Comp
-L +3.3V #PWR?
+L +3.3V #PWR501
 U 1 1 5B28C2B7
 P 2950 2600
-F 0 "#PWR?" H 2950 2450 50  0001 C CNN
+F 0 "#PWR501" H 2950 2450 50  0001 C CNN
 F 1 "+3.3V" H 2965 2773 50  0000 C CNN
 F 2 "" H 2950 2600 50  0000 C CNN

Commit message: various annotations and changes
Other:
- note added: "!! PMOS IS INVERTED !!\n"
Changed lines of the file:
@@
 	1    0    0    -1
 $EndComp
+Text Notes 2450 2150 0    118  ~ 0
+!! PMOS IS INVERTED !!\n
 $EndSCHEMATC
