File: Nestbox_v2/Nestbox_v2_RFID.sch (KiCad schematic (older format))
At the start: 10 parts, among them U401 MLX90109

Commit message: Annotated entire schematic
Parts:
- gave numbers to parts that had none: 1
- renumbered R402 to R401, R403 to R402
Changed lines of the file:
@@
 	4200 3650 4800 3650
 $Comp
-L R R403
+L R R402
 U 1 1 59EF80B5
 P 4500 4550
-F 0 "R403" V 4580 4550 50  0000 C CNN
+F 0 "R402" V 4580 4550 50  0000 C CNN
 F 1 "36k" V 4500 4550 50  0000 C CNN
 F 2 "" V 4430 4550 50  0001 C CNN
@@
 $EndComp
 $Comp
-L R R402
+L R R401
 U 1 1 59EF815C
 P 4100 3950
-F 0 "R402" V 4180 3950 50  0000 C CNN
+F 0 "R401" V 4180 3950 50  0000 C CNN
 F 1 "100k" V 4100 3950 50  0000 C CNN
 F 2 "" V 4030 3950 50  0001 C CNN
@@
 Connection ~ 5850 2300
 $Comp
-L +3.3V #PWR401
+L +3.3V #PWR0402
 U 1 1 59FF36B1
 P 9200 2450
-F 0 "#PWR401" H 9200 2300 50  0001 C CNN
+F 0 "#PWR0402" H 9200 2300 50  0001 C CNN
 F 1 "+3.3V" V 9215 2578 50  0000 L CNN
 F 2 "" H 9200 2450 50  0000 C CNN
@@
 RFID_VDD
 $Comp
-L Jumper_SELECT_Dual JP?
+L Jumper_SELECT_Dual JP401
 U 1 1 5A0303B0
 P 8950 2450
-F 0 "JP?" H 8950 2689 50  0000 C CNN
+F 0 "JP401" H 8950 2689 50  0000 C CNN
 F 1 "Jumper_SELECT_Dual" H 8950 2598 50  0000 C CNN
 F 2 "" H 8950 2450 50  0001 C CNN
@@
 RFID_VDD
 $Comp
-L +5V #PWR?
+L +5V #PWR0401
 U 1 1 5A0305A8
 P 8700 2450
-F 0 "#PWR?" H 8700 2300 50  0001 C CNN
+F 0 "#PWR0401" H 8700 2300 50  0001 C CNN
 F 1 "+5V" V 8715 2578 50  0000 L CNN
 F 2 "" H 8700 2450 50  0001 C CNN
@@
 TODO: Check Modu voltage levels\nFor 3.3V VDD and 5V VDD
 $Comp
-L GND #PWR?
+L GND #PWR0403
 U 1 1 5A0312F4
 P 4200 3650
-F 0 "#PWR?" H 4200 3400 50  0001 C CNN
+F 0 "#PWR0403" H 4200 3400 50  0001 C CNN
 F 1 "GND" V 4205 3522 50  0000 R CNN
 F 2 "" H 4200 3650 50  0001 C CNN
