File: Nestbox_v2/Nestbox_v2_detector.sch (KiCad schematic (older format))
At the start: 0 parts

Commit message: Adds schamtic of light barriers
- Light barriers using SFH4656 as emitter and RSOP38 as detector.
- Includes separate Connector to solder remote LED
Parts:
- added D? (x2): OSRAM_SFH4656, symbol OSRAM_SFH4656
- added P? (x2): CONN_01X02, symbol CONN_01X02
- added R? (x2): R, symbol R
- added U? (x2): TSOP38, symbol TSOP38
Connections:
- new net: D?.2 (C), P?.1 (P1), R?.1 (x2)
- new net +3V3: U?.3 (VS), U?.3 (VS)
- new net GND: R?.2, R?.2, U?.2 (GND), U?.2 (GND)
- new net LB1_DETECT: U?.1 (OUT)
- new net LB1_LED: D?.1 (A), P?.2 (P2)
- new net LB2_DETECT: U?.1 (OUT)
- new net LB2_LED: D?.1 (A), P?.2 (P2)
Changed lines of the file:
@@
 $Descr A4 11693 8268
 encoding utf-8
-Sheet 1 6
+Sheet 5 6
 Title ""
 Date ""
@@
 Comment4 ""
 $EndDescr
+$Comp
+L TSOP38 U?
+U 1 1 59FCFE81
+P 3500 1600
+F 0 "U?" H 3677 1358 60  0000 L CNN
+F 1 "TSOP38" H 3677 1252 60  0000 L CNN
+F 2 "" H 3500 1600 60  0001 C CNN
+F 3 "" H 3500 1600 60  0001 C CNN
+	1    3500 1600
+	1    0    0    -1
+$EndComp
+$Comp
+L TSOP38 U?
+U 1 1 59FCFEFD
+P 3500 2600
+F 0 "U?" H 3677 2358 60  0000 L CNN
+F 1 "TSOP38" H 3677 2252 60  0000 L CNN
+F 2 "" H 3500 2600 60  0001 C CNN
+F 3 "" H 3500 2600 60  0001 C CNN
+	1    3500 2600
+	1    0    0    -1
+$EndComp
+$Comp
+L +3.3V #PWR?
+U 1 1 59FD02D9
+P 3200 1750
+F 0 "#PWR?" H 3200 1600 50  0001 C CNN
+F 1 "+3.3V" V 3215 1878 50  0000 L CNN
+F 2 "" H 3200 1750 50  0000 C CNN
+F 3 "" H 3200 1750 50  0000 C CNN
+	1    3200 1750
+	0    -1   -1   0
+$EndComp
+$Comp
+L +3.3V #PWR?
+U 1 1 59FD02F5
+P 3200 2750
+F 0 "#PWR?" H 3200 2600 50  0001 C CNN
+F 1 "+3.3V" V 3215 2878 50  0000 L CNN
+F 2 "" H 3200 2750 50  0000 C CNN
+F 3 "" H 3200 2750 50  0000 C CNN
+	1    3200 2750
+	0    -1   -1   0
+$EndComp
+$Comp
+L GND #PWR?
+U 1 1 59FD0355
+P 3200 1900
+F 0 "#PWR?" H 3200 1650 50  0001 C CNN
+F 1 "GND" V 3205 1772 50  0000 R CNN
+F 2 "" H 3200 1900 50  0000 C CNN
+F 3 "" H 3200 1900 50  0000 C CNN
+	1    3200 1900
+	0    1    1    0
+$EndComp
+$Comp
+L GND #PWR?
+U 1 1 59FD0371
+P 3200 2900
+F 0 "#PWR?" H 3200 2650 50  0001 C CNN
+F 1 "GND" V 3205 2772 50  0000 R CNN
+F 2 "" H 3200 2900 50  0000 C CNN
+F 3 "" H 3200 2900 50  0000 C CNN
+	1    3200 2900
+	0    1    1    0
+$EndComp
+Text GLabel 3200 2050 0    60   Input ~ 0
+LB1_DETECT
+Text GLabel 3200 3050 0    60   Input ~ 0
+LB2_DETECT
+$Comp
+L OSRAM_SFH4656 D?
+U 1 1 59FDE056
+P 5050 1850
+F 0 "D?" V 5088 1732 50  0000 R CNN
+F 1 "OSRAM_SFH4656" V 4997 1732 50  0000 R CNN
+F 2 "" H 5050 1850 50  0000 C CNN
+F 3 "" H 5050 1850 50  0000 C CNN
+	1    5050 1850
+	0    -1   -1   0
+$EndComp
+$Comp
+L OSRAM_SFH4656 D?
+U 1 1 59FDE0CE
+P 5050 2900
+F 0 "D?" V 5088 2782 50  0000 R CNN
+F 1 "OSRAM_SFH4656" V 4997 2782 50  0000 R CNN
+F 2 "" H 5050 2900 50  0000 C CNN
+F 3 "" H 5050 2900 50  0000 C CNN
+	1    5050 2900
+	0    -1   -1   0
+$EndComp
+$Comp
+L R R?
+U 1 1 59FDE229
+P 5050 2250
+F 0 "R?" H 5120 2296 50  0000 L CNN
+F 1 "R" H 5120 2205 50  0000 L CNN
+F 2 "" V 4980 2250 50  0000 C CNN
+F 3 "" H 5050 2250 50  0000 C CNN
+	1    5050 2250
+	1    0    0    -1
+$EndComp
+$Comp
+L R R?
+U 1 1 59FDE287
+P 5050 3300
+F 0 "R?" H 5120 3346 50  0000 L CNN
+F 1 "R" H 5120 3255 50  0000 L CNN
+F 2 "" V 4980 3300 50  0000 C CNN
+F 3 "" H 5050 3300 50  0000 C CNN
+	1    5050 3300
+	1    0    0    -1
+$EndComp
+Wire Wire Line
+	5050 3050 5050 3150
+Wire Wire Line
+	5050 3450 5050 3550
+Wire Wire Line
+	5050 3550 5500 3550
+Wire Wire Line
+	5050 2750 5050 2650
+Wire Wire Line
+	4800 2650 5500 2650
+Wire Wire Line
+	5050 1700 5050 1600
+Wire Wire Line
+	4800 1600 5500 1600
+Wire Wire Line
+	5050 2000 5050 2100
+$Comp
+L CONN_01X02 P?
+U 1 1 59FDE676
+P 4600 1850
+F 0 "P?" H 4519 1575 50  0000 C CNN
+F 1 "CONN_01X02" H 4519 1666 50  0000 C CNN
+F 2 "" H 4600 1850 50  0000 C CNN
+F 3 "" H 4600 1850 50  0000 C CNN
+	1    4600 1850
+	-1   0    0    1
+$EndComp
+Connection ~ 5050 2050
+Wire Wire Line
+	4800 1800 4800 1600
+Connection ~ 5050 1600
+Wire Wire Line
+	4800 1900 4800 2050
+Wire Wire Line
+	4800 2050 5050 2050
+$Comp
+L CONN_01X02 P?
+U 1 1 59FDE836
+P 4600 2900
+F 0 "P?" H 4519 2625 50  0000 C CNN
+F 1 "CONN_01X02" H 4519 2716 50  0000 C CNN
+F 2 "" H 4600 2900 50  0000 C CNN
+F 3 "" H 4600 2900 50  0000 C CNN
+	1    4600 2900
+	-1   0    0    1
+$EndComp
+Wire Wire Line
+	4800 2850 4800 2650
+Connection ~ 5050 2650
+Wire Wire Line
+	4800 2950 4800 3100
+Wire Wire Line
+	4800 3100 5050 3100
+Connection ~ 5050 3100
+Wire Wire Line
+	5050 2400 5050 2500
+Wire Wire Line
+	5050 2500 5500 2500
+$Comp
+L GND #PWR?
+U 1 1 59FDEA04
+P 5500 2500
+F 0 "#PWR?" H 5500 2250 50  0001 C CNN
+F 1 "GND" V 5505 2372 50  0000 R CNN
+F 2 "" H 5500 2500 50  0000 C CNN
+F 3 "" H 5500 2500 50  0000 C CNN
+	1    5500 2500
+	0    -1   -1   0
+$EndComp
+$Comp
+L GND #PWR?
+U 1 1 59FDEA3E
+P 5500 3550
+F 0 "#PWR?" H 5500 3300 50  0001 C CNN
+F 1 "GND" V 5505 3422 50  0000 R CNN
+F 2 "" H 5500 3550 50  0000 C CNN
+F 3 "" H 5500 3550 50  0000 C CNN
+	1    5500 3550
+	0    -1   -1   0
+$EndComp
+Text GLabel 5500 1600 2    60   Input ~ 0
+LB1_LED
+Text GLabel 5500 2650 2    60   Input ~ 0
+LB2_LED
 $EndSCHEMATC

Commit message: Adds decoupling to TSOP38
- Electrical overstress (EOS) protection was added to TSOP38.
- Detection schematic was annotated.
Parts:
- added C1, C2: 1u, symbol C
- added R1, R3: 100E, symbol R
- gave numbers to parts that had none: 8
Connections:
- net +3V3: now also C1.1, C2.1, R1.2, R3.2; no longer U1.3 (VS), U2.3 (VS)
- net GND: now also C1.2, C2.2
- new net: R1.1, U1.3 (VS)
- new net: R3.1, U2.3 (VS)
Changed lines of the file:
@@
 $EndDescr
 $Comp
-L TSOP38 U?
+L TSOP38 U1
 U 1 1 59FCFE81
 P 3500 1600
-F 0 "U?" H 3677 1358 60  0000 L CNN
+F 0 "U1" H 3677 1358 60  0000 L CNN
 F 1 "TSOP38" H 3677 1252 60  0000 L CNN
 F 2 "" H 3500 1600 60  0001 C CNN
@@
 $EndComp
 $Comp
-L TSOP38 U?
+L TSOP38 U2
 U 1 1 59FCFEFD
 P 3500 2600
-F 0 "U?" H 3677 2358 60  0000 L CNN
+F 0 "U2" H 3677 2358 60  0000 L CNN
 F 1 "TSOP38" H 3677 2252 60  0000 L CNN
 F 2 "" H 3500 2600 60  0001 C CNN
@@
 $EndComp
 $Comp
-L +3.3V #PWR?
+L +3.3V #PWR1
 U 1 1 59FD02D9
-P 3200 1750
-F 0 "#PWR?" H 3200 1600 50  0001 C CNN
-F 1 "+3.3V" V 3215 1878 50  0000 L CNN
-F 2 "" H 3200 1750 50  0000 C CNN
-F 3 "" H 3200 1750 50  0000 C CNN
-	1    3200 1750
-	0    -1   -1   0
-$EndComp
-$Comp
-L +3.3V #PWR?
-U 1 1 59FD02F5
-P 3200 2750
-F 0 "#PWR?" H 3200 2600 50  0001 C CNN
-F 1 "+3.3V" V 3215 2878 50  0000 L CNN
-F 2 "" H 3200 2750 50  0000 C CNN
-F 3 "" H 3200 2750 50  0000 C CNN
-	1    3200 2750
-	0    -1   -1   0
-$EndComp
-$Comp
-L GND #PWR?
+P 2100 1750
+F 0 "#PWR1" H 2100 1600 50  0001 C CNN
+F 1 "+3.3V" V 2115 1878 50  0000 L CNN
+F 2 "" H 2100 1750 50  0000 C CNN
+F 3 "" H 2100 1750 50  0000 C CNN
+	1    2100 1750
+	0    -1   -1   0
+$EndComp
+$Comp
+L GND #PWR2
 U 1 1 59FD0355
-P 3200 1900
-F 0 "#PWR?" H 3200 1650 50  0001 C CNN
-F 1 "GND" V 3205 1772 50  0000 R CNN
-F 2 "" H 3200 1900 50  0000 C CNN
-F 3 "" H 3200 1900 50  0000 C CNN
-	1    3200 1900
-	0    1    1    0
-$EndComp
-$Comp
-L GND #PWR?
-U 1 1 59FD0371
-P 3200 2900
-F 0 "#PWR?" H 3200 2650 50  0001 C CNN
-F 1 "GND" V 3205 2772 50  0000 R CNN
-F 2 "" H 3200 2900 50  0000 C CNN
-F 3 "" H 3200 2900 50  0000 C CNN
-	1    3200 2900
+P 2100 2050
+F 0 "#PWR2" H 2100 1800 50  0001 C CNN
+F 1 "GND" V 2105 1922 50  0000 R CNN
+F 2 "" H 2100 2050 50  0000 C CNN
+F 3 "" H 2100 2050 50  0000 C CNN
+	1    2100 2050
 	0    1    1    0
 $EndComp
@@
 LB2_DETECT
 $Comp
-L OSRAM_SFH4656 D?
+L OSRAM_SFH4656 D1
 U 1 1 59FDE056
 P 5050 1850
-F 0 "D?" V 5088 1732 50  0000 R CNN
+F 0 "D1" V 5088 1732 50  0000 R CNN
 F 1 "OSRAM_SFH4656" V 4997 1732 50  0000 R CNN
 F 2 "" H 5050 1850 50  0000 C CNN
@@
 $EndComp
 $Comp
-L OSRAM_SFH4656 D?
+L OSRAM_SFH4656 D2
 U 1 1 59FDE0CE
 P 5050 2900
-F 0 "D?" V 5088 2782 50  0000 R CNN
+F 0 "D2" V 5088 2782 50  0000 R CNN
 F 1 "OSRAM_SFH4656" V 4997 2782 50  0000 R CNN
 F 2 "" H 5050 2900 50  0000 C CNN
@@
 $EndComp
 $Comp
-L R R?
+L R R2
 U 1 1 59FDE229
 P 5050 2250
-F 0 "R?" H 5120 2296 50  0000 L CNN
+F 0 "R2" H 5120 2296 50  0000 L CNN
 F 1 "R" H 5120 2205 50  0000 L CNN
 F 2 "" V 4980 2250 50  0000 C CNN
@@
 $EndComp
 $Comp
-L R R?
+L R R4
 U 1 1 59FDE287
 P 5050 3300
-F 0 "R?" H 5120 3346 50  0000 L CNN
+F 0 "R4" H 5120 3346 50  0000 L CNN
 F 1 "R" H 5120 3255 50  0000 L CNN
 F 2 "" V 4980 3300 50  0000 C CNN
@@
 	5050 2000 5050 2100
 $Comp
-L CONN_01X02 P?
+L CONN_01X02 P1
 U 1 1 59FDE676
 P 4600 1850
-F 0 "P?" H 4519 1575 50  0000 C CNN
+F 0 "P1" H 4519 1575 50  0000 C CNN
 F 1 "CONN_01X02" H 4519 1666 50  0000 C CNN
 F 2 "" H 4600 1850 50  0000 C CNN
@@
 	4800 2050 5050 2050
 $Comp
-L CONN_01X02 P?
+L CONN_01X02 P2
 U 1 1 59FDE836
 P 4600 2900
-F 0 "P?" H 4519 2625 50  0000 C CNN
+F 0 "P2" H 4519 2625 50  0000 C CNN
 F 1 "CONN_01X02" H 4519 2716 50  0000 C CNN
 F 2 "" H 4600 2900 50  0000 C CNN
@@
 	5050 2500 5500 2500
 $Comp
-L GND #PWR?
+L GND #PWR3
 U 1 1 59FDEA04
 P 5500 2500
-F 0 "#PWR?" H 5500 2250 50  0001 C CNN
+F 0 "#PWR3" H 5500 2250 50  0001 C CNN
 F 1 "GND" V 5505 2372 50  0000 R CNN
 F 2 "" H 5500 2500 50  0000 C CNN
@@
 $EndComp
 $Comp
-L GND #PWR?
+L GND #PWR6
 U 1 1 59FDEA3E
 P 5500 3550
-F 0 "#PWR?" H 5500 3300 50  0001 C CNN
+F 0 "#PWR6" H 5500 3300 50  0001 C CNN
 F 1 "GND" V 5505 3422 50  0000 R CNN
 F 2 "" H 5500 3550 50  0000 C CNN
@@
 Text GLabel 5500 2650 2    60   Input ~ 0
 LB2_LED
+$Comp
+L C C1
+U 1 1 59FF4C3B
+P 2200 1900
+F 0 "C1" H 2315 1946 50  0000 L CNN
+F 1 "1u" H 2315 1855 50  0000 L CNN
+F 2 "" H 2238 1750 50  0000 C CNN
+F 3 "" H 2200 1900 50  0000 C CNN
+	1    2200 1900
+	1    0    0    -1
+$EndComp
+$Comp
+L R R1
+U 1 1 59FF4CB3
+P 2800 1750
+F 0 "R1" V 2593 1750 50  0000 C CNN
+F 1 "100E" V 2684 1750 50  0000 C CNN
+F 2 "" V 2730 1750 50  0000 C CNN
+F 3 "" H 2800 1750 50  0000 C CNN
+	1    2800 1750
+	0    1    1    0
+$EndComp
+Wire Wire Line
+	2100 1750 2650 1750
+Connection ~ 2200 1750
+Wire Wire Line
+	2950 1750 3200 1750
+Wire Wire Line
+	2100 2050 2500 2050
+Wire Wire Line
+	2500 2050 2500 1900
+Wire Wire Line
+	2500 1900 3200 1900
+Connection ~ 2200 2050
+$Comp
+L +3.3V #PWR4
+U 1 1 59FF4F0F
+P 2100 2750
+F 0 "#PWR4" H 2100 2600 50  0001 C CNN
+F 1 "+3.3V" V 2115 2878 50  0000 L CNN
+F 2 "" H 2100 2750 50  0000 C CNN
+F 3 "" H 2100 2750 50  0000 C CNN
+	1    2100 2750
+	0    -1   -1   0
+$EndComp
+$Comp
+L GND #PWR5
+U 1 1 59FF4F15
+P 2100 3050
+F 0 "#PWR5" H 2100 2800 50  0001 C CNN
+F 1 "GND" V 2105 2922 50  0000 R CNN
+F 2 "" H 2100 3050 50  0000 C CNN
+F 3 "" H 2100 3050 50  0000 C CNN
+	1    2100 3050
+	0    1    1    0
+$EndComp
+$Comp
+L C C2
+U 1 1 59FF4F1B
+P 2200 2900
+F 0 "C2" H 2315 2946 50  0000 L CNN
+F 1 "1u" H 2315 2855 50  0000 L CNN
+F 2 "" H 2238 2750 50  0000 C CNN
+F 3 "" H 2200 2900 50  0000 C CNN
+	1    2200 2900
+	1    0    0    -1
+$EndComp
+Wire Wire Line
+	2100 2750 2650 2750
+Connection ~ 2200 2750
+Wire Wire Line
+	2100 3050 2500 3050
+Wire Wire Line
+	2500 3050 2500 2900
+Wire Wire Line
+	2500 2900 3200 2900
+Connection ~ 2200 3050
+$Comp
+L R R3
+U 1 1 59FF4F3F
+P 2800 2750
+F 0 "R3" V 2593 2750 50  0000 C CNN
+F 1 "100E" V 2684 2750 50  0000 C CNN
+F 2 "" V 2730 2750 50  0000 C CNN
+F 3 "" H 2800 2750 50  0000 C CNN
+	1    2800 2750
+	0    1    1    0
+$EndComp
+Wire Wire Line
+	2950 2750 3200 2750
 $EndSCHEMATC

Commit message: Annotated entire schematic
Parts:
- renumbered C1 to C501, C2 to C502, D1 to D501, D2 to D502, P1 to P501, P2 to P502, R1 to R501, R2 to R502, R3 to R503, R4 to R504, U1 to U501, U2 to U502
Changed lines of the file:
@@
 $EndDescr
 $Comp
-L TSOP38 U1
+L TSOP38 U501
 U 1 1 59FCFE81
 P 3500 1600
-F 0 "U1" H 3677 1358 60  0000 L CNN
+F 0 "U501" H 3677 1358 60  0000 L CNN
 F 1 "TSOP38" H 3677 1252 60  0000 L CNN
 F 2 "" H 3500 1600 60  0001 C CNN
@@
 $EndComp
 $Comp
-L TSOP38 U2
+L TSOP38 U502
 U 1 1 59FCFEFD
 P 3500 2600
-F 0 "U2" H 3677 2358 60  0000 L CNN
+F 0 "U502" H 3677 2358 60  0000 L CNN
 F 1 "TSOP38" H 3677 2252 60  0000 L CNN
 F 2 "" H 3500 2600 60  0001 C CNN
@@
 $EndComp
 $Comp
-L +3.3V #PWR1
+L +3.3V #PWR0501
 U 1 1 59FD02D9
 P 2100 1750
-F 0 "#PWR1" H 2100 1600 50  0001 C CNN
+F 0 "#PWR0501" H 2100 1600 50  0001 C CNN
 F 1 "+3.3V" V 2115 1878 50  0000 L CNN
 F 2 "" H 2100 1750 50  0000 C CNN
@@
 $EndComp
 $Comp
-L GND #PWR2
+L GND #PWR0502
 U 1 1 59FD0355
 P 2100 2050
-F 0 "#PWR2" H 2100 1800 50  0001 C CNN
+F 0 "#PWR0502" H 2100 1800 50  0001 C CNN
 F 1 "GND" V 2105 1922 50  0000 R CNN
 F 2 "" H 2100 2050 50  0000 C CNN
@@
 LB2_DETECT
 $Comp
-L OSRAM_SFH4656 D1
+L OSRAM_SFH4656 D501
 U 1 1 59FDE056
 P 5050 1850
-F 0 "D1" V 5088 1732 50  0000 R CNN
+F 0 "D501" V 5088 1732 50  0000 R CNN
 F 1 "OSRAM_SFH4656" V 4997 1732 50  0000 R CNN
 F 2 "" H 5050 1850 50  0000 C CNN
@@
 $EndComp
 $Comp
-L OSRAM_SFH4656 D2
+L OSRAM_SFH4656 D502
 U 1 1 59FDE0CE
 P 5050 2900
-F 0 "D2" V 5088 2782 50  0000 R CNN
+F 0 "D502" V 5088 2782 50  0000 R CNN
 F 1 "OSRAM_SFH4656" V 4997 2782 50  0000 R CNN
 F 2 "" H 5050 2900 50  0000 C CNN
@@
 $EndComp
 $Comp
-L R R2
+L R R502
 U 1 1 59FDE229
 P 5050 2250
-F 0 "R2" H 5120 2296 50  0000 L CNN
+F 0 "R502" H 5120 2296 50  0000 L CNN
 F 1 "R" H 5120 2205 50  0000 L CNN
 F 2 "" V 4980 2250 50  0000 C CNN
@@
 $EndComp
 $Comp
-L R R4
+L R R504
 U 1 1 59FDE287
 P 5050 3300
-F 0 "R4" H 5120 3346 50  0000 L CNN
+F 0 "R504" H 5120 3346 50  0000 L CNN
 F 1 "R" H 5120 3255 50  0000 L CNN
 F 2 "" V 4980 3300 50  0000 C CNN
@@
 	5050 2000 5050 2100
 $Comp
-L CONN_01X02 P1
+L CONN_01X02 P501
 U 1 1 59FDE676
 P 4600 1850
-F 0 "P1" H 4519 1575 50  0000 C CNN
+F 0 "P501" H 4519 1575 50  0000 C CNN
 F 1 "CONN_01X02" H 4519 1666 50  0000 C CNN
 F 2 "" H 4600 1850 50  0000 C CNN
@@
 	4800 2050 5050 2050
 $Comp
-L CONN_01X02 P2
+L CONN_01X02 P502
 U 1 1 59FDE836
 P 4600 2900
-F 0 "P2" H 4519 2625 50  0000 C CNN
+F 0 "P502" H 4519 2625 50  0000 C CNN
 F 1 "CONN_01X02" H 4519 2716 50  0000 C CNN
 F 2 "" H 4600 2900 50  0000 C CNN
@@
 	5050 2500 5500 2500
 $Comp
-L GND #PWR3
+L GND #PWR0503
 U 1 1 59FDEA04
 P 5500 2500
-F 0 "#PWR3" H 5500 2250 50  0001 C CNN
+F 0 "#PWR0503" H 5500 2250 50  0001 C CNN
 F 1 "GND" V 5505 2372 50  0000 R CNN
 F 2 "" H 5500 2500 50  0000 C CNN
@@
 $EndComp
 $Comp
-L GND #PWR6
+L GND #PWR0506
 U 1 1 59FDEA3E
 P 5500 3550
-F 0 "#PWR6" H 5500 3300 50  0001 C CNN
+F 0 "#PWR0506" H 5500 3300 50  0001 C CNN
 F 1 "GND" V 5505 3422 50  0000 R CNN
 F 2 "" H 5500 3550 50  0000 C CNN
@@
 LB2_LED
 $Comp
-L C C1
+L C C501
 U 1 1 59FF4C3B
 P 2200 1900
-F 0 "C1" H 2315 1946 50  0000 L CNN
+F 0 "C501" H 2315 1946 50  0000 L CNN
 F 1 "1u" H 2315 1855 50  0000 L CNN
 F 2 "" H 2238 1750 50  0000 C CNN
@@
 $EndComp
 $Comp
-L R R1
+L R R501
 U 1 1 59FF4CB3
 P 2800 1750
-F 0 "R1" V 2593 1750 50  0000 C CNN
+F 0 "R501" V 2593 1750 50  0000 C CNN
 F 1 "100E" V 2684 1750 50  0000 C CNN
 F 2 "" V 2730 1750 50  0000 C CNN
@@
 Connection ~ 2200 2050
 $Comp
-L +3.3V #PWR4
+L +3.3V #PWR0504
 U 1 1 59FF4F0F
 P 2100 2750
-F 0 "#PWR4" H 2100 2600 50  0001 C CNN
+F 0 "#PWR0504" H 2100 2600 50  0001 C CNN
 F 1 "+3.3V" V 2115 2878 50  0000 L CNN
 F 2 "" H 2100 2750 50  0000 C CNN
@@
 $EndComp
 $Comp
-L GND #PWR5
+L GND #PWR0505
 U 1 1 59FF4F15
 P 2100 3050
-F 0 "#PWR5" H 2100 2800 50  0001 C CNN
+F 0 "#PWR0505" H 2100 2800 50  0001 C CNN
 F 1 "GND" V 2105 2922 50  0000 R CNN
 F 2 "" H 2100 3050 50  0000 C CNN
@@
 $EndComp
 $Comp
-L C C2
+L C C502
 U 1 1 59FF4F1B
 P 2200 2900
-F 0 "C2" H 2315 2946 50  0000 L CNN
+F 0 "C502" H 2315 2946 50  0000 L CNN
 F 1 "1u" H 2315 2855 50  0000 L CNN
 F 2 "" H 2238 2750 50  0000 C CNN
@@
 Connection ~ 2200 3050
 $Comp
-L R R3
+L R R503
 U 1 1 59FF4F3F
 P 2800 2750
-F 0 "R3" V 2593 2750 50  0000 C CNN
+F 0 "R503" V 2593 2750 50  0000 C CNN
 F 1 "100E" V 2684 2750 50  0000 C CNN
 F 2 "" V 2730 2750 50  0000 C CNN
