File: Nestbox_v2/_saved_Nestbox_v2_control.sch (KiCad schematic (older format))
At the start: 25 parts, among them CON301 Micro_SD_Card, P301 TST/RST, P302 RX/TX, SW301 SMD-BUTTON_2P-3.0X2.5X1.2+0.4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, U301 MSP430FR5969, Y301 Crystal

Commit message: inserted some comments
Parts:
- added R? (x2): 0R, SeeedOPL-Resistor-2016:R0603, symbol DIP-RES-47K-5%-1_4W_PR-D2.3XL6.5MM_
- added R? (x2): DNP, SeeedOPL-Resistor-2016:R0603, symbol DIP-RES-47K-5%-1_4W_PR-D2.3XL6.5MM_
Connections:
- net LB1_LED: now also R?.1, R?.2; no longer U301.2 (P1.1/TA0.2/TA1CLK/COUT/A1/C1/VREF+/VeREF+)
- net LB2_LED: now also R?.1, R?.2; no longer JP?.2, U301.1 (P1.0/TA0.1/DMAE0/RTCCLK/A0/C0/VREF-/VeREF-_)
- net at U301.29 (P3.6/TB0.5): now also R?.1
- net at U301.30 (P3.7/TB0.6): now also R?.1
- new net: JP?.2, R?.2, U301.1 (P1.0/TA0.1/DMAE0/RTCCLK/A0/C0/VREF-/VeREF-_)
- new net: R?.2, U301.2 (P1.1/TA0.2/TA1CLK/COUT/A1/C1/VREF+/VeREF+)
Other:
- note added: "Alternative LED driver, in case the PWM \ndisturbes the analog inputs too much.\n"
Changed lines of the file:
@@
 Text GLabel 1300 4550 0    60   Input ~ 0
 LB2_DETECT
-Text GLabel 1150 3850 0    60   Input ~ 0
+Text GLabel 950  3850 0    60   Input ~ 0
 LB1_LED
 Text GLabel 1300 4450 0    60   Input ~ 0
 LB1_DETECT
 Wire Wire Line
-	1150 3850 1550 3850
-Wire Wire Line
 	1300 3950 1550 3950
-Text GLabel 1150 3750 0    60   Input ~ 0
+Text GLabel 950  3750 0    60   Input ~ 0
 LB2_LED
 Text GLabel 6700 4650 2    60   Input ~ 0
@@
 	8900 1850 8350 1850
 Wire Wire Line
-	8350 1900 8350 1850
-Wire Wire Line
-	7600 1900 8350 1900
+	8350 1850 8350 1900
+Wire Wire Line
+	8350 1900 7600 1900
 Connection ~ 8100 1900
 Connection ~ 7700 1900
@@
 RFID_FREQ_SEL
 Wire Wire Line
-	1150 3750 1550 3750
+	1250 3750 1550 3750
 Text Label 1350 2950 1    60   ~ 0
 RTC_CAL
@@
 Text GLabel 1300 4750 0    60   Input ~ 0
 LOAD_CELL_IN-
+$Comp
+L DIP-RES-47K-5%-1_4W_PR-D2.3XL6.5MM_ R?
+U 1 1 5A772C1E
+P 1100 3750
+F 0 "R?" H 950 3800 45  0000 L BNN
+F 1 "0R" H 1100 3800 45  0000 L BNN
+F 2 "SeeedOPL-Resistor-2016:R0603" H 1100 3750 40  0001 C CNN
+F 3 "" H 1100 3750 40  0001 C CNN
+F 4 "FHCFR-1_4W-473J" H 1130 3900 20  0001 C CNN "MPN"
+	1    1100 3750
+	1    0    0    -1
+$EndComp
+$Comp
+L DIP-RES-47K-5%-1_4W_PR-D2.3XL6.5MM_ R?
+U 1 1 5A773434
+P 1100 3850
+F 0 "R?" H 950 3900 45  0000 L BNN
+F 1 "0R" H 1100 3900 45  0000 L BNN
+F 2 "SeeedOPL-Resistor-2016:R0603" H 1100 3850 40  0001 C CNN
+F 3 "" H 1100 3850 40  0001 C CNN
+F 4 "FHCFR-1_4W-473J" H 1130 4000 20  0001 C CNN "MPN"
+	1    1100 3850
+	1    0    0    -1
+$EndComp
+Wire Wire Line
+	1550 3850 1250 3850
+$Comp
+L DIP-RES-47K-5%-1_4W_PR-D2.3XL6.5MM_ R?
+U 1 1 5A773875
+P 6550 4350
+F 0 "R?" H 6400 4400 45  0000 L BNN
+F 1 "DNP" H 6550 4400 45  0000 L BNN
+F 2 "SeeedOPL-Resistor-2016:R0603" H 6550 4350 40  0001 C CNN
+F 3 "" H 6550 4350 40  0001 C CNN
+F 4 "FHCFR-1_4W-473J" H 6580 4500 20  0001 C CNN "MPN"
+	1    6550 4350
+	1    0    0    -1
+$EndComp
+$Comp
+L DIP-RES-47K-5%-1_4W_PR-D2.3XL6.5MM_ R?
+U 1 1 5A773D27
+P 6550 4450
+F 0 "R?" H 6400 4500 45  0000 L BNN
+F 1 "DNP" H 6550 4500 45  0000 L BNN
+F 2 "SeeedOPL-Resistor-2016:R0603" H 6550 4450 40  0001 C CNN
+F 3 "" H 6550 4450 40  0001 C CNN
+F 4 "FHCFR-1_4W-473J" H 6580 4600 20  0001 C CNN "MPN"
+	1    6550 4450
+	1    0    0    -1
+$EndComp
+Wire Wire Line
+	6400 4350 6150 4350
+Wire Wire Line
+	6150 4450 6400 4450
+Text GLabel 6850 4350 2    60   Input ~ 0
+LB2_LED
+Wire Wire Line
+	6850 4350 6700 4350
+Text GLabel 6850 4450 2    60   Input ~ 0
+LB1_LED
+Wire Wire Line
+	6850 4450 6700 4450
+Text Notes 7300 4450 0    60   ~ 0
+Alternative LED driver, in case the PWM \ndisturbes the analog inputs too much.\n
 $EndSCHEMATC
