File: Nestbox_v2/_saved_Nestbox_v2_control.sch (KiCad schematic (older format))
At the start: 24 parts, among them CON301 Micro_SD_Card, P301 TST/RST, P302 RX/TX, SW301 SMD-BUTTON_2P-3.0X2.5X1.2+0.4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, U301 MSP430FR5969, Y301 Crystal

Commit message: various changes
Connections:
- net LOADCELL_DATA_READY: now reaches U301.27 (P3.4/TB0.3/SMCLK)
Changed lines of the file:
@@
 	8900 1850 8350 1850
 Wire Wire Line
-	8350 1900 8350 1850
+	8350 1850 8350 1900
 Wire Wire Line
-	7600 1900 8350 1900
+	8350 1900 7600 1900
 Connection ~ 8100 1900
 Connection ~ 7700 1900
@@
 Text GLabel 6700 4050 2    60   Input ~ 0
 LORA_RST_N
+Wire Wire Line
+	6150 4650 6700 4650
+Text Label 6300 4650 0    60   ~ 0
+LOADCELL_DATA_READY
 $EndSCHEMATC
