File: Nestbox_v2/Nestbox_v2_control.sch (KiCad schematic (older format))
At the start: 25 parts, among them CON301 Micro_SD_Card, P301 TST/RST, P302 RX/TX, SW301 SMD-BUTTON_2P-3.0X2.5X1.2+0.4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, U301 MSP430FR5969, Y301 Crystal

Commit message: design comments
Parts:
- removed JP?: Jumper, symbol Jumper
Connections:
- net labels added: LOADCELL_SPI_CS_N, SPI_CLK, SPI_MISO, SPI_MOSI
- net labels removed: LOAD_CELL_IN+, LOAD_CELL_IN-, RFID_FREQ_SEL, RTC_CAL
- wire segments 90 -> 86
Other:
- note removed: "ADC12INCHx = 00101b \nIf ADC12DIF = 1: Ain+ = A4, Ain- = A5 \n"
Changed lines of the file:
@@
 $Descr A4 11693 8268
 encoding utf-8
-Sheet 3 7
+Sheet 3 6
 Title "Octanis 3 Nestbox"
 Date ""
@@
 $EndComp
 $Comp
-L GND #PWR030
+L GND #PWR0312
 U 1 1 586416A7
 P 6150 3750
-F 0 "#PWR030" H 6150 3500 50  0001 C CNN
+F 0 "#PWR0312" H 6150 3500 50  0001 C CNN
 F 1 "GND" H 6150 3600 50  0000 C CNN
 F 2 "" H 6150 3750 50  0000 C CNN
@@
 $EndComp
 $Comp
-L +3.3V #PWR031
+L +3.3V #PWR0304
 U 1 1 586418DC
 P 4300 1900
-F 0 "#PWR031" H 4300 1750 50  0001 C CNN
+F 0 "#PWR0304" H 4300 1750 50  0001 C CNN
 F 1 "+3.3V" H 4300 2040 50  0000 C CNN
 F 2 "" H 4300 1900 50  0000 C CNN
@@
 $EndComp
 $Comp
-L GND #PWR032
+L GND #PWR0306
 U 1 1 58641ADD
 P 2500 2250
-F 0 "#PWR032" H 2500 2000 50  0001 C CNN
+F 0 "#PWR0306" H 2500 2000 50  0001 C CNN
 F 1 "GND" H 2500 2100 50  0000 C CNN
 F 2 "" H 2500 2250 50  0000 C CNN
@@
 $EndComp
 $Comp
-L +3.3V #PWR033
+L +3.3V #PWR0303
 U 1 1 58641B00
 P 2850 1700
-F 0 "#PWR033" H 2850 1550 50  0001 C CNN
+F 0 "#PWR0303" H 2850 1550 50  0001 C CNN
 F 1 "+3.3V" H 2850 1840 50  0000 C CNN
 F 2 "" H 2850 1700 50  0000 C CNN
@@
 $EndComp
 $Comp
-L GND #PWR034
+L GND #PWR0311
 U 1 1 58652F3A
 P 4700 2450
-F 0 "#PWR034" H 4700 2200 50  0001 C CNN
+F 0 "#PWR0311" H 4700 2200 50  0001 C CNN
 F 1 "GND" H 4700 2300 50  0000 C CNN
 F 2 "" H 4700 2450 50  0000 C CNN
@@
 $EndComp
 $Comp
-L GND #PWR035
+L GND #PWR0301
 U 1 1 5865358A
 P 3400 1600
-F 0 "#PWR035" H 3400 1350 50  0001 C CNN
+F 0 "#PWR0301" H 3400 1350 50  0001 C CNN
 F 1 "GND" H 3400 1450 50  0000 C CNN
 F 2 "" H 3400 1600 50  0000 C CNN
@@
 $EndComp
 $Comp
-L GNDA #PWR036
+L GNDA #PWR0307
 U 1 1 587B6902
 P 3300 2400
-F 0 "#PWR036" H 3300 2150 50  0001 C CNN
+F 0 "#PWR0307" H 3300 2150 50  0001 C CNN
 F 1 "GNDA" H 3300 2250 50  0000 C CNN
 F 2 "" H 3300 2400 50  0000 C CNN
@@
 $EndComp
 $Comp
-L GNDA #PWR037
+L GNDA #PWR0308
 U 1 1 587B69F1
 P 3600 2400
-F 0 "#PWR037" H 3600 2150 50  0001 C CNN
+F 0 "#PWR0308" H 3600 2150 50  0001 C CNN
 F 1 "GNDA" H 3600 2250 50  0000 C CNN
 F 2 "" H 3600 2400 50  0000 C CNN
@@
 $EndComp
 $Comp
-L GNDA #PWR038
+L GNDA #PWR0309
 U 1 1 587B6A2F
 P 3900 2400
-F 0 "#PWR038" H 3900 2150 50  0001 C CNN
+F 0 "#PWR0309" H 3900 2150 50  0001 C CNN
 F 1 "GNDA" H 3900 2250 50  0000 C CNN
 F 2 "" H 3900 2400 50  0000 C CNN
@@
 $EndComp
 $Comp
-L GND #PWR039
+L GND #PWR0314
 U 1 1 587B96DD
 P 10000 5300
-F 0 "#PWR039" H 10000 5050 50  0001 C CNN
+F 0 "#PWR0314" H 10000 5050 50  0001 C CNN
 F 1 "GND" H 10000 5150 50  0000 C CNN
 F 2 "" H 10000 5300 50  0000 C CNN
@@
 $EndComp
 $Comp
-L +3.3V #PWR040
+L +3.3V #PWR0313
 U 1 1 587B9736
 P 10000 4100
-F 0 "#PWR040" H 10000 3950 50  0001 C CNN
+F 0 "#PWR0313" H 10000 3950 50  0001 C CNN
 F 1 "+3.3V" H 10000 4240 50  0000 C CNN
 F 2 "" H 10000 4100 50  0000 C CNN
@@
 $EndComp
 $Comp
-L GND #PWR041
+L GND #PWR0317
 U 1 1 587B97E4
 P 9600 5400
-F 0 "#PWR041" H 9600 5150 50  0001 C CNN
+F 0 "#PWR0317" H 9600 5150 50  0001 C CNN
 F 1 "GND" H 9600 5250 50  0000 C CNN
 F 2 "" H 9600 5400 50  0000 C CNN
@@
 $EndComp
 $Comp
-L GND #PWR042
+L GND #PWR0316
 U 1 1 587B9834
 P 9300 5400
-F 0 "#PWR042" H 9300 5150 50  0001 C CNN
+F 0 "#PWR0316" H 9300 5150 50  0001 C CNN
 F 1 "GND" H 9300 5250 50  0000 C CNN
 F 2 "" H 9300 5400 50  0000 C CNN
@@
 Wire Wire Line
 	10000 4500 10000 4600
+Wire Wire Line
+	3700 6450 3700 7000
 Wire Wire Line
 	10000 5200 10000 5300
@@
 	9300 4950 9300 5050
 $Comp
-L GND #PWR043
+L GND #PWR0310
 U 1 1 587D2523
 P 2450 2450
-F 0 "#PWR043" H 2450 2200 50  0001 C CNN
+F 0 "#PWR0310" H 2450 2200 50  0001 C CNN
 F 1 "GND" H 2450 2300 50  0000 C CNN
 F 2 "" H 2450 2450 50  0000 C CNN
@@
 	4350 6650 4350 6700
 $Comp
-L +3.3V #PWR044
+L +3.3V #PWR0318
 U 1 1 58BC4BB7
 P 4850 6600
-F 0 "#PWR044" H 4850 6450 50  0001 C CNN
+F 0 "#PWR0318" H 4850 6450 50  0001 C CNN
 F 1 "+3.3V" H 4850 6740 50  0000 C CNN
 F 2 "" H 4850 6600 50  0000 C CNN
@@
 	10200 4850 10200 4900
 $Comp
-L GND #PWR045
+L GND #PWR0315
 U 1 1 58BF19D6
 P 10200 5300
-F 0 "#PWR045" H 10200 5050 50  0001 C CNN
+F 0 "#PWR0315" H 10200 5050 50  0001 C CNN
 F 1 "GND" H 10200 5150 50  0000 C CNN
 F 2 "" H 10200 5300 50  0000 C CNN
@@
 	6150 4250 6700 4250
 Text Label 6700 4150 2    60   ~ 0
-SD_MISO
+SPI_MISO
 Text Label 6700 4250 2    60   ~ 0
-SD_MOSI
+SPI_MOSI
 Wire Wire Line
 	6150 4750 6700 4750
-Text Label 6700 4750 2    60   ~ 0
-SD_CLK
-Text GLabel 1300 3950 0    60   Input ~ 0
+Text Label 6700 4750 0    60   ~ 0
+SPI_CLK
+Text GLabel 1300 4550 0    60   Input ~ 0
 RFID_MODU_N
-Text GLabel 3800 6450 3    60   Input ~ 0
+Text GLabel 1300 4750 0    60   Input ~ 0
 RFID_DATA
-Text GLabel 4000 2150 1    60   Input ~ 0
+Text GLabel 1300 4650 0    60   Input ~ 0
 RFID_CLOCK
 Wire Wire Line
-	1300 4450 1550 4450
-Wire Wire Line
-	1550 4550 1300 4550
+	1300 4550 1550 4550
+Wire Wire Line
+	1550 4650 1300 4650
 Wire Wire Line
 	1300 4750 1550 4750
@@
 Wire Wire Line
 	6150 4050 6700 4050
-Text Label 6300 4050 0    60   ~ 0
-SD_CS_B
-Text GLabel 1300 4550 0    60   Input ~ 0
+Text Label 6300 4550 0    60   ~ 0
+LOADCELL_SPI_CS_N
+Text GLabel 1300 3750 0    60   Input ~ 0
 LB2_DETECT
-Text GLabel 1150 3850 0    60   Input ~ 0
+Text GLabel 1300 3850 0    60   Input ~ 0
 LB1_LED
-Text GLabel 1300 4450 0    60   Input ~ 0
+Text GLabel 1300 3950 0    60   Input ~ 0
 LB1_DETECT
 Wire Wire Line
-	1150 3850 1550 3850
+	1300 3750 1550 3750
+Wire Wire Line
+	1550 3850 1300 3850
 Wire Wire Line
 	1300 3950 1550 3950
-Text GLabel 1150 3750 0    60   Input ~ 0
+Text GLabel 4100 2200 1    60   Input ~ 0
 LB2_LED
-Text GLabel 6700 4650 2    60   Input ~ 0
-LORA_RST_N
-Wire Wire Line
-	6150 4550 6500 4550
+Wire Wire Line
+	4100 2200 4100 2450
+Wire Wire Line
+	6150 4550 6700 4550
 $Comp
 L Micro_SD_Card CON301
@@
 SD_MOSI
 $Comp
-L +3.3V #PWR046
+L +3.3V #PWR0302
 U 1 1 59FCECA7
 P 7100 1600
-F 0 "#PWR046" H 7100 1450 50  0001 C CNN
+F 0 "#PWR0302" H 7100 1450 50  0001 C CNN
 F 1 "+3.3V" H 7100 1740 50  0000 C CNN
 F 2 "" H 7100 1600 50  0000 C CNN
@@
 $EndComp
 $Comp
-L GND #PWR047
+L GND #PWR0305
 U 1 1 59FCED84
 P 7600 1900
-F 0 "#PWR047" H 7600 1650 50  0001 C CNN
+F 0 "#PWR0305" H 7600 1650 50  0001 C CNN
 F 1 "GND" H 7600 1750 50  0000 C CNN
 F 2 "" H 7600 1900 50  0000 C CNN
@@
 SD_MISO
 Wire Wire Line
-	6150 3850 6750 3850
+	3600 6450 3600 7000
 Text Label 3500 7000 1    60   ~ 0
 DBG_LED1
-Text Label 6750 3850 2    60   ~ 0
+Text Label 3600 7000 1    60   ~ 0
 DBG_LED2
 Text Label 9300 4100 3    60   ~ 0
@@
 Text Label 9600 4100 3    60   ~ 0
 DBG_LED2
-Text Label 6300 3950 0    60   ~ 0
+Text Label 3700 7000 1    60   ~ 0
 DBG_Switch
 Wire Wire Line
@@
 Text Label 10850 4550 2    60   ~ 0
 DBG_Switch
-Text GLabel 3700 6450 3    60   Input ~ 0
+Text GLabel 3800 6450 3    60   Input ~ 0
 DATA_Enable_N
 $Comp
@@
 	8900 1850 8350 1850
 Wire Wire Line
-	8350 1850 8350 1900
-Wire Wire Line
-	8350 1900 7600 1900
+	8350 1900 8350 1850
+Wire Wire Line
+	7600 1900 8350 1900
 Connection ~ 8100 1900
 Connection ~ 7700 1900
@@
 Wire Wire Line
 	3900 6450 3900 7400
-Wire Wire Line
-	6150 3950 6700 3950
-Wire Wire Line
-	4000 2450 4000 2150
-Text GLabel 6500 4550 2    60   Input ~ 0
-RFID_FREQ_SEL
-Wire Wire Line
-	1150 3750 1550 3750
-Text Label 1350 2950 1    60   ~ 0
-RTC_CAL
-$Comp
-L Jumper JP?
-U 1 1 5A75C27E
-P 1350 3350
-F 0 "JP?" V 1304 3477 50  0000 L CNN
-F 1 "Jumper" V 1395 3477 50  0000 L CNN
-F 2 "" H 1350 3350 50  0001 C CNN
-F 3 "" H 1350 3350 50  0001 C CNN
-	1    1350 3350
-	0    1    1    0
-$EndComp
-Wire Wire Line
-	1350 2950 1350 3050
-Wire Wire Line
-	1350 3650 1350 3750
-Connection ~ 1350 3750
-Wire Wire Line
-	6700 4650 6150 4650
-Text Notes 600  5150 0    60   ~ 0
-ADC12INCHx = 00101b \nIf ADC12DIF = 1: Ain+ = A4, Ain- = A5 \n
-Wire Wire Line
-	1550 4650 1300 4650
-Text GLabel 1300 4650 0    60   Input ~ 0
-LOAD_CELL_IN+
-Text GLabel 1300 4750 0    60   Input ~ 0
-LOAD_CELL_IN-
+Text GLabel 6700 4050 2    60   Input ~ 0
+LORA_RST_N
 $EndSCHEMATC

Commit message: more comments on ADC
Changed lines of the file:
@@
 $Descr A4 11693 8268
 encoding utf-8
-Sheet 3 6
+Sheet 3 7
 Title "Octanis 3 Nestbox"
 Date ""
@@
 	8900 1850 8350 1850
 Wire Wire Line
-	8350 1900 8350 1850
-Wire Wire Line
-	7600 1900 8350 1900
+	8350 1850 8350 1900
+Wire Wire Line
+	8350 1900 7600 1900
 Connection ~ 8100 1900
 Connection ~ 7700 1900

Commit message: load cell AC excitation
Parts:
- added R? (x3): 47R, symbol R
- P301, P302: symbol Conn_01x02 -> CONN_01X02
Connections:
- net labels added: SPI_SCK, SPI_SD_CS_N
- net labels removed: SD_CLK, SD_CS_B, SD_MISO, SD_MOSI
- wire segments 86 -> 89
Other:
- moved on the sheet: C301, C302, R301
Changed lines of the file:
@@
 $EndComp
 $Comp
-L Conn_01x02 P301
+L CONN_01X02 P301
 U 1 1 58653CFC
 P 4450 6900
+AR Path="/58653CFC" Ref="P301"  Part="1"
+AR Path="/59EF7F04/58653CFC" Ref="P301"  Part="1"
 F 0 "P301" H 4450 7050 50  0000 C CNN
 F 1 "TST/RST" V 4550 6900 50  0000 C CNN
@@
 Debugging interface
 $Comp
-L Conn_01x02 P302
+L CONN_01X02 P302
 U 1 1 587BB574
 P 4000 7600
+AR Path="/587BB574" Ref="P302"  Part="1"
+AR Path="/59EF7F04/587BB574" Ref="P302"  Part="1"
 F 0 "P302" H 4000 7750 50  0000 C CNN
 F 1 "RX/TX" V 4100 7600 50  0000 C CNN
@@
 NoConn ~ 8900 2050
 Wire Wire Line
-	8900 1450 8400 1450
-Text Label 8400 1450 0    60   ~ 0
-SD_CS_B
-Wire Wire Line
-	8900 1550 8400 1550
-Wire Wire Line
-	8900 1750 8400 1750
-Wire Wire Line
-	8900 1950 8400 1950
-Text Label 8400 1550 0    60   ~ 0
-SD_MOSI
+	7800 1450 8900 1450
+Text Label 7800 1450 0    60   ~ 0
+SPI_SD_CS_N
+Wire Wire Line
+	7800 1550 8450 1550
+Wire Wire Line
+	7800 1950 8450 1950
+Text Label 7800 1550 0    60   ~ 0
+SPI_MOSI
 $Comp
 L +3.3V #PWR0302
 U 1 1 59FCECA7
-P 7100 1600
-F 0 "#PWR0302" H 7100 1450 50  0001 C CNN
-F 1 "+3.3V" H 7100 1740 50  0000 C CNN
-F 2 "" H 7100 1600 50  0000 C CNN
-F 3 "" H 7100 1600 50  0000 C CNN
-	1    7100 1600
+P 6500 1600
+F 0 "#PWR0302" H 6500 1450 50  0001 C CNN
+F 1 "+3.3V" H 6500 1740 50  0000 C CNN
+F 2 "" H 6500 1600 50  0000 C CNN
+F 3 "" H 6500 1600 50  0000 C CNN
+	1    6500 1600
 	0    -1   -1   0
 $EndComp
@@
 L GND #PWR0305
 U 1 1 59FCED84
-P 7600 1900
-F 0 "#PWR0305" H 7600 1650 50  0001 C CNN
-F 1 "GND" H 7600 1750 50  0000 C CNN
-F 2 "" H 7600 1900 50  0000 C CNN
-F 3 "" H 7600 1900 50  0000 C CNN
-	1    7600 1900
-	0    1    1    0
-$EndComp
-Text Label 8400 1750 0    60   ~ 0
-SD_CLK
-Text Label 8400 1950 0    60   ~ 0
-SD_MISO
+P 7000 1900
+F 0 "#PWR0305" H 7000 1650 50  0001 C CNN
+F 1 "GND" H 7000 1750 50  0000 C CNN
+F 2 "" H 7000 1900 50  0000 C CNN
+F 3 "" H 7000 1900 50  0000 C CNN
+	1    7000 1900
+	0    1    1    0
+$EndComp
+Text Label 7800 1750 0    60   ~ 0
+SPI_SCK
+Text Label 7800 1950 0    60   ~ 0
+SPI_MISO
 Wire Wire Line
 	3600 6450 3600 7000
@@
 L CP C301
 U 1 1 59FF0B56
-P 7700 1750
-F 0 "C301" H 7818 1796 50  0000 L CNN
-F 1 "100u" H 7818 1705 50  0000 L CNN
-F 2 "" H 7738 1600 50  0000 C CNN
-F 3 "" H 7700 1750 50  0000 C CNN
-F 4 "667-ECE-A0JKA101" H 7700 1750 60  0001 C CNN "Mouser-Part"
-	1    7700 1750
+P 7100 1750
+F 0 "C301" H 7218 1796 50  0000 L CNN
+F 1 "100u" H 7218 1705 50  0000 L CNN
+F 2 "" H 7138 1600 50  0000 C CNN
+F 3 "" H 7100 1750 50  0000 C CNN
+F 4 "667-ECE-A0JKA101" H 7100 1750 60  0001 C CNN "Mouser-Part"
+	1    7100 1750
 	1    0    0    -1
 $EndComp
@@
 L C C302
 U 1 1 59FF0C21
-P 8100 1750
-F 0 "C302" H 8215 1796 50  0000 L CNN
-F 1 "0.1u" H 8215 1705 50  0000 L CNN
-F 2 "" H 8138 1600 50  0000 C CNN
-F 3 "" H 8100 1750 50  0000 C CNN
-	1    8100 1750
-	1    0    0    -1
-$EndComp
-Wire Wire Line
-	7500 1600 8350 1600
-Connection ~ 7700 1600
-Wire Wire Line
-	8350 1600 8350 1650
-Wire Wire Line
-	8350 1650 8900 1650
-Connection ~ 8100 1600
-Wire Wire Line
-	8900 1850 8350 1850
-Wire Wire Line
-	8350 1850 8350 1900
-Wire Wire Line
-	8350 1900 7600 1900
-Connection ~ 8100 1900
-Connection ~ 7700 1900
+P 7500 1750
+F 0 "C302" H 7615 1796 50  0000 L CNN
+F 1 "0.1u" H 7615 1705 50  0000 L CNN
+F 2 "" H 7538 1600 50  0000 C CNN
+F 3 "" H 7500 1750 50  0000 C CNN
+	1    7500 1750
+	1    0    0    -1
+$EndComp
+Wire Wire Line
+	6900 1600 7750 1600
+Connection ~ 7100 1600
+Wire Wire Line
+	7750 1600 7750 1650
+Wire Wire Line
+	7750 1650 8900 1650
+Connection ~ 7500 1600
+Wire Wire Line
+	7750 1850 8900 1850
+Wire Wire Line
+	7750 1850 7750 1900
+Wire Wire Line
+	7750 1900 7000 1900
+Connection ~ 7500 1900
+Connection ~ 7100 1900
 $Comp
 L R R301
 U 1 1 59FF21A2
-P 7350 1600
-F 0 "R301" V 7143 1600 50  0000 C CNN
-F 1 "0E" V 7234 1600 50  0000 C CNN
-F 2 "" V 7280 1600 50  0000 C CNN
-F 3 "" H 7350 1600 50  0000 C CNN
-	1    7350 1600
-	0    1    1    0
-$EndComp
-Wire Wire Line
-	7100 1600 7200 1600
+P 6750 1600
+F 0 "R301" V 6543 1600 50  0000 C CNN
+F 1 "0E" V 6634 1600 50  0000 C CNN
+F 2 "" V 6680 1600 50  0000 C CNN
+F 3 "" H 6750 1600 50  0000 C CNN
+	1    6750 1600
+	0    1    1    0
+$EndComp
+Wire Wire Line
+	6500 1600 6600 1600
 $Comp
 L R R304
@@
 Text GLabel 6700 4050 2    60   Input ~ 0
 LORA_RST_N
+$Comp
+L R R?
+U 1 1 5AF9C4CE
+P 8600 1550
+F 0 "R?" V 8550 1750 50  0000 C CNN
+F 1 "47R" V 8600 1550 50  0000 C CNN
+F 2 "" V 8530 1550 50  0000 C CNN
+F 3 "" H 8600 1550 50  0000 C CNN
+	1    8600 1550
+	0    1    1    0
+$EndComp
+Wire Wire Line
+	8750 1550 8900 1550
+$Comp
+L R R?
+U 1 1 5AF9CD2C
+P 8600 1750
+F 0 "R?" V 8550 1950 50  0000 C CNN
+F 1 "47R" V 8600 1750 50  0000 C CNN
+F 2 "" V 8530 1750 50  0000 C CNN
+F 3 "" H 8600 1750 50  0000 C CNN
+	1    8600 1750
+	0    1    1    0
+$EndComp
+Wire Wire Line
+	8750 1750 8900 1750
+Wire Wire Line
+	8450 1750 7800 1750
+$Comp
+L R R?
+U 1 1 5AF9D016
+P 8600 1950
+F 0 "R?" V 8550 2150 50  0000 C CNN
+F 1 "47R" V 8600 1950 50  0000 C CNN
+F 2 "" V 8530 1950 50  0000 C CNN
+F 3 "" H 8600 1950 50  0000 C CNN
+	1    8600 1950
+	0    1    1    0
+$EndComp
+Wire Wire Line
+	8750 1950 8900 1950
 $EndSCHEMATC

Commit message: restructured top level sheet with hierarchical labels, assigned most GPIOs
Connections:
- net labels added: 5V_ENABLE, HK_5V_V, LDO_ENABLE, LOADCELL_DRDY, LOADCELL_SPI_CS, LORA_RESET_N, LORA_UART_RX, LORA_UART_TX, RFID_CLK, RFID_MODU, WIFI_EN, WIFI_UART_RX, WIFI_UART_TX
- net labels removed: DATA_Enable_N, DATA_RX, DATA_TX, HK_BUS_V, LOADCELL_SPI_CS_N, LORA_RST_N, LORA_RX, LORA_TX, RFID_CLOCK, RFID_MODU_N
- wire segments 89 -> 96
Other:
- moved on the sheet: P301, P302
Changed lines of the file:
@@
 LIBS:SeeedOPL-Transistor-2016
 LIBS:Nestbox_v2-cache
-EELAYER 26 0
+EELAYER 25 0
 EELAYER END
 $Descr A4 11693 8268
@@
 L CONN_01X02 P301
 U 1 1 58653CFC
-P 4450 6900
+P 4400 6900
 AR Path="/58653CFC" Ref="P301"  Part="1"
 AR Path="/59EF7F04/58653CFC" Ref="P301"  Part="1"
-F 0 "P301" H 4450 7050 50  0000 C CNN
-F 1 "TST/RST" V 4550 6900 50  0000 C CNN
-F 2 "Socket_Strips:Socket_Strip_Straight_1x02" H 4450 6900 50  0001 C CNN
-F 3 "" H 4450 6900 50  0000 C CNN
-F 4 "" H 4450 6900 50  0001 C CNN "MPN"
-F 5 "" H 4450 6900 50  0001 C CNN "SKU"
-F 6 "" H 4450 6900 50  0001 C CNN "MouserLink"
-	1    4450 6900
+F 0 "P301" H 4400 7050 50  0000 C CNN
+F 1 "TST/RST" V 4500 6900 50  0000 C CNN
+F 2 "Socket_Strips:Socket_Strip_Straight_1x02" H 4400 6900 50  0001 C CNN
+F 3 "" H 4400 6900 50  0000 C CNN
+F 4 "" H 4400 6900 50  0001 C CNN "MPN"
+F 5 "" H 4400 6900 50  0001 C CNN "SKU"
+F 6 "" H 4400 6900 50  0001 C CNN "MouserLink"
+	1    4400 6900
 	0    1    1    0
 $EndComp
@@
 L CONN_01X02 P302
 U 1 1 587BB574
-P 4000 7600
+P 3950 7600
 AR Path="/587BB574" Ref="P302"  Part="1"
 AR Path="/59EF7F04/587BB574" Ref="P302"  Part="1"
-F 0 "P302" H 4000 7750 50  0000 C CNN
-F 1 "RX/TX" V 4100 7600 50  0000 C CNN
-F 2 "Socket_Strips:Socket_Strip_Straight_1x02" H 4000 7600 50  0001 C CNN
-F 3 "" H 4000 7600 50  0000 C CNN
-F 4 "" H 4000 7600 50  0001 C CNN "MPN"
-F 5 "" H 4000 7600 50  0001 C CNN "SKU"
-F 6 "" H 4000 7600 50  0001 C CNN "MouserLink"
-	1    4000 7600
-	0    1    1    0
-$EndComp
-Text GLabel 6400 6500 2    60   Input ~ 0
-LORA_RX
+F 0 "P302" H 3950 7750 50  0000 C CNN
+F 1 "RX/TX" V 4050 7600 50  0000 C CNN
+F 2 "Socket_Strips:Socket_Strip_Straight_1x02" H 3950 7600 50  0001 C CNN
+F 3 "" H 3950 7600 50  0000 C CNN
+F 4 "" H 3950 7600 50  0001 C CNN "MPN"
+F 5 "" H 3950 7600 50  0001 C CNN "SKU"
+F 6 "" H 3950 7600 50  0001 C CNN "MouserLink"
+	1    3950 7600
+	0    1    1    0
+$EndComp
 Text Label 2950 2450 0    60   ~ 0
 AVCC
@@
 Wire Wire Line
 	2450 2400 2450 2450
-Text GLabel 6400 6400 2    60   Input ~ 0
-LORA_TX
 Wire Wire Line
 	4100 6650 4350 6650
@@
 Wire Wire Line
 	6150 4750 6700 4750
-Text Label 6700 4750 0    60   ~ 0
+Text Label 6350 4750 0    60   ~ 0
 SPI_CLK
-Text GLabel 1300 4550 0    60   Input ~ 0
-RFID_MODU_N
-Text GLabel 1300 4750 0    60   Input ~ 0
-RFID_DATA
-Text GLabel 1300 4650 0    60   Input ~ 0
-RFID_CLOCK
 Wire Wire Line
 	1300 4550 1550 4550
@@
 Wire Wire Line
 	1300 4750 1550 4750
-Text GLabel 1300 4150 0    60   Input ~ 0
-HK_BUS_V
-Text GLabel 1300 4250 0    60   Input ~ 0
-HK_BAT_V
 Text GLabel 1300 4350 0    60   Input ~ 0
 HK_SOLAR_V
@@
 Wire Wire Line
 	6150 4050 6700 4050
-Text Label 6300 4550 0    60   ~ 0
-LOADCELL_SPI_CS_N
 Text GLabel 1300 3750 0    60   Input ~ 0
 LB2_DETECT
 Text GLabel 1300 3850 0    60   Input ~ 0
 LB1_LED
-Text GLabel 1300 3950 0    60   Input ~ 0
+Text GLabel 1250 3350 0    60   Input ~ 0
 LB1_DETECT
 Wire Wire Line
@@
 Text Label 10850 4550 2    60   ~ 0
 DBG_Switch
-Text GLabel 3800 6450 3    60   Input ~ 0
-DATA_Enable_N
 $Comp
 L CP C301
@@
 	7750 1850 8900 1850
 Wire Wire Line
-	7750 1850 7750 1900
-Wire Wire Line
-	7750 1900 7000 1900
+	7750 1900 7750 1850
+Wire Wire Line
+	7000 1900 7750 1900
 Connection ~ 7500 1900
 Connection ~ 7100 1900
@@
 Wire Wire Line
 	4100 7350 4000 7350
-Text GLabel 4800 7350 2    60   Input ~ 0
-DATA_RX
 Connection ~ 3900 7350
 Wire Wire Line
 	3800 7350 3900 7350
-Text GLabel 3800 7350 0    60   Input ~ 0
-DATA_TX
 Wire Wire Line
 	4000 6450 4000 7400
 Wire Wire Line
 	3900 6450 3900 7400
-Text GLabel 6700 4050 2    60   Input ~ 0
-LORA_RST_N
 $Comp
 L R R?
@@
 Wire Wire Line
 	8750 1950 8900 1950
+Text HLabel 6700 4150 2    60   Input ~ 0
+SPI_MISO
+Text HLabel 6700 4250 2    60   Input ~ 0
+SPI_MOSI
+Text HLabel 6700 4550 2    60   Input ~ 0
+LOADCELL_SPI_CS
+Text HLabel 6700 4750 2    60   Input ~ 0
+SPI_CLK
+Wire Wire Line
+	6150 4650 6700 4650
+Text HLabel 6700 4650 2    60   Input ~ 0
+LOADCELL_DRDY
+Text HLabel 3800 6600 3    60   Input ~ 0
+RFID_DATA
+Wire Wire Line
+	3800 6600 3800 6450
+Text HLabel 1300 3950 0    60   Input ~ 0
+RFID_MODU
+Text HLabel 4000 2200 1    60   Input ~ 0
+RFID_CLK
+Wire Wire Line
+	4000 2200 4000 2450
+Text HLabel 1300 4150 0    60   Input ~ 0
+HK_5V_V
+Text HLabel 1300 4250 0    60   Input ~ 0
+HK_BAT_V
+Text HLabel 1300 4850 0    60   Input ~ 0
+5V_ENABLE
+Wire Wire Line
+	1300 4450 1550 4450
+Text HLabel 3200 6550 3    60   Input ~ 0
+LDO_ENABLE
+Text HLabel 3800 7350 0    60   Input ~ 0
+LORA_UART_TX
+Text HLabel 4800 7350 2    60   Input ~ 0
+LORA_UART_RX
+Text HLabel 6400 6400 2    60   Input ~ 0
+WIFI_UART_RX
+Text HLabel 6400 6500 2    60   Input ~ 0
+WIFI_UART_TX
+Text HLabel 6700 4050 2    60   Input ~ 0
+LORA_RESET_N
+Text HLabel 3400 6550 3    60   Input ~ 0
+WIFI_EN
+Wire Wire Line
+	3400 6550 3400 6450
+Wire Wire Line
+	1300 4850 1550 4850
+Wire Wire Line
+	3200 6550 3200 6450
 $EndSCHEMATC

Commit message: finished power supply schematics
Connections:
- net labels added: BAT_TEST_ENABLE, LOADCELL_EXC_A_N, LOADCELL_EXC_A_P, LOADCELL_EXC_B_N, LOADCELL_EXC_B_P, RFID_SLEEP_N
- net labels removed: RFID_MODU
- wire segments 96 -> 101
Changed lines of the file:
@@
 	3800 6600 3800 6450
 Text HLabel 1300 3950 0    60   Input ~ 0
-RFID_MODU
+RFID_SLEEP_N
 Text HLabel 4000 2200 1    60   Input ~ 0
 RFID_CLK
@@
 Wire Wire Line
 	3200 6550 3200 6450
+Wire Wire Line
+	6150 4350 6700 4350
+Wire Wire Line
+	6150 4450 6700 4450
+Wire Wire Line
+	6150 3850 6700 3850
+Wire Wire Line
+	6150 3950 6700 3950
+Text HLabel 6700 4450 2    60   Input ~ 0
+LOADCELL_EXC_A_P
+Text HLabel 6700 4350 2    60   Input ~ 0
+LOADCELL_EXC_A_N
+Text HLabel 6700 3950 2    60   Input ~ 0
+LOADCELL_EXC_B_P
+Text HLabel 6700 3850 2    60   Input ~ 0
+LOADCELL_EXC_B_N
+Text HLabel 3300 6550 3    60   Input ~ 0
+BAT_TEST_ENABLE
+Wire Wire Line
+	3300 6550 3300 6450
 $EndSCHEMATC

Commit message: added PIR and lightbarrier headers
Parts:
- gave numbers to parts that had none: 3
- renumbered C306 to C301, C303 to C302, C304 to C303, C305 to C304, C307 to C305, C301 to C306, C302 to C307, P302 to P301, P301 to P302, R306 to R301, R301 to R302, R304 to R306, R305 to R307, R302 to R308, R303 to R309
Connections:
- net labels added: HK_5V_PG, HK_BAT_I, LB_EXTERNAL_DETECT, LB_INTERNAL_DETECT, PIR_EN, PIR_IN
- net labels removed: HK_5V_V, LB1_DETECT, LB2_DETECT, LB2_LED
- wire segments 101 -> 102
