File: Nestbox_v2/Nestbox_v2_control.sch (KiCad schematic (older format))
At the start: 27 parts, among them CON301 Micro_SD_Card, P301 RX/TX, P302 TST/RST, P303 DEBUG_3V3, SW301 SMD-BUTTON_2P-3.0X2.5X1.2+0.4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, U301 MSP430FR5969, Y301 Crystal

Commit message: added stitching vias at power stage; reverse polarity protection and SD car enable mosfet
Parts:
- added Q301: NTR3A052PZT1G, TO_SOT_Packages_SMD:SOT-23, symbol Q_PMOS_DGS
Connections:
- net +3V3: now also Q301.1 (D); no longer R302.2
- net SD_CARD_ENABLE: now reaches U301.14 (PJ.2/TMS/ACLK/SROSCOFF/C8)
- net SD_CARD_ENABLE: now also Q301.2 (G)
- new net: Q301.3 (S), R302.2
Changed lines of the file:
@@
 $EndComp
 $Comp
-L GND #PWR022
+L GND #PWR313
 U 1 1 586416A7
 P 6150 3750
-F 0 "#PWR022" H 6150 3500 50  0001 C CNN
+F 0 "#PWR313" H 6150 3500 50  0001 C CNN
 F 1 "GND" H 6150 3600 50  0000 C CNN
 F 2 "" H 6150 3750 50  0000 C CNN
@@
 $EndComp
 $Comp
-L +3.3V #PWR023
+L +3.3V #PWR308
 U 1 1 586418DC
 P 4300 1900
-F 0 "#PWR023" H 4300 1750 50  0001 C CNN
+F 0 "#PWR308" H 4300 1750 50  0001 C CNN
 F 1 "+3.3V" H 4300 2040 50  0000 C CNN
 F 2 "" H 4300 1900 50  0000 C CNN
@@
 $EndComp
 $Comp
-L GND #PWR024
+L GND #PWR302
 U 1 1 58641ADD
 P 2500 2250
-F 0 "#PWR024" H 2500 2000 50  0001 C CNN
+F 0 "#PWR302" H 2500 2000 50  0001 C CNN
 F 1 "GND" H 2500 2100 50  0000 C CNN
 F 2 "" H 2500 2250 50  0000 C CNN
@@
 $EndComp
 $Comp
-L +3.3V #PWR025
+L +3.3V #PWR303
 U 1 1 58641B00
 P 2850 1700
-F 0 "#PWR025" H 2850 1550 50  0001 C CNN
+F 0 "#PWR303" H 2850 1550 50  0001 C CNN
 F 1 "+3.3V" H 2850 1840 50  0000 C CNN
 F 2 "" H 2850 1700 50  0000 C CNN
@@
 $EndComp
 $Comp
-L GND #PWR026
+L GND #PWR309
 U 1 1 58652F3A
 P 4700 2450
-F 0 "#PWR026" H 4700 2200 50  0001 C CNN
+F 0 "#PWR309" H 4700 2200 50  0001 C CNN
 F 1 "GND" H 4700 2300 50  0000 C CNN
 F 2 "" H 4700 2450 50  0000 C CNN
@@
 $EndComp
 $Comp
-L GND #PWR027
+L GND #PWR305
 U 1 1 5865358A
 P 3400 1600
-F 0 "#PWR027" H 3400 1350 50  0001 C CNN
+F 0 "#PWR305" H 3400 1350 50  0001 C CNN
 F 1 "GND" H 3400 1450 50  0000 C CNN
 F 2 "" H 3400 1600 50  0000 C CNN
@@
 $EndComp
 $Comp
-L GNDA #PWR028
+L GNDA #PWR304
 U 1 1 587B6902
 P 3300 2400
-F 0 "#PWR028" H 3300 2150 50  0001 C CNN
+F 0 "#PWR304" H 3300 2150 50  0001 C CNN
 F 1 "GNDA" H 3300 2250 50  0000 C CNN
 F 2 "" H 3300 2400 50  0000 C CNN
@@
 $EndComp
 $Comp
-L GNDA #PWR029
+L GNDA #PWR306
 U 1 1 587B69F1
 P 3600 2400
-F 0 "#PWR029" H 3600 2150 50  0001 C CNN
+F 0 "#PWR306" H 3600 2150 50  0001 C CNN
 F 1 "GNDA" H 3600 2250 50  0000 C CNN
 F 2 "" H 3600 2400 50  0000 C CNN
@@
 $EndComp
 $Comp
-L GNDA #PWR030
+L GNDA #PWR307
 U 1 1 587B6A2F
 P 3900 2400
-F 0 "#PWR030" H 3900 2150 50  0001 C CNN
+F 0 "#PWR307" H 3900 2150 50  0001 C CNN
 F 1 "GNDA" H 3900 2250 50  0000 C CNN
 F 2 "" H 3900 2400 50  0000 C CNN
@@
 $EndComp
 $Comp
-L GND #PWR031
+L GND #PWR319
 U 1 1 587B96DD
 P 10000 5300
-F 0 "#PWR031" H 10000 5050 50  0001 C CNN
+F 0 "#PWR319" H 10000 5050 50  0001 C CNN
 F 1 "GND" H 10000 5150 50  0000 C CNN
 F 2 "" H 10000 5300 50  0000 C CNN
@@
 $EndComp
 $Comp
-L +3.3V #PWR032
+L +3.3V #PWR318
 U 1 1 587B9736
 P 10000 4100
-F 0 "#PWR032" H 10000 3950 50  0001 C CNN
+F 0 "#PWR318" H 10000 3950 50  0001 C CNN
 F 1 "+3.3V" H 10000 4240 50  0000 C CNN
 F 2 "" H 10000 4100 50  0000 C CNN
@@
 $EndComp
 $Comp
-L GND #PWR033
+L GND #PWR317
 U 1 1 587B97E4
 P 9600 5400
-F 0 "#PWR033" H 9600 5150 50  0001 C CNN
+F 0 "#PWR317" H 9600 5150 50  0001 C CNN
 F 1 "GND" H 9600 5250 50  0000 C CNN
 F 2 "" H 9600 5400 50  0000 C CNN
@@
 $EndComp
 $Comp
-L GND #PWR034
+L GND #PWR316
 U 1 1 587B9834
 P 9300 5400
-F 0 "#PWR034" H 9300 5150 50  0001 C CNN
+F 0 "#PWR316" H 9300 5150 50  0001 C CNN
 F 1 "GND" H 9300 5250 50  0000 C CNN
 F 2 "" H 9300 5400 50  0000 C CNN
@@
 	9300 4950 9300 5050
 $Comp
-L GND #PWR035
+L GND #PWR301
 U 1 1 587D2523
 P 2450 2450
-F 0 "#PWR035" H 2450 2200 50  0001 C CNN
+F 0 "#PWR301" H 2450 2200 50  0001 C CNN
 F 1 "GND" H 2450 2300 50  0000 C CNN
 F 2 "" H 2450 2450 50  0000 C CNN
@@
 	4350 6650 4350 6700
 $Comp
-L +3.3V #PWR036
+L +3.3V #PWR310
 U 1 1 58BC4BB7
 P 4850 6600
-F 0 "#PWR036" H 4850 6450 50  0001 C CNN
+F 0 "#PWR310" H 4850 6450 50  0001 C CNN
 F 1 "+3.3V" H 4850 6740 50  0000 C CNN
 F 2 "" H 4850 6600 50  0000 C CNN
@@
 	10200 4850 10200 4900
 $Comp
-L GND #PWR037
+L GND #PWR320
 U 1 1 58BF19D6
 P 10200 5300
-F 0 "#PWR037" H 10200 5050 50  0001 C CNN
+F 0 "#PWR320" H 10200 5050 50  0001 C CNN
 F 1 "GND" H 10200 5150 50  0000 C CNN
 F 2 "" H 10200 5300 50  0000 C CNN
@@
 SPI_MOSI
 $Comp
-L +3.3V #PWR038
-U 1 1 59FCECA7
-P 6500 1600
-F 0 "#PWR038" H 6500 1450 50  0001 C CNN
-F 1 "+3.3V" H 6500 1740 50  0000 C CNN
-F 2 "" H 6500 1600 50  0000 C CNN
-F 3 "" H 6500 1600 50  0000 C CNN
-	1    6500 1600
-	0    -1   -1   0
-$EndComp
-$Comp
-L GND #PWR039
+L GND #PWR315
 U 1 1 59FCED84
 P 7000 1900
-F 0 "#PWR039" H 7000 1650 50  0001 C CNN
+F 0 "#PWR315" H 7000 1650 50  0001 C CNN
 F 1 "GND" H 7000 1750 50  0000 C CNN
 F 2 "" H 7000 1900 50  0000 C CNN
@@
 	0    1    1    0
 $EndComp
-Wire Wire Line
-	6500 1600 6600 1600
 $Comp
 L R R306
@@
 $EndComp
 $Comp
-L +3.3V #PWR040
+L +3.3V #PWR312
 U 1 1 5B0C49AB
 P 5900 7400
-F 0 "#PWR040" H 5900 7250 50  0001 C CNN
+F 0 "#PWR312" H 5900 7250 50  0001 C CNN
 F 1 "+3.3V" H 5900 7540 50  0000 C CNN
 F 2 "" H 5900 7400 50  0000 C CNN
@@
 $EndComp
 $Comp
-L GND #PWR041
+L GND #PWR311
 U 1 1 5B0C4B76
 P 5800 7400
-F 0 "#PWR041" H 5800 7150 50  0001 C CNN
+F 0 "#PWR311" H 5800 7150 50  0001 C CNN
 F 1 "GND" H 5800 7250 50  0000 C CNN
 F 2 "" H 5800 7400 50  0000 C CNN
@@
 PIR_IN2
 Connection ~ 10200 4550
+$Comp
+L +3.3V #PWR314
+U 1 1 5B1824F8
+P 6550 950
+F 0 "#PWR314" H 6550 800 50  0001 C CNN
+F 1 "+3.3V" H 6565 1123 50  0000 C CNN
+F 2 "" H 6550 950 50  0000 C CNN
+F 3 "" H 6550 950 50  0000 C CNN
+	1    6550 950
+	1    0    0    -1
+$EndComp
+$Comp
+L Q_PMOS_DGS Q301
+U 1 1 5B1824FE
+P 6450 1250
+F 0 "Q301" H 6650 1300 50  0000 L CNN
+F 1 "NTR3A052PZT1G" H 6650 1200 50  0000 L CNN
+F 2 "TO_SOT_Packages_SMD:SOT-23" H 6650 1350 50  0001 C CNN
+F 3 "" H 6450 1250 50  0001 C CNN
+	1    6450 1250
+	1    0    0    -1
+$EndComp
+Wire Wire Line
+	6100 1250 6250 1250
+Wire Wire Line
+	6550 1050 6550 950
+Wire Wire Line
+	6600 1600 6550 1600
+Wire Wire Line
+	6550 1600 6550 1450
+Text Label 6100 1250 2    60   ~ 0
+SD_CARD_ENABLE
+Text Label 3300 6550 3    60   ~ 0
+SD_CARD_ENABLE
 $EndSCHEMATC

Commit message: finished routing. DRC clean
Parts:
- removed R302: 0E, Resistors_SMD:R_0603, symbol R
- CON301: footprint SeeedOPL-Connector-2016:MICRO-SD9+4P-SMD-16.1X14.5X1.85MM -> Octanis3:MICRO-SD9+4P-SMD-16.1X14.5X1.85MM
Connections:
- net GNDA is gone; now on net GND: U301.41 (AVSS), U301.44 (AVSS), U301.47 (AVSS)
- net SPI_SCK is gone; now on net SPI_CLK: R304.2
- net GND: now also CON301.9 (SHIELD)
- net at C306.1, C307.1, CON301.4 (VDD): now also Q301.3 (S)
Changed lines of the file:
@@
 $EndComp
 $Comp
-L GND #PWR313
+L GND #PWR023
 U 1 1 586416A7
 P 6150 3750
-F 0 "#PWR313" H 6150 3500 50  0001 C CNN
+F 0 "#PWR023" H 6150 3500 50  0001 C CNN
 F 1 "GND" H 6150 3600 50  0000 C CNN
 F 2 "" H 6150 3750 50  0000 C CNN
@@
 $EndComp
 $Comp
-L +3.3V #PWR308
+L +3.3V #PWR024
 U 1 1 586418DC
 P 4300 1900
-F 0 "#PWR308" H 4300 1750 50  0001 C CNN
+F 0 "#PWR024" H 4300 1750 50  0001 C CNN
 F 1 "+3.3V" H 4300 2040 50  0000 C CNN
 F 2 "" H 4300 1900 50  0000 C CNN
@@
 $EndComp
 $Comp
-L GND #PWR302
+L GND #PWR025
 U 1 1 58641ADD
 P 2500 2250
-F 0 "#PWR302" H 2500 2000 50  0001 C CNN
+F 0 "#PWR025" H 2500 2000 50  0001 C CNN
 F 1 "GND" H 2500 2100 50  0000 C CNN
 F 2 "" H 2500 2250 50  0000 C CNN
@@
 $EndComp
 $Comp
-L +3.3V #PWR303
+L +3.3V #PWR026
 U 1 1 58641B00
 P 2850 1700
-F 0 "#PWR303" H 2850 1550 50  0001 C CNN
+F 0 "#PWR026" H 2850 1550 50  0001 C CNN
 F 1 "+3.3V" H 2850 1840 50  0000 C CNN
 F 2 "" H 2850 1700 50  0000 C CNN
@@
 $EndComp
 $Comp
-L GND #PWR309
+L GND #PWR027
 U 1 1 58652F3A
 P 4700 2450
-F 0 "#PWR309" H 4700 2200 50  0001 C CNN
+F 0 "#PWR027" H 4700 2200 50  0001 C CNN
 F 1 "GND" H 4700 2300 50  0000 C CNN
 F 2 "" H 4700 2450 50  0000 C CNN
@@
 $EndComp
 $Comp
-L GND #PWR305
+L GND #PWR028
 U 1 1 5865358A
 P 3400 1600
-F 0 "#PWR305" H 3400 1350 50  0001 C CNN
+F 0 "#PWR028" H 3400 1350 50  0001 C CNN
 F 1 "GND" H 3400 1450 50  0000 C CNN
 F 2 "" H 3400 1600 50  0000 C CNN
@@
 	1    2850 2000
 	0    -1   -1   0
-$EndComp
-$Comp
-L GNDA #PWR304
-U 1 1 587B6902
-P 3300 2400
-F 0 "#PWR304" H 3300 2150 50  0001 C CNN
-F 1 "GNDA" H 3300 2250 50  0000 C CNN
-F 2 "" H 3300 2400 50  0000 C CNN
-F 3 "" H 3300 2400 50  0000 C CNN
-	1    3300 2400
-	-1   0    0    1
-$EndComp
-$Comp
-L GNDA #PWR306
-U 1 1 587B69F1
-P 3600 2400
-F 0 "#PWR306" H 3600 2150 50  0001 C CNN
-F 1 "GNDA" H 3600 2250 50  0000 C CNN
-F 2 "" H 3600 2400 50  0000 C CNN
-F 3 "" H 3600 2400 50  0000 C CNN
-	1    3600 2400
-	-1   0    0    1
-$EndComp
-$Comp
-L GNDA #PWR307
-U 1 1 587B6A2F
-P 3900 2400
-F 0 "#PWR307" H 3900 2150 50  0001 C CNN
-F 1 "GNDA" H 3900 2250 50  0000 C CNN
-F 2 "" H 3900 2400 50  0000 C CNN
-F 3 "" H 3900 2400 50  0000 C CNN
-	1    3900 2400
-	-1   0    0    1
 $EndComp
 $Comp
@@
 $EndComp
 $Comp
-L GND #PWR319
+L GND #PWR029
 U 1 1 587B96DD
 P 10000 5300
-F 0 "#PWR319" H 10000 5050 50  0001 C CNN
+F 0 "#PWR029" H 10000 5050 50  0001 C CNN
 F 1 "GND" H 10000 5150 50  0000 C CNN
 F 2 "" H 10000 5300 50  0000 C CNN
@@
 $EndComp
 $Comp
-L +3.3V #PWR318
+L +3.3V #PWR030
 U 1 1 587B9736
 P 10000 4100
-F 0 "#PWR318" H 10000 3950 50  0001 C CNN
+F 0 "#PWR030" H 10000 3950 50  0001 C CNN
 F 1 "+3.3V" H 10000 4240 50  0000 C CNN
 F 2 "" H 10000 4100 50  0000 C CNN
@@
 $EndComp
 $Comp
-L GND #PWR317
+L GND #PWR031
 U 1 1 587B97E4
 P 9600 5400
-F 0 "#PWR317" H 9600 5150 50  0001 C CNN
+F 0 "#PWR031" H 9600 5150 50  0001 C CNN
 F 1 "GND" H 9600 5250 50  0000 C CNN
 F 2 "" H 9600 5400 50  0000 C CNN
@@
 $EndComp
 $Comp
-L GND #PWR316
+L GND #PWR032
 U 1 1 587B9834
 P 9300 5400
-F 0 "#PWR316" H 9300 5150 50  0001 C CNN
+F 0 "#PWR032" H 9300 5150 50  0001 C CNN
 F 1 "GND" H 9300 5250 50  0000 C CNN
 F 2 "" H 9300 5400 50  0000 C CNN
@@
 	9300 4950 9300 5050
 $Comp
-L GND #PWR301
+L GND #PWR033
 U 1 1 587D2523
 P 2450 2450
-F 0 "#PWR301" H 2450 2200 50  0001 C CNN
+F 0 "#PWR033" H 2450 2200 50  0001 C CNN
 F 1 "GND" H 2450 2300 50  0000 C CNN
 F 2 "" H 2450 2450 50  0000 C CNN
@@
 	4350 6650 4350 6700
 $Comp
-L +3.3V #PWR310
+L +3.3V #PWR034
 U 1 1 58BC4BB7
 P 4850 6600
-F 0 "#PWR310" H 4850 6450 50  0001 C CNN
+F 0 "#PWR034" H 4850 6450 50  0001 C CNN
 F 1 "+3.3V" H 4850 6740 50  0000 C CNN
 F 2 "" H 4850 6600 50  0000 C CNN
@@
 	10200 4850 10200 4900
 $Comp
-L GND #PWR320
+L GND #PWR035
 U 1 1 58BF19D6
 P 10200 5300
-F 0 "#PWR320" H 10200 5050 50  0001 C CNN
+F 0 "#PWR035" H 10200 5050 50  0001 C CNN
 F 1 "GND" H 10200 5150 50  0000 C CNN
 F 2 "" H 10200 5300 50  0000 C CNN
@@
 Wire Wire Line
 	6150 4750 6700 4750
-Text Label 6350 4750 0    60   ~ 0
+Text Label 6200 4750 0    60   ~ 0
 SPI_CLK
 Wire Wire Line
@@
 F 0 "CON301" H 9750 2367 50  0000 C CNN
 F 1 "Micro_SD_Card" H 9750 2276 50  0000 C CNN
-F 2 "SeeedOPL-Connector-2016:MICRO-SD9+4P-SMD-16.1X14.5X1.85MM" H 10950 1950 50  0001 C CNN
+F 2 "Octanis3:MICRO-SD9+4P-SMD-16.1X14.5X1.85MM" H 10950 1950 50  0001 C CNN
 F 3 "" H 9800 1650 50  0000 C CNN
 	1    9800 1650
@@
 SPI_MOSI
 $Comp
-L GND #PWR315
+L GND #PWR036
 U 1 1 59FCED84
 P 7000 1900
-F 0 "#PWR315" H 7000 1650 50  0001 C CNN
+F 0 "#PWR036" H 7000 1650 50  0001 C CNN
 F 1 "GND" H 7000 1750 50  0000 C CNN
 F 2 "" H 7000 1900 50  0000 C CNN
@@
 	0    1    1    0
 $EndComp
-Text Label 7800 1750 0    60   ~ 0
-SPI_SCK
+Text Label 7900 1750 0    60   ~ 0
+SPI_CLK
 Text Label 7800 1950 0    60   ~ 0
 SPI_MISO
@@
 $EndComp
 Wire Wire Line
-	6900 1600 7750 1600
+	6550 1600 7750 1600
 Connection ~ 7100 1600
 Wire Wire Line
@@
 Connection ~ 7500 1900
 Connection ~ 7100 1900
-$Comp
-L R R302
-U 1 1 59FF21A2
-P 6750 1600
-F 0 "R302" V 6543 1600 50  0000 C CNN
-F 1 "0E" V 6634 1600 50  0000 C CNN
-F 2 "Resistors_SMD:R_0603" V 6680 1600 50  0001 C CNN
-F 3 "" H 6750 1600 50  0000 C CNN
-	1    6750 1600
-	0    1    1    0
-$EndComp
 $Comp
 L R R306
@@
 	8750 1750 8900 1750
 Wire Wire Line
-	8450 1750 7800 1750
+	8450 1750 7900 1750
 $Comp
 L R R305
@@
 $EndComp
 $Comp
-L +3.3V #PWR312
+L +3.3V #PWR037
 U 1 1 5B0C49AB
 P 5900 7400
-F 0 "#PWR312" H 5900 7250 50  0001 C CNN
+F 0 "#PWR037" H 5900 7250 50  0001 C CNN
 F 1 "+3.3V" H 5900 7540 50  0000 C CNN
 F 2 "" H 5900 7400 50  0000 C CNN
@@
 $EndComp
 $Comp
-L GND #PWR311
+L GND #PWR038
 U 1 1 5B0C4B76
 P 5800 7400
-F 0 "#PWR311" H 5800 7150 50  0001 C CNN
+F 0 "#PWR038" H 5800 7150 50  0001 C CNN
 F 1 "GND" H 5800 7250 50  0000 C CNN
 F 2 "" H 5800 7400 50  0000 C CNN
@@
 Connection ~ 10200 4550
 $Comp
-L +3.3V #PWR314
+L +3.3V #PWR039
 U 1 1 5B1824F8
 P 6550 950
-F 0 "#PWR314" H 6550 800 50  0001 C CNN
+F 0 "#PWR039" H 6550 800 50  0001 C CNN
 F 1 "+3.3V" H 6565 1123 50  0000 C CNN
 F 2 "" H 6550 950 50  0000 C CNN
@@
 	6550 1050 6550 950
 Wire Wire Line
-	6600 1600 6550 1600
-Wire Wire Line
 	6550 1600 6550 1450
 Text Label 6100 1250 2    60   ~ 0
@@
 Text Label 3300 6550 3    60   ~ 0
 SD_CARD_ENABLE
+Wire Wire Line
+	10600 2250 10750 2250
+Wire Wire Line
+	10750 2250 10750 2300
+$Comp
+L GND #PWR040
+U 1 1 5B1863F0
+P 10750 2300
+F 0 "#PWR040" H 10750 2050 50  0001 C CNN
+F 1 "GND" H 10750 2150 50  0000 C CNN
+F 2 "" H 10750 2300 50  0000 C CNN
+F 3 "" H 10750 2300 50  0000 C CNN
+	1    10750 2300
+	1    0    0    -1
+$EndComp
+$Comp
+L GND #PWR041
+U 1 1 5B187286
+P 3300 2400
+F 0 "#PWR041" H 3300 2150 50  0001 C CNN
+F 1 "GND" H 3300 2250 50  0000 C CNN
+F 2 "" H 3300 2400 50  0000 C CNN
+F 3 "" H 3300 2400 50  0000 C CNN
+	1    3300 2400
+	-1   0    0    1
+$EndComp
+$Comp
+L GND #PWR042
+U 1 1 5B1872E2
+P 3600 2400
+F 0 "#PWR042" H 3600 2150 50  0001 C CNN
+F 1 "GND" H 3600 2250 50  0000 C CNN
+F 2 "" H 3600 2400 50  0000 C CNN
+F 3 "" H 3600 2400 50  0000 C CNN
+	1    3600 2400
+	-1   0    0    1
+$EndComp
+$Comp
+L GND #PWR043
+U 1 1 5B18733E
+P 3900 2400
+F 0 "#PWR043" H 3900 2150 50  0001 C CNN
+F 1 "GND" H 3900 2250 50  0000 C CNN
+F 2 "" H 3900 2400 50  0000 C CNN
+F 3 "" H 3900 2400 50  0000 C CNN
+	1    3900 2400
+	-1   0    0    1
+$EndComp
 $EndSCHEMATC

Commit message: corrected transistor pins
Parts:
- removed Q301: NTR3A052PZT1G, TO_SOT_Packages_SMD:SOT-23, symbol Q_PMOS_DGS
- added Q301: NTR3A052PZT1G, TO_SOT_Packages_SMD:TSOT-23, symbol Q_PMOS_GSD
Connections:
- net +3V3: now also Q301.3 (D)
- net SD_CARD_ENABLE: now also Q301.1 (G)
- net at C306.1, C307.1, CON301.4 (VDD): now also Q301.2 (S)
Changed lines of the file:
@@
 $EndComp
 $Comp
-L GND #PWR023
+L GND #PWR313
 U 1 1 586416A7
 P 6150 3750
-F 0 "#PWR023" H 6150 3500 50  0001 C CNN
+F 0 "#PWR313" H 6150 3500 50  0001 C CNN
 F 1 "GND" H 6150 3600 50  0000 C CNN
 F 2 "" H 6150 3750 50  0000 C CNN
@@
 $EndComp
 $Comp
-L +3.3V #PWR024
+L +3.3V #PWR308
 U 1 1 586418DC
 P 4300 1900
-F 0 "#PWR024" H 4300 1750 50  0001 C CNN
+F 0 "#PWR308" H 4300 1750 50  0001 C CNN
 F 1 "+3.3V" H 4300 2040 50  0000 C CNN
 F 2 "" H 4300 1900 50  0000 C CNN
@@
 $EndComp
 $Comp
-L GND #PWR025
+L GND #PWR302
 U 1 1 58641ADD
 P 2500 2250
-F 0 "#PWR025" H 2500 2000 50  0001 C CNN
+F 0 "#PWR302" H 2500 2000 50  0001 C CNN
 F 1 "GND" H 2500 2100 50  0000 C CNN
 F 2 "" H 2500 2250 50  0000 C CNN
@@
 $EndComp
 $Comp
-L +3.3V #PWR026
+L +3.3V #PWR303
 U 1 1 58641B00
 P 2850 1700
-F 0 "#PWR026" H 2850 1550 50  0001 C CNN
+F 0 "#PWR303" H 2850 1550 50  0001 C CNN
 F 1 "+3.3V" H 2850 1840 50  0000 C CNN
 F 2 "" H 2850 1700 50  0000 C CNN
@@
 $EndComp
 $Comp
-L GND #PWR027
+L GND #PWR309
 U 1 1 58652F3A
 P 4700 2450
-F 0 "#PWR027" H 4700 2200 50  0001 C CNN
+F 0 "#PWR309" H 4700 2200 50  0001 C CNN
 F 1 "GND" H 4700 2300 50  0000 C CNN
 F 2 "" H 4700 2450 50  0000 C CNN
@@
 $EndComp
 $Comp
-L GND #PWR028
+L GND #PWR305
 U 1 1 5865358A
 P 3400 1600
-F 0 "#PWR028" H 3400 1350 50  0001 C CNN
+F 0 "#PWR305" H 3400 1350 50  0001 C CNN
 F 1 "GND" H 3400 1450 50  0000 C CNN
 F 2 "" H 3400 1600 50  0000 C CNN
@@
 $EndComp
 $Comp
-L GND #PWR029
+L GND #PWR319
 U 1 1 587B96DD
 P 10000 5300
-F 0 "#PWR029" H 10000 5050 50  0001 C CNN
+F 0 "#PWR319" H 10000 5050 50  0001 C CNN
 F 1 "GND" H 10000 5150 50  0000 C CNN
 F 2 "" H 10000 5300 50  0000 C CNN
@@
 $EndComp
 $Comp
-L +3.3V #PWR030
+L +3.3V #PWR318
 U 1 1 587B9736
 P 10000 4100
-F 0 "#PWR030" H 10000 3950 50  0001 C CNN
+F 0 "#PWR318" H 10000 3950 50  0001 C CNN
 F 1 "+3.3V" H 10000 4240 50  0000 C CNN
 F 2 "" H 10000 4100 50  0000 C CNN
@@
 $EndComp
 $Comp
-L GND #PWR031
+L GND #PWR317
 U 1 1 587B97E4
 P 9600 5400
-F 0 "#PWR031" H 9600 5150 50  0001 C CNN
+F 0 "#PWR317" H 9600 5150 50  0001 C CNN
 F 1 "GND" H 9600 5250 50  0000 C CNN
 F 2 "" H 9600 5400 50  0000 C CNN
@@
 $EndComp
 $Comp
-L GND #PWR032
+L GND #PWR316
 U 1 1 587B9834
 P 9300 5400
-F 0 "#PWR032" H 9300 5150 50  0001 C CNN
+F 0 "#PWR316" H 9300 5150 50  0001 C CNN
 F 1 "GND" H 9300 5250 50  0000 C CNN
 F 2 "" H 9300 5400 50  0000 C CNN
@@
 	9300 4950 9300 5050
 $Comp
-L GND #PWR033
+L GND #PWR301
 U 1 1 587D2523
 P 2450 2450
-F 0 "#PWR033" H 2450 2200 50  0001 C CNN
+F 0 "#PWR301" H 2450 2200 50  0001 C CNN
 F 1 "GND" H 2450 2300 50  0000 C CNN
 F 2 "" H 2450 2450 50  0000 C CNN
@@
 	4350 6650 4350 6700
 $Comp
-L +3.3V #PWR034
+L +3.3V #PWR310
 U 1 1 58BC4BB7
 P 4850 6600
-F 0 "#PWR034" H 4850 6450 50  0001 C CNN
+F 0 "#PWR310" H 4850 6450 50  0001 C CNN
 F 1 "+3.3V" H 4850 6740 50  0000 C CNN
 F 2 "" H 4850 6600 50  0000 C CNN
@@
 	10200 4850 10200 4900
 $Comp
-L GND #PWR035
+L GND #PWR320
 U 1 1 58BF19D6
 P 10200 5300
-F 0 "#PWR035" H 10200 5050 50  0001 C CNN
+F 0 "#PWR320" H 10200 5050 50  0001 C CNN
 F 1 "GND" H 10200 5150 50  0000 C CNN
 F 2 "" H 10200 5300 50  0000 C CNN
@@
 SPI_MOSI
 $Comp
-L GND #PWR036
+L GND #PWR315
 U 1 1 59FCED84
 P 7000 1900
-F 0 "#PWR036" H 7000 1650 50  0001 C CNN
+F 0 "#PWR315" H 7000 1650 50  0001 C CNN
 F 1 "GND" H 7000 1750 50  0000 C CNN
 F 2 "" H 7000 1900 50  0000 C CNN
@@
 $EndComp
 $Comp
-L +3.3V #PWR037
+L +3.3V #PWR312
 U 1 1 5B0C49AB
 P 5900 7400
-F 0 "#PWR037" H 5900 7250 50  0001 C CNN
+F 0 "#PWR312" H 5900 7250 50  0001 C CNN
 F 1 "+3.3V" H 5900 7540 50  0000 C CNN
 F 2 "" H 5900 7400 50  0000 C CNN
@@
 $EndComp
 $Comp
-L GND #PWR038
+L GND #PWR311
 U 1 1 5B0C4B76
 P 5800 7400
-F 0 "#PWR038" H 5800 7150 50  0001 C CNN
+F 0 "#PWR311" H 5800 7150 50  0001 C CNN
 F 1 "GND" H 5800 7250 50  0000 C CNN
 F 2 "" H 5800 7400 50  0000 C CNN
@@
 Connection ~ 10200 4550
 $Comp
-L +3.3V #PWR039
+L +3.3V #PWR314
 U 1 1 5B1824F8
 P 6550 950
-F 0 "#PWR039" H 6550 800 50  0001 C CNN
+F 0 "#PWR314" H 6550 800 50  0001 C CNN
 F 1 "+3.3V" H 6565 1123 50  0000 C CNN
 F 2 "" H 6550 950 50  0000 C CNN
 F 3 "" H 6550 950 50  0000 C CNN
 	1    6550 950
-	1    0    0    -1
-$EndComp
-$Comp
-L Q_PMOS_DGS Q301
-U 1 1 5B1824FE
-P 6450 1250
-F 0 "Q301" H 6650 1300 50  0000 L CNN
-F 1 "NTR3A052PZT1G" H 6650 1200 50  0000 L CNN
-F 2 "TO_SOT_Packages_SMD:SOT-23" H 6650 1350 50  0001 C CNN
-F 3 "" H 6450 1250 50  0001 C CNN
-	1    6450 1250
 	1    0    0    -1
 $EndComp
@@
 	10750 2250 10750 2300
 $Comp
-L GND #PWR040
+L GND #PWR321
 U 1 1 5B1863F0
 P 10750 2300
-F 0 "#PWR040" H 10750 2050 50  0001 C CNN
+F 0 "#PWR321" H 10750 2050 50  0001 C CNN
 F 1 "GND" H 10750 2150 50  0000 C CNN
 F 2 "" H 10750 2300 50  0000 C CNN
@@
 $EndComp
 $Comp
-L GND #PWR041
+L GND #PWR304
 U 1 1 5B187286
 P 3300 2400
-F 0 "#PWR041" H 3300 2150 50  0001 C CNN
+F 0 "#PWR304" H 3300 2150 50  0001 C CNN
 F 1 "GND" H 3300 2250 50  0000 C CNN
 F 2 "" H 3300 2400 50  0000 C CNN
@@
 $EndComp
 $Comp
-L GND #PWR042
+L GND #PWR306
 U 1 1 5B1872E2
 P 3600 2400
-F 0 "#PWR042" H 3600 2150 50  0001 C CNN
+F 0 "#PWR306" H 3600 2150 50  0001 C CNN
 F 1 "GND" H 3600 2250 50  0000 C CNN
 F 2 "" H 3600 2400 50  0000 C CNN
@@
 $EndComp
 $Comp
-L GND #PWR043
+L GND #PWR307
 U 1 1 5B18733E
 P 3900 2400
-F 0 "#PWR043" H 3900 2150 50  0001 C CNN
+F 0 "#PWR307" H 3900 2150 50  0001 C CNN
 F 1 "GND" H 3900 2250 50  0000 C CNN
 F 2 "" H 3900 2400 50  0000 C CNN
@@
 	-1   0    0    1
 $EndComp
+$Comp
+L Q_PMOS_GSD Q301
+U 1 1 5B18BF22
+P 6450 1250
+F 0 "Q301" H 6650 1300 50  0000 L CNN
+F 1 "NTR3A052PZT1G" H 6650 1200 50  0000 L CNN
+F 2 "TO_SOT_Packages_SMD:TSOT-23" H 6650 1350 50  0001 C CNN
+F 3 "" H 6450 1250 50  0001 C CNN
+	1    6450 1250
+	1    0    0    -1
+$EndComp
 $EndSCHEMATC

Commit message: annotated schematic with necessary changes to load cell circuit. added pull-ups for enable PMOSes
Parts:
- added R?: 82k, Resistors_SMD:R_0603, symbol R
- C306: MPN (none) -> 293D107X0016D2TE3
Connections:
- net +3V3: now also R?.1
- net SD_CARD_ENABLE: now also R?.2
Changed lines of the file:
@@
 F 3 "" H 7100 1750 50  0000 C CNN
 F 4 "667-ECE-A0JKA101" H 7100 1750 60  0001 C CNN "Mouser-Part"
+F 5 "293D107X0016D2TE3" H 7100 1750 60  0001 C CNN "MPN"
 	1    7100 1750
 	1    0    0    -1
@@
 $EndComp
 Wire Wire Line
-	6100 1250 6250 1250
+	5800 1250 6250 1250
 Wire Wire Line
 	6550 1050 6550 950
 Wire Wire Line
 	6550 1600 6550 1450
-Text Label 6100 1250 2    60   ~ 0
+Text Label 5800 1250 2    60   ~ 0
 SD_CARD_ENABLE
 Text Label 3300 6550 3    60   ~ 0
@@
 	1    0    0    -1
 $EndComp
+$Comp
+L R R?
+U 1 1 5B28B132
+P 6150 1050
+F 0 "R?" H 6220 1096 50  0000 L CNN
+F 1 "82k" H 6220 1005 50  0000 L CNN
+F 2 "Resistors_SMD:R_0603" V 6080 1050 50  0001 C CNN
+F 3 "" H 6150 1050 50  0000 C CNN
+	1    6150 1050
+	1    0    0    -1
+$EndComp
+Wire Wire Line
+	6150 1200 6150 1250
+Connection ~ 6150 1250
+$Comp
+L +3.3V #PWR?
+U 1 1 5B28B3EE
+P 6150 850
+F 0 "#PWR?" H 6150 700 50  0001 C CNN
+F 1 "+3.3V" H 6165 1023 50  0000 C CNN
+F 2 "" H 6150 850 50  0000 C CNN
+F 3 "" H 6150 850 50  0000 C CNN
+	1    6150 850
+	1    0    0    -1
+$EndComp
+Wire Wire Line
+	6150 850  6150 900
 $EndSCHEMATC
