File: Nestbox_v2/Nestbox_v2_control.sch (KiCad schematic (older format))
At the start: 28 parts, among them CON301 Micro_SD_Card, P301 RX/TX, P302 TST/RST, P303 DEBUG_3V3, Q301 NTR3A052PZT1G, SW301 SMD-BUTTON_2P-3.0X2.5X1.2+0.4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, U301 MSP430FR5969, Y301 Crystal

Commit message: TAPEOUT second batch nestbox main + EM pcb. added pull-ups, corrected pmos of load cell, WIFI AND SDCARD ENABLE PMOS ARE STILL WRONGLY ORIENTED
Parts:
- added TP_RTC301: CONN_01X01, Socket_Strips:Socket_Strip_Straight_1x01_Pitch2.00mm, symbol CONN_01X01
- C304: footprint Capacitors_SMD:C_0603 -> Capacitors_SMD:C_0805
- C306: footprint Capacitors_SMD:C_0603 -> Capacitors_Tantalum_SMD:CP_Tantalum_Case-D_EIA-7343-31_Reflow
- gave numbers to parts that had none: 1
Connections:
- net LB1_LED: now also TP_RTC301.1 (P1)
Changed lines of the file:
@@
 $EndComp
 $Comp
-L GND #PWR313
+L GND #PWR314
 U 1 1 586416A7
 P 6150 3750
-F 0 "#PWR313" H 6150 3500 50  0001 C CNN
+F 0 "#PWR314" H 6150 3500 50  0001 C CNN
 F 1 "GND" H 6150 3600 50  0000 C CNN
 F 2 "" H 6150 3750 50  0000 C CNN
@@
 $EndComp
 $Comp
-L GND #PWR319
+L GND #PWR320
 U 1 1 587B96DD
 P 10000 5300
-F 0 "#PWR319" H 10000 5050 50  0001 C CNN
+F 0 "#PWR320" H 10000 5050 50  0001 C CNN
 F 1 "GND" H 10000 5150 50  0000 C CNN
 F 2 "" H 10000 5300 50  0000 C CNN
@@
 $EndComp
 $Comp
-L +3.3V #PWR318
+L +3.3V #PWR319
 U 1 1 587B9736
 P 10000 4100
-F 0 "#PWR318" H 10000 3950 50  0001 C CNN
+F 0 "#PWR319" H 10000 3950 50  0001 C CNN
 F 1 "+3.3V" H 10000 4240 50  0000 C CNN
 F 2 "" H 10000 4100 50  0000 C CNN
@@
 $EndComp
 $Comp
-L GND #PWR317
+L GND #PWR318
 U 1 1 587B97E4
 P 9600 5400
-F 0 "#PWR317" H 9600 5150 50  0001 C CNN
+F 0 "#PWR318" H 9600 5150 50  0001 C CNN
 F 1 "GND" H 9600 5250 50  0000 C CNN
 F 2 "" H 9600 5400 50  0000 C CNN
@@
 $EndComp
 $Comp
-L GND #PWR316
+L GND #PWR317
 U 1 1 587B9834
 P 9300 5400
-F 0 "#PWR316" H 9300 5150 50  0001 C CNN
+F 0 "#PWR317" H 9300 5150 50  0001 C CNN
 F 1 "GND" H 9300 5250 50  0000 C CNN
 F 2 "" H 9300 5400 50  0000 C CNN
@@
 	10200 4850 10200 4900
 $Comp
-L GND #PWR320
+L GND #PWR321
 U 1 1 58BF19D6
 P 10200 5300
-F 0 "#PWR320" H 10200 5050 50  0001 C CNN
+F 0 "#PWR321" H 10200 5050 50  0001 C CNN
 F 1 "GND" H 10200 5150 50  0000 C CNN
 F 2 "" H 10200 5300 50  0000 C CNN
@@
 SPI_MOSI
 $Comp
-L GND #PWR315
+L GND #PWR316
 U 1 1 59FCED84
 P 7000 1900
-F 0 "#PWR315" H 7000 1650 50  0001 C CNN
+F 0 "#PWR316" H 7000 1650 50  0001 C CNN
 F 1 "GND" H 7000 1750 50  0000 C CNN
 F 2 "" H 7000 1900 50  0000 C CNN
@@
 F 0 "C306" H 7218 1796 50  0000 L CNN
 F 1 "100u" H 7218 1705 50  0000 L CNN
-F 2 "Capacitors_SMD:C_0603" H 7138 1600 50  0001 C CNN
+F 2 "Capacitors_Tantalum_SMD:CP_Tantalum_Case-D_EIA-7343-31_Reflow" H 7138 1600 50  0001 C CNN
 F 3 "" H 7100 1750 50  0000 C CNN
 F 4 "667-ECE-A0JKA101" H 7100 1750 60  0001 C CNN "Mouser-Part"
@@
 F 0 "C304" V 4248 2000 50  0000 C CNN
 F 1 "10u" V 4339 2000 50  0000 C CNN
-F 2 "Capacitors_SMD:C_0603" H 4538 1850 50  0001 C CNN
+F 2 "Capacitors_SMD:C_0805" H 4538 1850 50  0001 C CNN
 F 3 "" H 4500 2000 50  0000 C CNN
 	1    4500 2000
@@
 Connection ~ 10200 4550
 $Comp
-L +3.3V #PWR314
+L +3.3V #PWR315
 U 1 1 5B1824F8
 P 6550 950
-F 0 "#PWR314" H 6550 800 50  0001 C CNN
+F 0 "#PWR315" H 6550 800 50  0001 C CNN
 F 1 "+3.3V" H 6565 1123 50  0000 C CNN
 F 2 "" H 6550 950 50  0000 C CNN
@@
 	10750 2250 10750 2300
 $Comp
-L GND #PWR321
+L GND #PWR322
 U 1 1 5B1863F0
 P 10750 2300
-F 0 "#PWR321" H 10750 2050 50  0001 C CNN
+F 0 "#PWR322" H 10750 2050 50  0001 C CNN
 F 1 "GND" H 10750 2150 50  0000 C CNN
 F 2 "" H 10750 2300 50  0000 C CNN
@@
 $EndComp
 $Comp
-L R R?
+L R R302
 U 1 1 5B28B132
 P 6150 1050
-F 0 "R?" H 6220 1096 50  0000 L CNN
+F 0 "R302" H 6220 1096 50  0000 L CNN
 F 1 "82k" H 6220 1005 50  0000 L CNN
 F 2 "Resistors_SMD:R_0603" V 6080 1050 50  0001 C CNN
@@
 Connection ~ 6150 1250
 $Comp
-L +3.3V #PWR?
+L +3.3V #PWR313
 U 1 1 5B28B3EE
 P 6150 850
-F 0 "#PWR?" H 6150 700 50  0001 C CNN
+F 0 "#PWR313" H 6150 700 50  0001 C CNN
 F 1 "+3.3V" H 6165 1023 50  0000 C CNN
 F 2 "" H 6150 850 50  0000 C CNN
@@
 Wire Wire Line
 	6150 850  6150 900
+Wire Wire Line
+	1450 3750 1450 3500
+Wire Wire Line
+	1450 3500 1400 3500
+Connection ~ 1450 3750
+$Comp
+L CONN_01X01 TP_RTC301
+U 1 1 5B29DDF6
+P 1400 3300
+F 0 "TP_RTC301" H 1400 3400 50  0000 C CNN
+F 1 "CONN_01X01" V 1500 3300 50  0000 C CNN
+F 2 "Socket_Strips:Socket_Strip_Straight_1x01_Pitch2.00mm" H 1400 3300 50  0001 C CNN
+F 3 "" H 1400 3300 50  0001 C CNN
+	1    1400 3300
+	0    -1   -1   0
+$EndComp
 $EndSCHEMATC
