File: Breadboards/PIR_wakeup/nestbox.kicad_pcb (KiCad board)
At the start: 2 copper layers, 42.8 x 27.5 mm, 14 parts

Commit message: Updated holes again
Used mounting hole component this time
Parts:
- added ?: , Mounting_Holes:MountingHole_5mm, F.Cu at (147.3, 116.1)
- added ?: , Mounting_Holes:MountingHole_5mm, F.Cu at (152.7, 97.7)
- added ?: , Mounting_Holes:MountingHole_5mm, F.Cu at (118.9, 116.1)
- added ?: , Mounting_Holes:MountingHole_5mm, F.Cu at (118.7, 98.6)
- moved C1 5.05 mm to (130.2, 117.0)
- moved R2 4.06 mm to (126.3, 113.9)
Routing:
- net Net-(C1-Pad1): track 12.3 -> 14.2 mm
- net GND: track 16.2 -> 15.6 mm
Other:
- outline, holes or cut-outs redrawn
- board text added: "Octanis PIR wakeup v1 Lennard"
Changed lines of the file:
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@@
     (links 29)
     (no_connects 0)
-    (area 113.699999 93.524999 156.600001 121.125001)
+    (area 113.156499 90.7015 158.179001 123.2665)
     (thickness 1.6)
-    (drawings 13)
-    (tracks 71)
+    (drawings 10)
+    (tracks 73)
     (zones 0)
-    (modules 14)
+    (modules 18)
     (nets 11)
   )
@@
     (add_net "Net-(RV1-Pad2)")
   )
+  (module Mounting_Holes:MountingHole_5mm (layer F.Cu)
+    (at 147.2565 116.078)
+    (descr "Mounting Hole 5mm, no annular")
+    (tags "mounting hole 5mm no annular")
+    (attr virtual)
+    (fp_text reference "" (at 0 -6) (layer F.SilkS)
+      (effects (font (size 1 1) (thickness 0.15)))
+    )
+    (fp_text value "" (at 0 6) (layer F.Fab)
+      (effects (font (size 1 1) (thickness 0.15)))
+    )
+    (fp_text user %R (at 0.3 0) (layer F.Fab)
+      (effects (font (size 1 1) (thickness 0.15)))
+    )
+    (fp_circle (center 0 0) (end 5 0) (layer Cmts.User) (width 0.15))
+    (fp_circle (center 0 0) (end 5.25 0) (layer F.CrtYd) (width 0.05))
+    (pad 1 np_thru_hole circle (at 0 0) (size 5 5) (drill 5) (layers *.Cu *.Mask))
+  )
+  (module Mounting_Holes:MountingHole_5mm (layer F.Cu)
+    (at 152.654 97.7265)
+    (descr "Mounting Hole 5mm, no annular")
+    (tags "mounting hole 5mm no annular")
+    (attr virtual)
+    (fp_text reference "" (at 0 -6) (layer F.SilkS)
+      (effects (font (size 1 1) (thickness 0.15)))
+    )
+    (fp_text value "" (at 0 6) (layer F.Fab)
+      (effects (font (size 1 1) (thickness 0.15)))
+    )
+    (fp_text user %R (at 0.3 0) (layer F.Fab)
+      (effects (font (size 1 1) (thickness 0.15)))
+    )
+    (fp_circle (center 0 0) (end 5 0) (layer Cmts.User) (width 0.15))
+    (fp_circle (center 0 0) (end 5.25 0) (layer F.CrtYd) (width 0.05))
+    (pad 1 np_thru_hole circle (at 0 0) (size 5 5) (drill 5) (layers *.Cu *.Mask))
+  )
+  (module Mounting_Holes:MountingHole_5mm (layer F.Cu)
+    (at 118.9355 116.1415)
+    (descr "Mounting Hole 5mm, no annular")
+    (tags "mounting hole 5mm no annular")
+    (attr virtual)
+    (fp_text reference "" (at 0 -6) (layer F.SilkS)
+      (effects (font (size 1 1) (thickness 0.15)))
+    )
+    (fp_text value "" (at 0 6) (layer F.Fab)
+      (effects (font (size 1 1) (thickness 0.15)))
+    )
+    (fp_text user %R (at 0.3 0) (layer F.Fab)
+      (effects (font (size 1 1) (thickness 0.15)))
+    )
+    (fp_circle (center 0 0) (end 5 0) (layer Cmts.User) (width 0.15))
+    (fp_circle (center 0 0) (end 5.25 0) (layer F.CrtYd) (width 0.05))
+    (pad 1 np_thru_hole circle (at 0 0) (size 5 5) (drill 5) (layers *.Cu *.Mask))
+  )
   (module IRA-S210ST01 (layer F.Cu)
     (at 124.0155 106.68 270)
@@
   )
   (module Capacitors_SMD:C_0603_HandSoldering (layer F.Cu)
-    (at 126.3015 113.7285 270)
+    (at 130.175 116.967 270)
     (descr "Capacitor SMD 0603, hand soldering")
     (tags "capacitor 0603")
@@
   )
   (module Resistors_SMD:R_0603_HandSoldering (layer F.Cu)
-    (at 122.2375 113.919 270)
+    (at 126.3015 113.8555 270)
     (descr "Resistor SMD 0603, hand soldering")
     (tags "resistor 0603")
@@
     )
   )
-  (gr_circle (center 153.28 96.71) (end 155.78 96.71) (layer Edge.Cuts) (width 0.15))
-  (gr_circle (center 153.14 117.92) (end 155.64 117.92) (layer Edge.Cuts) (width 0.15))
-  (gr_circle (center 116.68 118.16) (end 119.18 118.16) (layer Edge.Cuts) (width 0.15))
-  (gr_circle (center 116.89 96.62) (end 119.39 96.62) (layer Edge.Cuts) (width 0.15))
+  (module Mounting_Holes:MountingHole_5mm (layer F.Cu)
+    (at 118.6815 98.6155)
+    (descr "Mounting Hole 5mm, no annular")
+    (tags "mounting hole 5mm no annular")
+    (attr virtual)
+    (fp_text reference "" (at 0 -6) (layer F.SilkS)
+      (effects (font (size 1 1) (thickness 0.15)))
+    )
+    (fp_text value "" (at 0 6) (layer F.Fab)
+      (effects (font (size 1 1) (thickness 0.15)))
+    )
+    (fp_text user %R (at 0.3 0) (layer F.Fab)
+      (effects (font (size 1 1) (thickness 0.15)))
+    )
+    (fp_circle (center 0 0) (end 5 0) (layer Cmts.User) (width 0.15))
+    (fp_circle (center 0 0) (end 5.25 0) (layer F.CrtYd) (width 0.05))
+    (pad 1 np_thru_hole circle (at 0 0) (size 5 5) (drill 5) (layers *.Cu *.Mask))
+  )
+  (gr_text "Octanis PIR wakeup v1\nLennard" (at 124.3965 95.758) (layer F.SilkS)
+    (effects (font (size 0.75 0.75) (thickness 0.125)) (justify left))
+  )
   (gr_text GND (at 155.025 112.3315 90) (layer F.SilkS)
     (effects (font (size 0.75 0.75) (thickness 0.15)))
@@
   (segment (start 135.76422 108.9602) (end 132.0648 108.9602) (width 0.5) (layer F.Cu) (net 1))
   (segment (start 132.0648 108.9602) (end 132.05 108.975) (width 0.5) (layer F.Cu) (net 1))
+  (segment (start 130.175 117.917) (end 130.175 119.4435) (width 0.5) (layer F.Cu) (net 2))
+  (via (at 130.175 119.4435) (size 0.7) (drill 0.4) (layers F.Cu B.Cu) (net 2))
+  (segment (start 126.3015 114.9555) (end 126.3015 117.1575) (width 0.5) (layer F.Cu) (net 2))
+  (via (at 126.3015 117.1575) (size 0.7) (drill 0.4) (layers F.Cu B.Cu) (net 2))
   (segment (start 145.15 108.32) (end 145.15 105.7385) (width 0.5) (layer F.Cu) (net 2))
   (via (at 145.161 105.7275) (size 0.7) (drill 0.4) (layers F.Cu B.Cu) (net 2))
@@
   (via (at 144.2085 105.7275) (size 0.7) (drill 0.4) (layers F.Cu B.Cu) (net 2))
   (segment (start 144.2 105.736) (end 144.2085 105.7275) (width 0.5) (layer F.Cu) (net 2))
-  (segment (start 126.3015 114.6785) (end 126.3015 117.0305) (width 0.5) (layer F.Cu) (net 2))
-  (via (at 126.3015 117.0305) (size 0.7) (drill 0.4) (layers F.Cu B.Cu) (net 2))
-  (segment (start 122.2375 115.019) (end 122.2375 117.0305) (width 0.5) (layer F.Cu) (net 2))
-  (via (at 122.2375 117.0305) (size 0.7) (drill 0.4) (layers F.Cu B.Cu) (net 2))
   (segment (start 149 100.55) (end 149 98.5) (width 0.5) (layer F.Cu) (net 2))
   (via (at 149 98.5) (size 0.7) (drill 0.4) (layers F.Cu B.Cu) (net 2))
@@
   (segment (start 138.05 104.925) (end 138.05 108.92442) (width 0.5) (layer F.Cu) (net 6))
   (segment (start 138.05 108.92442) (end 138.08578 108.9602) (width 0.5) (layer F.Cu) (net 6))
-  (segment (start 130.1775 112.776) (end 126.304 112.776) (width 0.5) (layer F.Cu) (net 7))
-  (segment (start 126.304 112.776) (end 126.261 112.819) (width 0.5) (layer F.Cu) (net 7))
-  (segment (start 126.261 112.819) (end 122.2375 112.819) (width 0.5) (layer F.Cu) (net 7))
-  (segment (start 122.21945 108.47605) (end 122.21945 112.80095) (width 0.5) (layer F.Cu) (net 7))
-  (segment (start 122.21945 112.80095) (end 122.2375 112.819) (width 0.5) (layer F.Cu) (net 7))
+  (segment (start 126.3015 112.7555) (end 124.376 112.7555) (width 0.5) (layer F.Cu) (net 7))
+  (segment (start 122.21945 110.59895) (end 122.21945 108.47605) (width 0.5) (layer F.Cu) (net 7))
+  (segment (start 124.376 112.7555) (end 122.21945 110.59895) (width 0.5) (layer F.Cu) (net 7))
+  (segment (start 130.1775 112.776) (end 126.322 112.776) (width 0.5) (layer F.Cu) (net 7))
+  (segment (start 126.322 112.776) (end 126.3015 112.7555) (width 0.5) (layer F.Cu) (net 7))
+  (segment (start 130.1775 112.776) (end 130.1775 116.0145) (width 0.5) (layer F.Cu) (net 7))
+  (segment (start 130.1775 116.0145) (end 130.175 116.017) (width 0.5) (layer F.Cu) (net 7))
   (segment (start 152.7175 109.7915) (end 150.3045 109.7915) (width 0.5) (layer F.Cu) (net 8))
   (segment (start 149.266 110.83) (end 146.1 110.83) (width 0.5) (layer F.Cu) (net 8))
