File: RFID_BOARD_MLX90109/RFID_MLX90109.sch (KiCad schematic (older format))
At the start: 15 parts, among them J1 CONN_01X05, Q1 Q_NMOS_GSD, U1 MLX90109

Commit message: correct size of the PCB drawn with connector arrangement done as well
Parts:
- C2, C3: value C -> 6.8n
- C4: value C -> DNP
- R1, R5: value R -> DNP
- R2: value R -> 0R
- R4: value 33k -> 19k
- R6: value R -> 0
Other:
- note added: "0.81 V"
- note added: "13.85nF\nor 117uH\n"
- note removed: "0.87 V"
Changed lines of the file:
@@
 P 4500 4550
 F 0 "R4" V 4580 4550 50  0000 C CNN
-F 1 "33k" V 4500 4550 50  0000 C CNN
+F 1 "19k" V 4500 4550 50  0000 C CNN
 F 2 "Resistors_SMD:R_0603" V 4430 4550 50  0001 C CNN
 F 3 "" H 4500 4550 50  0001 C CNN
@@
 P 5250 3050
 F 0 "C4" H 5275 3150 50  0000 L CNN
-F 1 "C" H 5275 2950 50  0000 L CNN
+F 1 "DNP" H 5275 2950 50  0000 L CNN
 F 2 "Capacitors_SMD:C_0603" H 5288 2900 50  0001 C CNN
 F 3 "" H 5250 3050 50  0001 C CNN
@@
 Pull to GND for Operation\nPull to VDD for Standby\n
 Text Notes 4600 3950 2    60   ~ 0
-0.87 V
+0.81 V
 $Comp
 L C C3
@@
 P 5250 2800
 F 0 "C3" H 5275 2900 50  0000 L CNN
-F 1 "C" H 5275 2700 50  0000 L CNN
+F 1 "6.8n" H 5275 2700 50  0000 L CNN
 F 2 "Capacitors_SMD:C_0603" H 5288 2650 50  0001 C CNN
 F 3 "" H 5250 2800 50  0001 C CNN
@@
 P 5250 2550
 F 0 "C2" H 5275 2650 50  0000 L CNN
-F 1 "C" H 5275 2450 50  0000 L CNN
+F 1 "6.8n" H 5275 2450 50  0000 L CNN
 F 2 "Capacitors_SMD:C_0603" H 5288 2400 50  0001 C CNN
 F 3 "" H 5250 2550 50  0001 C CNN
@@
 P 3550 3800
 F 0 "R1" V 3343 3800 50  0000 C CNN
-F 1 "R" V 3434 3800 50  0000 C CNN
+F 1 "DNP" V 3434 3800 50  0000 C CNN
 F 2 "Resistors_SMD:R_0603" V 3480 3800 50  0001 C CNN
 F 3 "" H 3550 3800 50  0001 C CNN
@@
 P 3800 3250
 F 0 "R2" H 3730 3204 50  0000 R CNN
-F 1 "R" H 3730 3295 50  0000 R CNN
+F 1 "0R" H 3730 3295 50  0000 R CNN
 F 2 "Resistors_SMD:R_0603" V 3730 3250 50  0001 C CNN
 F 3 "" H 3800 3250 50  0001 C CNN
@@
 P 6000 4400
 F 0 "R5" H 5930 4354 50  0000 R CNN
-F 1 "R" H 5930 4445 50  0000 R CNN
+F 1 "DNP" H 5930 4445 50  0000 R CNN
 F 2 "Resistors_SMD:R_0603" V 5930 4400 50  0001 C CNN
 F 3 "" H 6000 4400 50  0001 C CNN
@@
 P 6250 3950
 F 0 "R6" V 6457 3950 50  0000 C CNN
-F 1 "R" V 6366 3950 50  0000 C CNN
+F 1 "0" V 6366 3950 50  0000 C CNN
 F 2 "Resistors_SMD:R_0603" V 6180 3950 50  0001 C CNN
 F 3 "" H 6250 3950 50  0001 C CNN
@@
 	6000 4150 6900 4150
 NoConn ~ 1700 900
+Text Notes 6100 1500 0    60   ~ 0
+13.85nF\nor 117uH\n
 $EndSCHEMATC
