File: Nestbox_v3/Nestbox_v2_RFID.sch (KiCad schematic (older format))
At the start: 8 parts, among them J701 RFID_CONN_01X05, Q701 Q_NMOS_GSD

Commit message: removed unnecessary footprints from PCB
Parts:
- removed JP701: V_RFID_Jumper_SELECT_Dual, Pin_Headers:Pin_Header_Straight_1x03_Pitch2.54mm, symbol Jumper_SELECT_Dual
Connections:
- net RFID_VDD is gone; now on net +5V: J701.1 (P1), R701.2
Other:
- note removed: "These resistors are DNP!\n"
Changed lines of the file:
@@
 Comment4 ""
 $EndDescr
-Text Label 6750 4200 2    60   ~ 0
-RFID_VDD
 $Comp
-L Jumper_SELECT_Dual JP701
-U 1 1 5A0303B0
-P 5550 2300
-F 0 "JP701" H 5550 2539 50  0000 C CNN
-F 1 "V_RFID_Jumper_SELECT_Dual" H 5550 2448 50  0000 C CNN
-F 2 "Pin_Headers:Pin_Header_Straight_1x03_Pitch2.54mm" H 5550 2300 50  0001 C CNN
-F 3 "" H 5550 2300 50  0001 C CNN
-	1    5550 2300
+L +5V #PWR064
+U 1 1 5A0305A8
+P 6750 4150
+F 0 "#PWR064" H 6750 4000 50  0001 C CNN
+F 1 "+5V" V 6765 4278 50  0000 L CNN
+F 2 "" H 6750 4150 50  0001 C CNN
+F 3 "" H 6750 4150 50  0001 C CNN
+	1    6750 4150
 	1    0    0    -1
-$EndComp
-Text Label 5550 2900 1    60   ~ 0
-RFID_VDD
-$Comp
-L +5V #PWR702
-U 1 1 5A0305A8
-P 5200 2300
-F 0 "#PWR702" H 5200 2150 50  0001 C CNN
-F 1 "+5V" V 5215 2428 50  0000 L CNN
-F 2 "" H 5200 2300 50  0001 C CNN
-F 3 "" H 5200 2300 50  0001 C CNN
-	1    5200 2300
-	0    -1   -1   0
 $EndComp
 $Comp
@@
 $EndComp
 $Comp
-L GND #PWR703
+L GND #PWR065
 U 1 1 5AF8ABAA
 P 5600 3450
-F 0 "#PWR703" H 5600 3200 50  0001 C CNN
+F 0 "#PWR065" H 5600 3200 50  0001 C CNN
 F 1 "GND" H 5605 3277 50  0000 C CNN
 F 2 "" H 5600 3450 50  0001 C CNN
@@
 $EndComp
 $Comp
-L GND #PWR704
+L GND #PWR066
 U 1 1 5AF8AC8E
 P 5600 5800
-F 0 "#PWR704" H 5600 5550 50  0001 C CNN
+F 0 "#PWR066" H 5600 5550 50  0001 C CNN
 F 1 "GND" H 5605 5627 50  0000 C CNN
 F 2 "" H 5600 5800 50  0001 C CNN
@@
 $EndComp
 $Comp
-L GND #PWR706
+L GND #PWR067
 U 1 1 5AF8B903
 P 6750 4750
-F 0 "#PWR706" H 6750 4500 50  0001 C CNN
+F 0 "#PWR067" H 6750 4500 50  0001 C CNN
 F 1 "GND" H 6755 4577 50  0000 C CNN
 F 2 "" H 6750 4750 50  0001 C CNN
@@
 Text HLabel 5450 3850 0    60   Input ~ 0
 RFID_CLOCK
-Text Notes 7150 3550 0    60   ~ 0
-These resistors are DNP!\n
-Text Label 5150 5100 3    60   ~ 0
-RFID_VDD
 $Comp
-L GND #PWR701
+L GND #PWR068
 U 1 1 5B088780
 P 4350 5000
-F 0 "#PWR701" H 4350 4750 50  0001 C CNN
+F 0 "#PWR068" H 4350 4750 50  0001 C CNN
 F 1 "GND" H 4355 4827 50  0000 C CNN
 F 2 "" H 4350 5000 50  0001 C CNN
@@
 	1    0    0    -1
 $EndComp
-$Comp
-L +BATT #PWR705
-U 1 1 5B08AE2C
-P 5950 2300
-F 0 "#PWR705" H 5950 2150 50  0001 C CNN
-F 1 "+BATT" H 5950 2440 50  0000 C CNN
-F 2 "" H 5950 2300 50  0001 C CNN
-F 3 "" H 5950 2300 50  0001 C CNN
-	1    5950 2300
-	0    1    1    0
-$EndComp
 Wire Wire Line
 	5600 5700 5600 5800
@@
 Wire Wire Line
 	6750 4200 6850 4200
-Wire Wire Line
-	5550 2400 5550 2900
 Wire Wire Line
 	5150 5100 5150 5000
@@
 Wire Wire Line
 	6750 4750 6750 4600
-Wire Wire Line
-	5800 2300 5950 2300
-Wire Wire Line
-	5200 2300 5300 2300
 Wire Wire Line
 	5450 3850 5600 3850
@@
 	1    0    0    -1
 $EndComp
+Wire Wire Line
+	6750 4150 6750 4200
+$Comp
+L +5V #PWR?
+U 1 1 5BCBE932
+P 5150 5100
+F 0 "#PWR?" H 5150 4950 50  0001 C CNN
+F 1 "+5V" V 5165 5228 50  0000 L CNN
+F 2 "" H 5150 5100 50  0001 C CNN
+F 3 "" H 5150 5100 50  0001 C CNN
+	1    5150 5100
+	-1   0    0    1
+$EndComp
 $EndSCHEMATC

Commit message: exchanged both inductor footprints.
Parts:
- Q701: value Q_NMOS_GSD -> DMG3402L
- R701: value 50k -> 82k
- R702, R703: value 18k -> 47k
- R704, R705: value 33k -> 82k
Changed lines of the file:
@@
 P 5600 4050
 F 0 "R702" H 5670 4096 50  0000 L CNN
-F 1 "18k" H 5670 4005 50  0000 L CNN
+F 1 "47k" H 5670 4005 50  0000 L CNN
 F 2 "Resistors_SMD:R_0603" V 5530 4050 50  0001 C CNN
 F 3 "" H 5600 4050 50  0001 C CNN
@@
 P 5600 4850
 F 0 "R703" H 5670 4896 50  0000 L CNN
-F 1 "18k" H 5670 4805 50  0000 L CNN
+F 1 "47k" H 5670 4805 50  0000 L CNN
 F 2 "Resistors_SMD:R_0603" V 5530 4850 50  0001 C CNN
 F 3 "" H 5600 4850 50  0001 C CNN
@@
 P 5600 3650
 F 0 "R704" H 5670 3696 50  0000 L CNN
-F 1 "33k" H 5670 3605 50  0000 L CNN
+F 1 "82k" H 5670 3605 50  0000 L CNN
 F 2 "Resistors_SMD:R_0603" V 5530 3650 50  0001 C CNN
 F 3 "" H 5600 3650 50  0001 C CNN
@@
 P 5600 5550
 F 0 "R705" H 5670 5596 50  0000 L CNN
-F 1 "33k" H 5670 5505 50  0000 L CNN
+F 1 "82k" H 5670 5505 50  0000 L CNN
 F 2 "Resistors_SMD:R_0603" V 5530 5550 50  0001 C CNN
 F 3 "" H 5600 5550 50  0001 C CNN
@@
 P 5150 4850
 F 0 "R701" H 5220 4896 50  0000 L CNN
-F 1 "50k" H 5220 4805 50  0000 L CNN
+F 1 "82k" H 5220 4805 50  0000 L CNN
 F 2 "Resistors_SMD:R_0603" V 5080 4850 50  0001 C CNN
 F 3 "" H 5150 4850 50  0001 C CNN
@@
 P 4250 4800
 F 0 "Q701" H 4450 4850 50  0000 L CNN
-F 1 "Q_NMOS_GSD" H 4450 4750 50  0000 L CNN
+F 1 "DMG3402L" H 4450 4750 50  0000 L CNN
 F 2 "TO_SOT_Packages_SMD:TSOT-23" H 4450 4900 50  0001 C CNN
 F 3 "" H 4250 4800 50  0001 C CNN

Commit message: added MPN for all components for PCBA
Parts:
- Q701: MPN (none) -> DMG3402L-7
- R701, R704, R705: MPN (none) -> RC0603FR-0782KL
- R702, R703: MPN (none) -> RC0603FR-0747KL
Changed lines of the file:
@@
-EESchema Schematic File Version 2
+EESchema Schematic File Version 4
 LIBS:power
 LIBS:device
@@
 LIBS:contrib
 LIBS:valves
-LIBS:Octanis3
 LIBS:Nestbox_v2-cache
-EELAYER 25 0
+EELAYER 26 0
 EELAYER END
 $Descr A4 11693 8268
@@
 F 2 "Resistors_SMD:R_0603" V 5530 4050 50  0001 C CNN
 F 3 "" H 5600 4050 50  0001 C CNN
+F 4 "RC0603FR-0747KL" H 0   0   50  0001 C CNN "MPN"
 	1    5600 4050
 	1    0    0    -1
@@
 F 2 "Resistors_SMD:R_0603" V 5530 4850 50  0001 C CNN
 F 3 "" H 5600 4850 50  0001 C CNN
+F 4 "RC0603FR-0747KL" H 0   0   50  0001 C CNN "MPN"
 	1    5600 4850
 	1    0    0    -1
@@
 F 2 "Resistors_SMD:R_0603" V 5530 3650 50  0001 C CNN
 F 3 "" H 5600 3650 50  0001 C CNN
+F 4 "RC0603FR-0782KL" H 0   0   50  0001 C CNN "MPN"
 	1    5600 3650
 	1    0    0    -1
@@
 F 2 "Resistors_SMD:R_0603" V 5530 5550 50  0001 C CNN
 F 3 "" H 5600 5550 50  0001 C CNN
+F 4 "RC0603FR-0782KL" H 0   0   50  0001 C CNN "MPN"
 	1    5600 5550
 	1    0    0    -1
@@
 F 2 "Resistors_SMD:R_0603" V 5080 4850 50  0001 C CNN
 F 3 "" H 5150 4850 50  0001 C CNN
+F 4 "RC0603FR-0782KL" H 0   0   50  0001 C CNN "MPN"
 	1    5150 4850
 	1    0    0    -1
@@
 F 2 "TO_SOT_Packages_SMD:TSOT-23" H 4450 4900 50  0001 C CNN
 F 3 "" H 4250 4800 50  0001 C CNN
+F 4 "DMG3402L-7" H 0   0   50  0001 C CNN "MPN"
 	1    4250 4800
 	1    0    0    -1
