File: Nestbox_v3/Nestbox_v2_control.sch (KiCad schematic (older format))
At the start: 26 parts, among them P301 RX/TX, P302 TST/RST, P303 DEBUG_3V3, Q301 NTR3A052PZT1G, SW301 SMD-BUTTON_2P-3.0X2.5X1.2+0.4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, U301 MSP430FR5969, Y301 Crystal

Commit message: removed unnecessary footprints from PCB
Parts:
- J301: renamed from J?; footprint (none) -> Pin_Headers:Pin_Header_Straight_1x04
Connections:
- net LB1_LED renamed RTC_CAL
Changed lines of the file:
@@
 $EndComp
 $Comp
-L GND #PWR314
+L GND #PWR025
 U 1 1 586416A7
 P 6150 3750
-F 0 "#PWR314" H 6150 3500 50  0001 C CNN
+F 0 "#PWR025" H 6150 3500 50  0001 C CNN
 F 1 "GND" H 6150 3600 50  0000 C CNN
 F 2 "" H 6150 3750 50  0000 C CNN
@@
 $EndComp
 $Comp
-L +3.3V #PWR308
+L +3.3V #PWR026
 U 1 1 586418DC
 P 4300 1900
-F 0 "#PWR308" H 4300 1750 50  0001 C CNN
+F 0 "#PWR026" H 4300 1750 50  0001 C CNN
 F 1 "+3.3V" H 4300 2040 50  0000 C CNN
 F 2 "" H 4300 1900 50  0000 C CNN
@@
 $EndComp
 $Comp
-L GND #PWR302
+L GND #PWR027
 U 1 1 58641ADD
 P 2500 2250
-F 0 "#PWR302" H 2500 2000 50  0001 C CNN
+F 0 "#PWR027" H 2500 2000 50  0001 C CNN
 F 1 "GND" H 2500 2100 50  0000 C CNN
 F 2 "" H 2500 2250 50  0000 C CNN
@@
 $EndComp
 $Comp
-L +3.3V #PWR303
+L +3.3V #PWR028
 U 1 1 58641B00
 P 2850 1700
-F 0 "#PWR303" H 2850 1550 50  0001 C CNN
+F 0 "#PWR028" H 2850 1550 50  0001 C CNN
 F 1 "+3.3V" H 2850 1840 50  0000 C CNN
 F 2 "" H 2850 1700 50  0000 C CNN
@@
 $EndComp
 $Comp
-L GND #PWR309
+L GND #PWR029
 U 1 1 58652F3A
 P 4700 2450
-F 0 "#PWR309" H 4700 2200 50  0001 C CNN
+F 0 "#PWR029" H 4700 2200 50  0001 C CNN
 F 1 "GND" H 4700 2300 50  0000 C CNN
 F 2 "" H 4700 2450 50  0000 C CNN
@@
 $EndComp
 $Comp
-L GND #PWR305
+L GND #PWR030
 U 1 1 5865358A
 P 3400 1600
-F 0 "#PWR305" H 3400 1350 50  0001 C CNN
+F 0 "#PWR030" H 3400 1350 50  0001 C CNN
 F 1 "GND" H 3400 1450 50  0000 C CNN
 F 2 "" H 3400 1600 50  0000 C CNN
@@
 $EndComp
 $Comp
-L GND #PWR320
+L GND #PWR031
 U 1 1 587B96DD
 P 10000 5300
-F 0 "#PWR320" H 10000 5050 50  0001 C CNN
+F 0 "#PWR031" H 10000 5050 50  0001 C CNN
 F 1 "GND" H 10000 5150 50  0000 C CNN
 F 2 "" H 10000 5300 50  0000 C CNN
@@
 $EndComp
 $Comp
-L +3.3V #PWR319
+L +3.3V #PWR032
 U 1 1 587B9736
 P 10000 4100
-F 0 "#PWR319" H 10000 3950 50  0001 C CNN
+F 0 "#PWR032" H 10000 3950 50  0001 C CNN
 F 1 "+3.3V" H 10000 4240 50  0000 C CNN
 F 2 "" H 10000 4100 50  0000 C CNN
@@
 $EndComp
 $Comp
-L GND #PWR318
+L GND #PWR033
 U 1 1 587B97E4
 P 9600 5400
-F 0 "#PWR318" H 9600 5150 50  0001 C CNN
+F 0 "#PWR033" H 9600 5150 50  0001 C CNN
 F 1 "GND" H 9600 5250 50  0000 C CNN
 F 2 "" H 9600 5400 50  0000 C CNN
@@
 $EndComp
 $Comp
-L GND #PWR317
+L GND #PWR034
 U 1 1 587B9834
 P 9300 5400
-F 0 "#PWR317" H 9300 5150 50  0001 C CNN
+F 0 "#PWR034" H 9300 5150 50  0001 C CNN
 F 1 "GND" H 9300 5250 50  0000 C CNN
 F 2 "" H 9300 5400 50  0000 C CNN
@@
 AVCC
 Wire Wire Line
-	4300 1900 4300 2000
-Wire Wire Line
-	4300 2000 4300 2400
-Wire Wire Line
-	4300 2400 4300 2450
+	4300 1900 4300 2450
 Connection ~ 4300 2400
 Connection ~ 4300 2000
@@
 	2850 2450 3200 2450
 Wire Wire Line
-	2850 2200 2850 2250
-Wire Wire Line
-	2850 2250 2850 2450
+	2850 2200 2850 2450
 Wire Wire Line
 	2800 2250 2850 2250
@@
 	3400 1600 3400 1650
 Wire Wire Line
-	3200 1650 3400 1650
-Wire Wire Line
-	3400 1650 3650 1650
+	3200 1650 3650 1650
 Connection ~ 3400 1650
 Wire Wire Line
@@
 	4200 6450 4200 6600
 Wire Wire Line
-	4200 6600 4450 6600
-Wire Wire Line
-	4450 6600 4500 6600
+	4200 6600 4500 6600
 Wire Wire Line
 	4450 6600 4450 6700
 Wire Wire Line
-	10000 4500 10000 4550
-Wire Wire Line
-	10000 4550 10000 4600
+	10000 4500 10000 4600
 Wire Wire Line
 	3700 6450 3700 7000
@@
 	9300 4950 9300 5050
 $Comp
-L GND #PWR301
+L GND #PWR035
 U 1 1 587D2523
 P 2450 2450
-F 0 "#PWR301" H 2450 2200 50  0001 C CNN
+F 0 "#PWR035" H 2450 2200 50  0001 C CNN
 F 1 "GND" H 2450 2300 50  0000 C CNN
 F 2 "" H 2450 2450 50  0000 C CNN
@@
 	4350 6650 4350 6700
 $Comp
-L +3.3V #PWR310
+L +3.3V #PWR036
 U 1 1 58BC4BB7
 P 4850 6600
-F 0 "#PWR310" H 4850 6450 50  0001 C CNN
+F 0 "#PWR036" H 4850 6450 50  0001 C CNN
 F 1 "+3.3V" H 4850 6740 50  0000 C CNN
 F 2 "" H 4850 6600 50  0000 C CNN
@@
 	10200 4850 10200 4900
 $Comp
-L GND #PWR321
+L GND #PWR037
 U 1 1 58BF19D6
 P 10200 5300
-F 0 "#PWR321" H 10200 5050 50  0001 C CNN
+F 0 "#PWR037" H 10200 5050 50  0001 C CNN
 F 1 "GND" H 10200 5150 50  0000 C CNN
 F 2 "" H 10200 5300 50  0000 C CNN
@@
 	6150 4050 6700 4050
 Wire Wire Line
-	1300 3750 1450 3750
-Wire Wire Line
-	1450 3750 1550 3750
-Wire Wire Line
 	1550 3850 1300 3850
 Wire Wire Line
@@
 	6150 4550 6700 4550
 $Comp
-L GND #PWR316
+L GND #PWR038
 U 1 1 59FCED84
 P 7550 1600
-F 0 "#PWR316" H 7550 1350 50  0001 C CNN
+F 0 "#PWR038" H 7550 1350 50  0001 C CNN
 F 1 "GND" H 7550 1450 50  0000 C CNN
 F 2 "" H 7550 1600 50  0000 C CNN
@@
 DBG_Switch
 Wire Wire Line
-	10000 4550 10200 4550
-Wire Wire Line
-	10200 4550 10850 4550
+	10000 4550 10850 4550
 Connection ~ 10000 4550
 Text Label 10850 4550 2    60   ~ 0
@@
 	4650 2000 4700 2000
 Wire Wire Line
-	4700 2000 4700 2400
-Wire Wire Line
-	4700 2400 4700 2450
+	4700 2000 4700 2450
 Wire Wire Line
 	4650 2400 4700 2400
@@
 Connection ~ 3900 7350
 Wire Wire Line
-	4000 6450 4000 7350
-Wire Wire Line
-	4000 7350 4000 7400
-Wire Wire Line
-	3900 6450 3900 7350
-Wire Wire Line
-	3900 7350 3900 7400
+	4000 6450 4000 7400
+Wire Wire Line
+	3900 6450 3900 7400
 Text HLabel 6700 4150 2    60   Input ~ 0
 SPI_MISO
@@
 Text HLabel 1500 4650 0    60   Input ~ 0
 LB_EXTERNAL_DETECT
-Text HLabel 1300 3750 0    60   Output ~ 0
-LB1_LED
 Text HLabel 1300 3850 0    60   Output ~ 0
 PIR_EN
@@
 $EndComp
 $Comp
-L +3.3V #PWR312
+L +3.3V #PWR039
 U 1 1 5B0C49AB
 P 5900 7400
-F 0 "#PWR312" H 5900 7250 50  0001 C CNN
+F 0 "#PWR039" H 5900 7250 50  0001 C CNN
 F 1 "+3.3V" H 5900 7540 50  0000 C CNN
 F 2 "" H 5900 7400 50  0000 C CNN
@@
 $EndComp
 $Comp
-L GND #PWR311
+L GND #PWR040
 U 1 1 5B0C4B76
 P 5800 7400
-F 0 "#PWR311" H 5800 7150 50  0001 C CNN
+F 0 "#PWR040" H 5800 7150 50  0001 C CNN
 F 1 "GND" H 5800 7250 50  0000 C CNN
 F 2 "" H 5800 7400 50  0000 C CNN
@@
 SD_CARD_ENABLE
 $Comp
-L GND #PWR304
+L GND #PWR041
 U 1 1 5B187286
 P 3300 2400
-F 0 "#PWR304" H 3300 2150 50  0001 C CNN
+F 0 "#PWR041" H 3300 2150 50  0001 C CNN
 F 1 "GND" H 3300 2250 50  0000 C CNN
 F 2 "" H 3300 2400 50  0000 C CNN
@@
 $EndComp
 $Comp
-L GND #PWR306
+L GND #PWR042
 U 1 1 5B1872E2
 P 3600 2400
-F 0 "#PWR306" H 3600 2150 50  0001 C CNN
+F 0 "#PWR042" H 3600 2150 50  0001 C CNN
 F 1 "GND" H 3600 2250 50  0000 C CNN
 F 2 "" H 3600 2400 50  0000 C CNN
@@
 $EndComp
 $Comp
-L GND #PWR307
+L GND #PWR043
 U 1 1 5B18733E
 P 3900 2400
-F 0 "#PWR307" H 3900 2150 50  0001 C CNN
+F 0 "#PWR043" H 3900 2150 50  0001 C CNN
 F 1 "GND" H 3900 2250 50  0000 C CNN
 F 2 "" H 3900 2400 50  0000 C CNN
@@
 $EndComp
 $Comp
-L +3.3V #PWR313
+L +3.3V #PWR044
 U 1 1 5B28B3EE
 P 8400 900
-F 0 "#PWR313" H 8400 750 50  0001 C CNN
+F 0 "#PWR044" H 8400 750 50  0001 C CNN
 F 1 "+3.3V" H 8415 1073 50  0000 C CNN
 F 2 "" H 8400 900 50  0000 C CNN
@@
 NoConn ~ 1550 4350
 $Comp
-L CONN_01X04 J?
+L CONN_01X04 J301
 U 1 1 5BCBB74D
 P 10850 1450
-F 0 "J?" H 10850 1700 50  0000 C CNN
+F 0 "J301" H 10850 1700 50  0000 C CNN
 F 1 "CONN_01X04" V 10950 1450 50  0000 C CNN
-F 2 "" H 10850 1450 50  0001 C CNN
+F 2 "Pin_Headers:Pin_Header_Straight_1x04" H 10850 1450 50  0001 C CNN
 F 3 "" H 10850 1450 50  0001 C CNN
 	1    10850 1450
@@
 	8400 1300 9350 1300
 Wire Wire Line
-	8400 900  8400 950
-Wire Wire Line
-	8400 950  8400 1000
-Wire Wire Line
-	7550 1600 7650 1600
-Wire Wire Line
-	7650 1600 8050 1600
-Wire Wire Line
-	8050 1600 10650 1600
+	8400 900  8400 1000
+Wire Wire Line
+	7550 1600 10650 1600
 Wire Wire Line
 	8050 1400 8050 1600
@@
 Connection ~ 7650 1600
 Wire Wire Line
-	7650 950  8050 950
-Wire Wire Line
-	8050 950  8400 950
-Wire Wire Line
-	8400 950  9650 950
+	7650 950  9650 950
 Connection ~ 8400 950
 Wire Wire Line
@@
 Wire Wire Line
 	6150 4750 6700 4750
+Wire Wire Line
+	1450 3750 1550 3750
+Text Label 1450 3650 0    60   ~ 0
+RTC_CAL
 $EndSCHEMATC

Commit message: finished V3 pcb. ORDERED
Parts:
- added R303, R304: 0R, Resistors_SMD:R_0603, symbol R
Connections:
- net +3V3: no longer C307.1
- net RX: now also R304.1; no longer J301.2 (P2)
- net TX: now also R303.1; no longer J301.1 (P1)
- net at J301.3 (P3), Q301.3 (D): now also C307.1
- new net: J301.1 (P1), R303.2
- new net: J301.2 (P2), R304.2
Other:
- moved on the sheet: C307, J301
Changed lines of the file:
@@
 L C C307
 U 1 1 59FF0C21
-P 8050 1250
-F 0 "C307" H 8165 1296 50  0000 L CNN
-F 1 "0.1u" H 8165 1205 50  0000 L CNN
-F 2 "Capacitors_SMD:C_0603" H 8088 1100 50  0001 C CNN
-F 3 "" H 8050 1250 50  0000 C CNN
-	1    8050 1250
+P 9500 1650
+F 0 "C307" H 9615 1696 50  0000 L CNN
+F 1 "0.1u" H 9615 1605 50  0000 L CNN
+F 2 "Capacitors_SMD:C_0603" H 9538 1500 50  0001 C CNN
+F 3 "" H 9500 1650 50  0000 C CNN
+	1    9500 1650
 	1    0    0    -1
 $EndComp
@@
 L CONN_01X04 J301
 U 1 1 5BCBB74D
-P 10850 1450
-F 0 "J301" H 10850 1700 50  0000 C CNN
-F 1 "CONN_01X04" V 10950 1450 50  0000 C CNN
-F 2 "Pin_Headers:Pin_Header_Straight_1x04" H 10850 1450 50  0001 C CNN
-F 3 "" H 10850 1450 50  0001 C CNN
-	1    10850 1450
+P 11250 1450
+F 0 "J301" H 11250 1700 50  0000 C CNN
+F 1 "CONN_01X04" V 11350 1450 50  0000 C CNN
+F 2 "Pin_Headers:Pin_Header_Straight_1x04" H 11250 1450 50  0001 C CNN
+F 3 "" H 11250 1450 50  0001 C CNN
+	1    11250 1450
 	1    0    0    -1
 $EndComp
@@
 RX
 Wire Wire Line
-	9650 1500 10650 1500
-Wire Wire Line
-	10650 1400 10500 1400
-Wire Wire Line
-	10650 1300 10500 1300
-Text Label 10500 1300 0    60   ~ 0
+	9500 1500 11050 1500
+Text Label 10450 1300 0    60   ~ 0
 TX
-Text Label 10500 1400 0    60   ~ 0
+Text Label 10450 1400 0    60   ~ 0
 RX
 Wire Wire Line
@@
 	8400 900  8400 1000
 Wire Wire Line
-	7550 1600 10650 1600
-Wire Wire Line
-	8050 1400 8050 1600
+	7550 1600 9100 1600
 Connection ~ 8050 1600
 Wire Wire Line
@@
 	7650 950  9650 950
 Connection ~ 8400 950
-Wire Wire Line
-	8050 950  8050 1100
 Connection ~ 8050 950
 Wire Wire Line
@@
 Text Label 1450 3650 0    60   ~ 0
 RTC_CAL
+$Comp
+L R R303
+U 1 1 5BCD0C24
+P 10800 1300
+F 0 "R303" V 10750 1100 50  0000 L CNN
+F 1 "0R" V 10800 1250 50  0000 L CNN
+F 2 "Resistors_SMD:R_0603" V 10730 1300 50  0001 C CNN
+F 3 "" H 10800 1300 50  0000 C CNN
+	1    10800 1300
+	0    -1   -1   0
+$EndComp
+Wire Wire Line
+	10950 1300 11050 1300
+Wire Wire Line
+	10650 1300 10450 1300
+$Comp
+L R R304
+U 1 1 5BCD0ECB
+P 10800 1400
+F 0 "R304" V 10750 1200 50  0000 L CNN
+F 1 "0R" V 10800 1350 50  0000 L CNN
+F 2 "Resistors_SMD:R_0603" V 10730 1400 50  0001 C CNN
+F 3 "" H 10800 1400 50  0000 C CNN
+	1    10800 1400
+	0    -1   -1   0
+$EndComp
+Wire Wire Line
+	10950 1400 11050 1400
+Wire Wire Line
+	10650 1400 10450 1400
+Wire Wire Line
+	11050 1600 9650 1600
+Wire Wire Line
+	9650 1900 9650 1600
+Wire Wire Line
+	9100 1900 9650 1900
+Wire Wire Line
+	9500 1900 9500 1800
+Connection ~ 9650 1500
+Wire Wire Line
+	9100 1600 9100 1900
+Connection ~ 9500 1900
 $EndSCHEMATC

Commit message: exchanged both inductor footprints.
Parts:
- C302, C303: value 25 pF -> 24p; MPN CC0603JRNPO9BN120 -> (none); SKU 302010067 -> (none)
- C307: value 0.1u -> 100n
- R301: value 47K -> 47k; MPN FHCFR-1_4W-473J -> (none)
- R306, R307: value 1K -> 1k
- R308, R309: value 10K -> 10k
Changed lines of the file:
@@
 P 3650 1800
 F 0 "C303" H 3500 1850 45  0000 L BNN
-F 1 "25 pF" H 3500 1700 45  0000 L BNN
+F 1 "24p" H 3500 1700 45  0000 L BNN
 F 2 "Capacitors_SMD:C_0603" H 3650 1800 60  0001 C CNN
 F 3 "" H 3650 1800 60  0001 C CNN
-F 4 "CC0603JRNPO9BN120" H 3680 1950 20  0001 C CNN "MPN"
-F 5 "302010067" H 3680 1950 20  0001 C CNN "SKU"
-F 6 "" H 3680 1950 20  0001 C CNN "Field6"
 	1    3650 1800
 	0    -1   -1   0
@@
 P 3200 1800
 F 0 "C302" H 3050 1850 45  0000 L BNN
-F 1 "25 pF" H 3050 1700 45  0000 L BNN
+F 1 "24p" H 3050 1700 45  0000 L BNN
 F 2 "Capacitors_SMD:C_0603" H 3200 1800 60  0001 C CNN
 F 3 "" H 3200 1800 60  0001 C CNN
-F 4 "CC0603JRNPO9BN120" H 3230 1950 20  0001 C CNN "MPN"
-F 5 "302010067" H 3230 1950 20  0001 C CNN "SKU"
-F 6 "" H 3230 1950 20  0001 C CNN "Field6"
 	1    3200 1800
 	0    -1   -1   0
@@
 P 4650 6600
 F 0 "R301" H 4500 6650 45  0000 L BNN
-F 1 "47K" H 4500 6500 45  0000 L BNN
+F 1 "47k" H 4500 6500 45  0000 L BNN
 F 2 "Resistors_SMD:R_0603" H 4650 6600 40  0001 C CNN
 F 3 "" H 4650 6600 40  0001 C CNN
-F 4 "FHCFR-1_4W-473J" H 4680 6750 20  0001 C CNN "MPN"
-F 5 "" H 4680 6750 20  0001 C CNN "Field5"
-F 6 "" H 4680 6750 20  0001 C CNN "Field6"
 	1    4650 6600
 	1    0    0    -1
@@
 P 9500 1650
 F 0 "C307" H 9615 1696 50  0000 L CNN
-F 1 "0.1u" H 9615 1605 50  0000 L CNN
+F 1 "100n" H 9615 1605 50  0000 L CNN
 F 2 "Capacitors_SMD:C_0603" H 9538 1500 50  0001 C CNN
 F 3 "" H 9500 1650 50  0000 C CNN
@@
 P 9300 5200
 F 0 "R306" H 9370 5246 50  0000 L CNN
-F 1 "1K" H 9370 5155 50  0000 L CNN
+F 1 "1k" H 9370 5155 50  0000 L CNN
 F 2 "Resistors_SMD:R_0603" V 9230 5200 50  0001 C CNN
 F 3 "" H 9300 5200 50  0000 C CNN
@@
 P 9600 5200
 F 0 "R307" H 9670 5246 50  0000 L CNN
-F 1 "1K" H 9670 5155 50  0000 L CNN
+F 1 "1k" H 9670 5155 50  0000 L CNN
 F 2 "Resistors_SMD:R_0603" V 9530 5200 50  0001 C CNN
 F 3 "" H 9600 5200 50  0000 C CNN
@@
 P 10200 4700
 F 0 "R309" H 10270 4746 50  0000 L CNN
-F 1 "10K" H 10270 4655 50  0000 L CNN
+F 1 "10k" H 10270 4655 50  0000 L CNN
 F 2 "Resistors_SMD:R_0603" V 10130 4700 50  0001 C CNN
 F 3 "" H 10200 4700 50  0000 C CNN
@@
 P 10000 4350
 F 0 "R308" H 10070 4396 50  0000 L CNN
-F 1 "10K" H 10070 4305 50  0000 L CNN
+F 1 "10k" H 10070 4305 50  0000 L CNN
 F 2 "Resistors_SMD:R_0603" V 9930 4350 50  0001 C CNN
 F 3 "" H 10000 4350 50  0000 C CNN
@@
 	11050 1600 9650 1600
 Wire Wire Line
-	9650 1900 9650 1600
-Wire Wire Line
-	9100 1900 9650 1900
+	9650 1600 9650 1900
+Wire Wire Line
+	9650 1900 9100 1900
 Wire Wire Line
 	9500 1900 9500 1800
 Connection ~ 9650 1500
 Wire Wire Line
-	9100 1600 9100 1900
+	9100 1900 9100 1600
 Connection ~ 9500 1900
 $EndSCHEMATC

Commit message: added MPN for all components for PCBA
Parts:
- C301, C305, C307, C308: MPN (none) -> CC0603KRX7R9BB104
- C302, C303: MPN (none) -> CC0603JRNPO9BN240
- C304: MPN (none) -> CC0805KKX5R8BB106
- Q301: MPN (none) -> NTR3A052PZT1G
- R301: MPN (none) -> RC0603FR-0747KL
- R302: MPN (none) -> RC0603FR-0782KL
- R303, R304: MPN (none) -> RC0603JR-070RL
- R306, R307: MPN (none) -> RC0603FR-071KL
- R308, R309: MPN (none) -> RC0603JR-0710KL
Changed lines of the file:
@@
-EESchema Schematic File Version 2
+EESchema Schematic File Version 4
 LIBS:power
 LIBS:device
@@
 LIBS:contrib
 LIBS:valves
-LIBS:Octanis3
 LIBS:Nestbox_v2-cache
-EELAYER 25 0
+EELAYER 26 0
 EELAYER END
 $Descr A4 11693 8268
@@
 F 2 "Capacitors_SMD:C_0603" H 3650 1800 60  0001 C CNN
 F 3 "" H 3650 1800 60  0001 C CNN
+F 4 "CC0603JRNPO9BN240" H 0   0   50  0001 C CNN "MPN"
 	1    3650 1800
 	0    -1   -1   0
@@
 F 2 "Capacitors_SMD:C_0603" H 3200 1800 60  0001 C CNN
 F 3 "" H 3200 1800 60  0001 C CNN
+F 4 "CC0603JRNPO9BN240" H 0   0   50  0001 C CNN "MPN"
 	1    3200 1800
 	0    -1   -1   0
@@
 F 2 "Resistors_SMD:R_0603" H 4650 6600 40  0001 C CNN
 F 3 "" H 4650 6600 40  0001 C CNN
+F 4 "RC0603FR-0747KL" H 0   0   50  0001 C CNN "MPN"
 	1    4650 6600
 	1    0    0    -1
@@
 F 2 "Capacitors_SMD:C_0603" H 9538 1500 50  0001 C CNN
 F 3 "" H 9500 1650 50  0000 C CNN
+F 4 "CC0603KRX7R9BB104" H 0   0   50  0001 C CNN "MPN"
 	1    9500 1650
 	1    0    0    -1
@@
 F 2 "Resistors_SMD:R_0603" V 9230 5200 50  0001 C CNN
 F 3 "" H 9300 5200 50  0000 C CNN
+F 4 "RC0603FR-071KL" H 0   0   50  0001 C CNN "MPN"
 	1    9300 5200
 	1    0    0    -1
@@
 F 2 "Resistors_SMD:R_0603" V 9530 5200 50  0001 C CNN
 F 3 "" H 9600 5200 50  0000 C CNN
+F 4 "RC0603FR-071KL" H 0   0   50  0001 C CNN "MPN"
 	1    9600 5200
 	1    0    0    -1
@@
 F 2 "Resistors_SMD:R_0603" V 10130 4700 50  0001 C CNN
 F 3 "" H 10200 4700 50  0000 C CNN
+F 4 "RC0603JR-0710KL" H 0   0   50  0001 C CNN "MPN"
 	1    10200 4700
 	1    0    0    -1
@@
 F 2 "Resistors_SMD:R_0603" V 9930 4350 50  0001 C CNN
 F 3 "" H 10000 4350 50  0000 C CNN
+F 4 "RC0603JR-0710KL" H 0   0   50  0001 C CNN "MPN"
 	1    10000 4350
 	1    0    0    -1
@@
 F 2 "Capacitors_SMD:C_0603" H 10238 4900 50  0001 C CNN
 F 3 "" H 10200 5050 50  0000 C CNN
+F 4 "CC0603KRX7R9BB104" H 0   0   50  0001 C CNN "MPN"
 	1    10200 5050
 	1    0    0    -1
@@
 F 2 "Capacitors_SMD:C_0805" H 4538 1850 50  0001 C CNN
 F 3 "" H 4500 2000 50  0000 C CNN
+F 4 "CC0805KKX5R8BB106" H 0   0   50  0001 C CNN "MPN"
 	1    4500 2000
 	0    1    1    0
@@
 F 2 "Capacitors_SMD:C_0603" H 4538 2250 50  0001 C CNN
 F 3 "" H 4500 2400 50  0000 C CNN
+F 4 "CC0603KRX7R9BB104" H 0   0   50  0001 C CNN "MPN"
 	1    4500 2400
 	0    1    1    0
@@
 F 2 "Capacitors_SMD:C_0603" H 2688 2100 50  0001 C CNN
 F 3 "" H 2650 2250 50  0000 C CNN
+F 4 "CC0603KRX7R9BB104" H 0   0   50  0001 C CNN "MPN"
 	1    2650 2250
 	0    1    1    0
@@
 F 2 "TO_SOT_Packages_SMD:TSOT-23" H 9750 1400 50  0001 C CNN
 F 3 "" H 9550 1300 50  0001 C CNN
+F 4 "NTR3A052PZT1G" H 0   0   50  0001 C CNN "MPN"
 	1    9550 1300
 	1    0    0    1
@@
 F 2 "Resistors_SMD:R_0603" V 8330 1150 50  0001 C CNN
 F 3 "" H 8400 1150 50  0000 C CNN
+F 4 "RC0603FR-0782KL" H 0   0   50  0001 C CNN "MPN"
 	1    8400 1150
 	1    0    0    -1
@@
 F 2 "Resistors_SMD:R_0603" V 10730 1300 50  0001 C CNN
 F 3 "" H 10800 1300 50  0000 C CNN
+F 4 "RC0603JR-070RL	" H 0   0   50  0001 C CNN "MPN"
 	1    10800 1300
 	0    -1   -1   0
@@
 F 2 "Resistors_SMD:R_0603" V 10730 1400 50  0001 C CNN
 F 3 "" H 10800 1400 50  0000 C CNN
+F 4 "RC0603JR-070RL	" H 0   0   50  0001 C CNN "MPN"
 	1    10800 1400
 	0    -1   -1   0

Commit message: reworked silk layer for PCBA. generated position files. reviewed parts MPN for final order
Parts:
- C302, C303: value 24p -> 25p; MPN CC0603JRNPO9BN240 -> CC0603JRNPO9BN250; MouserLink (none) -> https://www.mouser.ch/ProductDetail/Yageo/CC0603JRNPO9BN250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
- L301: MPN (none) -> BLM18AG121SN1D; SKU 303030020 -> (none)
Changed lines of the file:
@@
-EESchema Schematic File Version 4
+EESchema Schematic File Version 2
 LIBS:power
 LIBS:device
@@
 LIBS:contrib
 LIBS:valves
+LIBS:Octanis3
 LIBS:Nestbox_v2-cache
-EELAYER 26 0
+EELAYER 25 0
 EELAYER END
 $Descr A4 11693 8268
@@
 F 2 "SeeedOPL-Inductor-2016:L0603" H 2850 2000 60  0001 C CNN
 F 3 "" H 2850 2000 60  0001 C CNN
-F 4 "303030020" H 2880 2150 20  0001 C CNN "SKU"
-F 5 "" H 2880 2150 20  0001 C CNN "Field6"
+F 4 "BLM18AG121SN1D" H 2880 2150 20  0001 C CNN "MPN"
 	1    2850 2000
 	0    -1   -1   0
@@
 P 3650 1800
 F 0 "C303" H 3500 1850 45  0000 L BNN
-F 1 "24p" H 3500 1700 45  0000 L BNN
+F 1 "25p" H 3500 1700 45  0000 L BNN
 F 2 "Capacitors_SMD:C_0603" H 3650 1800 60  0001 C CNN
 F 3 "" H 3650 1800 60  0001 C CNN
-F 4 "CC0603JRNPO9BN240" H 0   0   50  0001 C CNN "MPN"
+F 4 "CC0603JRNPO9BN250" H 0   0   50  0001 C CNN "MPN"
+F 5 "https://www.mouser.ch/ProductDetail/Yageo/CC0603JRNPO9BN250?qs=%2fha2pyFaduiZbois2HzNxX5Fn2jxNU0T9riId%252bCiJb5t99D1z%252b76Cw%3d%3d" H 3650 1800 60  0001 C CNN "MouserLink"
 	1    3650 1800
 	0    -1   -1   0
@@
 P 3200 1800
 F 0 "C302" H 3050 1850 45  0000 L BNN
-F 1 "24p" H 3050 1700 45  0000 L BNN
+F 1 "25p" H 3050 1700 45  0000 L BNN
 F 2 "Capacitors_SMD:C_0603" H 3200 1800 60  0001 C CNN
 F 3 "" H 3200 1800 60  0001 C CNN
-F 4 "CC0603JRNPO9BN240" H 0   0   50  0001 C CNN "MPN"
+F 4 "CC0603JRNPO9BN250" H 0   0   50  0001 C CNN "MPN"
+F 5 "https://www.mouser.ch/ProductDetail/Yageo/CC0603JRNPO9BN250?qs=%2fha2pyFaduiZbois2HzNxX5Fn2jxNU0T9riId%252bCiJb5t99D1z%252b76Cw%3d%3d" H 3200 1800 60  0001 C CNN "MouserLink"
 	1    3200 1800
 	0    -1   -1   0
