File: Nestbox_v3/Nestbox_v2_control.sch (KiCad schematic (older format))
At the start: 28 parts, among them J301 CONN_01X04, P301 RX/TX, P302 TST/RST, P303 DEBUG_3V3, Q301 NTR3A052PZT1G, SW301 SMD-BUTTON_2P-3.0X2.5X1.2+0.4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, U301 MSP430FR5969, Y301 Crystal

Commit message: production status nestbox v3
Connections:
- net RTC_CAL renamed ESP_VCC_sense
Changed lines of the file:
@@
 $EndComp
 $Comp
-L GND #PWR025
+L GND #PWR030
 U 1 1 586416A7
 P 6150 3750
-F 0 "#PWR025" H 6150 3500 50  0001 C CNN
+F 0 "#PWR030" H 6150 3500 50  0001 C CNN
 F 1 "GND" H 6150 3600 50  0000 C CNN
 F 2 "" H 6150 3750 50  0000 C CNN
@@
 $EndComp
 $Comp
-L +3.3V #PWR026
+L +3.3V #PWR031
 U 1 1 586418DC
 P 4300 1900
-F 0 "#PWR026" H 4300 1750 50  0001 C CNN
+F 0 "#PWR031" H 4300 1750 50  0001 C CNN
 F 1 "+3.3V" H 4300 2040 50  0000 C CNN
 F 2 "" H 4300 1900 50  0000 C CNN
@@
 $EndComp
 $Comp
-L GND #PWR027
+L GND #PWR032
 U 1 1 58641ADD
 P 2500 2250
-F 0 "#PWR027" H 2500 2000 50  0001 C CNN
+F 0 "#PWR032" H 2500 2000 50  0001 C CNN
 F 1 "GND" H 2500 2100 50  0000 C CNN
 F 2 "" H 2500 2250 50  0000 C CNN
@@
 $EndComp
 $Comp
-L +3.3V #PWR028
+L +3.3V #PWR033
 U 1 1 58641B00
 P 2850 1700
-F 0 "#PWR028" H 2850 1550 50  0001 C CNN
+F 0 "#PWR033" H 2850 1550 50  0001 C CNN
 F 1 "+3.3V" H 2850 1840 50  0000 C CNN
 F 2 "" H 2850 1700 50  0000 C CNN
@@
 $EndComp
 $Comp
-L GND #PWR029
+L GND #PWR034
 U 1 1 58652F3A
 P 4700 2450
-F 0 "#PWR029" H 4700 2200 50  0001 C CNN
+F 0 "#PWR034" H 4700 2200 50  0001 C CNN
 F 1 "GND" H 4700 2300 50  0000 C CNN
 F 2 "" H 4700 2450 50  0000 C CNN
@@
 $EndComp
 $Comp
-L GND #PWR030
+L GND #PWR035
 U 1 1 5865358A
 P 3400 1600
-F 0 "#PWR030" H 3400 1350 50  0001 C CNN
+F 0 "#PWR035" H 3400 1350 50  0001 C CNN
 F 1 "GND" H 3400 1450 50  0000 C CNN
 F 2 "" H 3400 1600 50  0000 C CNN
@@
 $EndComp
 $Comp
-L GND #PWR031
+L GND #PWR036
 U 1 1 587B96DD
 P 10000 5300
-F 0 "#PWR031" H 10000 5050 50  0001 C CNN
+F 0 "#PWR036" H 10000 5050 50  0001 C CNN
 F 1 "GND" H 10000 5150 50  0000 C CNN
 F 2 "" H 10000 5300 50  0000 C CNN
@@
 $EndComp
 $Comp
-L +3.3V #PWR032
+L +3.3V #PWR037
 U 1 1 587B9736
 P 10000 4100
-F 0 "#PWR032" H 10000 3950 50  0001 C CNN
+F 0 "#PWR037" H 10000 3950 50  0001 C CNN
 F 1 "+3.3V" H 10000 4240 50  0000 C CNN
 F 2 "" H 10000 4100 50  0000 C CNN
@@
 $EndComp
 $Comp
-L GND #PWR033
+L GND #PWR038
 U 1 1 587B97E4
 P 9600 5400
-F 0 "#PWR033" H 9600 5150 50  0001 C CNN
+F 0 "#PWR038" H 9600 5150 50  0001 C CNN
 F 1 "GND" H 9600 5250 50  0000 C CNN
 F 2 "" H 9600 5400 50  0000 C CNN
@@
 $EndComp
 $Comp
-L GND #PWR034
+L GND #PWR039
 U 1 1 587B9834
 P 9300 5400
-F 0 "#PWR034" H 9300 5150 50  0001 C CNN
+F 0 "#PWR039" H 9300 5150 50  0001 C CNN
 F 1 "GND" H 9300 5250 50  0000 C CNN
 F 2 "" H 9300 5400 50  0000 C CNN
@@
 	9300 4950 9300 5050
 $Comp
-L GND #PWR035
+L GND #PWR040
 U 1 1 587D2523
 P 2450 2450
-F 0 "#PWR035" H 2450 2200 50  0001 C CNN
+F 0 "#PWR040" H 2450 2200 50  0001 C CNN
 F 1 "GND" H 2450 2300 50  0000 C CNN
 F 2 "" H 2450 2450 50  0000 C CNN
@@
 	4350 6650 4350 6700
 $Comp
-L +3.3V #PWR036
+L +3.3V #PWR041
 U 1 1 58BC4BB7
 P 4850 6600
-F 0 "#PWR036" H 4850 6450 50  0001 C CNN
+F 0 "#PWR041" H 4850 6450 50  0001 C CNN
 F 1 "+3.3V" H 4850 6740 50  0000 C CNN
 F 2 "" H 4850 6600 50  0000 C CNN
@@
 	10200 4850 10200 4900
 $Comp
-L GND #PWR037
+L GND #PWR042
 U 1 1 58BF19D6
 P 10200 5300
-F 0 "#PWR037" H 10200 5050 50  0001 C CNN
+F 0 "#PWR042" H 10200 5050 50  0001 C CNN
 F 1 "GND" H 10200 5150 50  0000 C CNN
 F 2 "" H 10200 5300 50  0000 C CNN
@@
 	6150 4550 6700 4550
 $Comp
-L GND #PWR038
+L GND #PWR043
 U 1 1 59FCED84
 P 7550 1600
-F 0 "#PWR038" H 7550 1350 50  0001 C CNN
+F 0 "#PWR043" H 7550 1350 50  0001 C CNN
 F 1 "GND" H 7550 1450 50  0000 C CNN
 F 2 "" H 7550 1600 50  0000 C CNN
@@
 $EndComp
 $Comp
-L +3.3V #PWR039
+L +3.3V #PWR044
 U 1 1 5B0C49AB
 P 5900 7400
-F 0 "#PWR039" H 5900 7250 50  0001 C CNN
+F 0 "#PWR044" H 5900 7250 50  0001 C CNN
 F 1 "+3.3V" H 5900 7540 50  0000 C CNN
 F 2 "" H 5900 7400 50  0000 C CNN
@@
 $EndComp
 $Comp
-L GND #PWR040
+L GND #PWR045
 U 1 1 5B0C4B76
 P 5800 7400
-F 0 "#PWR040" H 5800 7150 50  0001 C CNN
+F 0 "#PWR045" H 5800 7150 50  0001 C CNN
 F 1 "GND" H 5800 7250 50  0000 C CNN
 F 2 "" H 5800 7400 50  0000 C CNN
@@
 SD_CARD_ENABLE
 $Comp
-L GND #PWR041
+L GND #PWR046
 U 1 1 5B187286
 P 3300 2400
-F 0 "#PWR041" H 3300 2150 50  0001 C CNN
+F 0 "#PWR046" H 3300 2150 50  0001 C CNN
 F 1 "GND" H 3300 2250 50  0000 C CNN
 F 2 "" H 3300 2400 50  0000 C CNN
@@
 $EndComp
 $Comp
-L GND #PWR042
+L GND #PWR047
 U 1 1 5B1872E2
 P 3600 2400
-F 0 "#PWR042" H 3600 2150 50  0001 C CNN
+F 0 "#PWR047" H 3600 2150 50  0001 C CNN
 F 1 "GND" H 3600 2250 50  0000 C CNN
 F 2 "" H 3600 2400 50  0000 C CNN
@@
 $EndComp
 $Comp
-L GND #PWR043
+L GND #PWR048
 U 1 1 5B18733E
 P 3900 2400
-F 0 "#PWR043" H 3900 2150 50  0001 C CNN
+F 0 "#PWR048" H 3900 2150 50  0001 C CNN
 F 1 "GND" H 3900 2250 50  0000 C CNN
 F 2 "" H 3900 2400 50  0000 C CNN
@@
 $EndComp
 $Comp
-L +3.3V #PWR044
+L +3.3V #PWR049
 U 1 1 5B28B3EE
 P 8400 900
-F 0 "#PWR044" H 8400 750 50  0001 C CNN
+F 0 "#PWR049" H 8400 750 50  0001 C CNN
 F 1 "+3.3V" H 8415 1073 50  0000 C CNN
 F 2 "" H 8400 900 50  0000 C CNN
@@
 	6150 4750 6700 4750
 Wire Wire Line
-	1450 3750 1550 3750
+	1300 3750 1550 3750
 Text Label 1450 3650 0    60   ~ 0
 RTC_CAL
@@
 	9100 1900 9100 1600
 Connection ~ 9500 1900
+Text HLabel 1300 3750 0    60   Input ~ 0
+ESP_VCC_sense
 $EndSCHEMATC
