File: Nestbox_v3/Nestbox_v2_detector.sch (KiCad schematic (older format))
At the start: 2 parts, among them J401 LB_DETECT_CONN_01X04, J402 CONN_01X05

Commit message: removed any unnecessary functions and connectors. corrected transistor bug
Parts:
- removed J401: LB_DETECT_CONN_01X04, Terminal_Blocks:TerminalBlock_Pheonix_MPT-2.54mm_4pol, symbol CONN_01X04
Other:
- note removed: "INTERNAL\nEXTERNAL\n"
Changed lines of the file:
@@
 $EndDescr
-$Comp
-L +3.3V #PWR401
-U 1 1 59FD02D9
-P 2750 2200
-F 0 "#PWR401" H 2750 2050 50  0001 C CNN
-F 1 "+3.3V" V 2765 2328 50  0000 L CNN
-F 2 "" H 2750 2200 50  0000 C CNN
-F 3 "" H 2750 2200 50  0000 C CNN
-	1    2750 2200
-	0    -1   -1   0
-$EndComp
-$Comp
-L GND #PWR402
-U 1 1 59FD0355
-P 2750 2500
-F 0 "#PWR402" H 2750 2250 50  0001 C CNN
-F 1 "GND" V 2755 2372 50  0000 R CNN
-F 2 "" H 2750 2500 50  0000 C CNN
-F 3 "" H 2750 2500 50  0000 C CNN
-	1    2750 2500
-	0    1    1    0
-$EndComp
-$Comp
-L CONN_01X04 J401
-U 1 1 5B0A4507
-P 3100 2350
-F 0 "J401" H 3100 2600 50  0000 C CNN
-F 1 "LB_DETECT_CONN_01X04" V 3200 2350 50  0000 C CNN
-F 2 "Terminal_Blocks:TerminalBlock_Pheonix_MPT-2.54mm_4pol" H 3100 2350 50  0001 C CNN
-F 3 "" H 3100 2350 50  0001 C CNN
-	1    3100 2350
-	1    0    0    -1
-$EndComp
-Text HLabel 2750 2300 0    60   Output ~ 0
-LB1_DETECT
-Text HLabel 2750 2400 0    60   Output ~ 0
-LB2_DETECT
-Wire Wire Line
-	2750 2200 2900 2200
-Wire Wire Line
-	2750 2300 2900 2300
-Wire Wire Line
-	2750 2400 2900 2400
-Wire Wire Line
-	2750 2500 2900 2500
-Text Notes 1600 2450 0    60   ~ 0
-INTERNAL\nEXTERNAL\n
 $Comp
 L GND #PWR404

Commit message: production status nestbox v3
Connections:
- net +3V3 renamed VDDA
Changed lines of the file:
@@
 $EndDescr
 $Comp
-L GND #PWR045
+L GND #PWR050
 U 1 1 5B0B21F9
 P 2900 3650
-F 0 "#PWR045" H 2900 3400 50  0001 C CNN
+F 0 "#PWR050" H 2900 3400 50  0001 C CNN
 F 1 "GND" V 2905 3522 50  0000 R CNN
 F 2 "" H 2900 3650 50  0000 C CNN
@@
 	1    2900 3650
 	0    1    1    0
-$EndComp
-$Comp
-L +3.3V #PWR046
-U 1 1 5B0B220D
-P 2900 3250
-F 0 "#PWR046" H 2900 3100 50  0001 C CNN
-F 1 "+3.3V" V 2915 3378 50  0000 L CNN
-F 2 "" H 2900 3250 50  0000 C CNN
-F 3 "" H 2900 3250 50  0000 C CNN
-	1    2900 3250
-	0    -1   -1   0
 $EndComp
 Wire Wire Line
@@
 Wire Wire Line
 	2900 3550 2550 3550
+Wire Wire Line
+	2900 3250 2600 3250
+$Comp
+L VDDA #PWR051
+U 1 1 5BF586EC
+P 2600 3250
+F 0 "#PWR051" H 2600 3100 50  0001 C CNN
+F 1 "VDDA" H 2600 3400 50  0000 C CNN
+F 2 "" H 2600 3250 50  0001 C CNN
+F 3 "" H 2600 3250 50  0001 C CNN
+	1    2600 3250
+	1    0    0    -1
+$EndComp
 $EndSCHEMATC
