File: RFID_BOARD_V3_EM4095/RFID_board_PANNEL.kicad_pcb (KiCad board)
At the start: 2 copper layers, 97 x 100 mm, 285 parts, among them J1 CONN_01X05, J2 CONN_01X01, J3 CONN_01X01, U1 EM4095

Commit message: production status nestbox v3
Parts:
- removed the C1 at (165.5, 90.3)
- removed the C1 at (165.5, 59.8)
- removed the C11 at (165.5, 92.0)
- removed the C11 at (165.5, 61.5)
- removed the C12 at (157.0, 97.5)
- removed the C12 at (157.0, 67.0)
- removed the C2 at (157.0, 99.5)
- removed the C2 at (157.0, 69.0)
- removed the C5 at (171.0, 103.5)
- removed the C5 at (171.0, 73.0)
- removed the C6 at (169.0, 103.5)
- removed the C6 at (169.0, 73.0)
- removed the C7 at (163.0, 103.5)
- removed the C7 at (163.0, 73.0)
- removed the C8 at (160.5, 102.5)
- removed the C8 at (160.5, 72.0)
- removed the CRES1 at (161.5, 86.5)
- removed the CRES1 at (161.5, 56.0)
- removed the CRES2 at (161.5, 88.5)
- removed the CRES2 at (161.5, 58.0)
- removed the CRES3 at (161.5, 90.5)
- removed the CRES3 at (161.5, 60.0)
- removed the Cdiv1 at (158.0, 89.5)
- removed the Cdiv1 at (158.0, 59.0)
- removed the Cdiv2 at (158.0, 93.5)
- removed the Cdiv2 at (158.0, 63.0)
- removed the FID1 at (172.0, 85.0)
- removed the FID1 at (172.0, 54.5)
- removed the G*** at (164.0, 104.0)
- removed the G*** at (164.0, 91.5)
- removed the G*** at (164.0, 73.5)
- removed the G*** at (164.0, 61.0)
- removed the J1 at (159.9, 108.5)
- removed the J1 at (159.9, 78.0)
- removed the J2 at (167.5, 84.5)
- removed the J2 at (167.5, 54.0)
- removed the J3 at (160.4, 84.5)
- removed the J3 at (160.4, 54.0)
- removed the R3 at (165.0, 103.5)
- removed the R3 at (165.0, 73.0)
- removed the U1 at (165.0, 97.4)
- removed the U1 at (165.0, 66.9)
- removed the mouse-bite-2mm-slot at (164.0, 82.0)
- removed the mouse-bite-2mm-slot at (164.0, 51.5)
- added C1: 10u, Capacitors_SMD:C_0805, F.Cu at (17.0, -26.2)
- added C1: 10u, Capacitors_SMD:C_0805, F.Cu at (17.0, -56.7)
- added C11: 100n, Capacitors_SMD:C_0603, F.Cu at (17.0, -24.5)
- added C11: 100n, Capacitors_SMD:C_0603, F.Cu at (17.0, -55.0)
- added C12: 10u, Capacitors_SMD:C_0805, F.Cu at (8.50, -19.0)
- added C12: 10u, Capacitors_SMD:C_0805, F.Cu at (8.50, -49.5)
- added C2: 100n, Capacitors_SMD:C_0603, F.Cu at (8.50, -17.0)
- added C2: 100n, Capacitors_SMD:C_0603, F.Cu at (8.50, -47.5)
- added C5: 10n (22n max), Capacitors_SMD:C_0603, F.Cu at (22.5, -13.0)
- added C5: 10n (22n max), Capacitors_SMD:C_0603, F.Cu at (22.5, -43.5)
- added C6: 10n, Capacitors_SMD:C_0603, F.Cu at (20.5, -13.0)
- added C6: 10n, Capacitors_SMD:C_0603, F.Cu at (20.5, -43.5)
- added C7: 100n, Capacitors_SMD:C_0603, F.Cu at (14.5, -13.0)
- added C7: 100n, Capacitors_SMD:C_0603, F.Cu at (14.5, -43.5)
- added C8: DNP or 100n, Capacitors_SMD:C_0603, F.Cu at (12.0, -14.0)
- added C8: DNP or 100n, Capacitors_SMD:C_0603, F.Cu at (12.0, -44.5)
- added CRES1: C_fine_tuning (10nF, 50V), Capacitors_SMD:C_0603, F.Cu at (13.0, -30.0)
- added CRES1: C_fine_tuning (10nF, 50V), Capacitors_SMD:C_0603, F.Cu at (13.0, -60.5)
- added CRES2: 1.8n 250V, Capacitors_SMD:C_0805, F.Cu at (13.0, -28.0)
- added CRES2: 1.8n 250V, Capacitors_SMD:C_0805, F.Cu at (13.0, -58.5)
- added CRES3: 1n 450V, Capacitors_SMD:C_0805, F.Cu at (13.0, -26.0)
- added CRES3: 1n 450V, Capacitors_SMD:C_0805, F.Cu at (13.0, -56.5)
- added Cdiv1: 10p 500V, Capacitors_SMD:C_0805, F.Cu at (9.50, -27.0)
- added Cdiv1: 10p 500V, Capacitors_SMD:C_0805, F.Cu at (9.50, -57.5)
- added Cdiv2: 1.5n, Capacitors_SMD:C_0603, F.Cu at (9.50, -23.0)
- added Cdiv2: 1.5n, Capacitors_SMD:C_0603, F.Cu at (9.50, -53.5)
- added FID1: Fiducial_1mm_Dia_2.54mm_Outer_CopperTop, Fiducials:Fiducial_1mm_Dia_2.54mm_Outer_CopperTop, F.Cu at (23.5, -31.5)
- added FID1: Fiducial_1mm_Dia_2.54mm_Outer_CopperTop, Fiducials:Fiducial_1mm_Dia_2.54mm_Outer_CopperTop, F.Cu at (23.5, -62.0)
- added G***: LOGO, Octanis3:VogelwarteLogo3, B.Cu at (15.5, -12.5)
- added G***: LOGO, Octanis3:octanis_open_incubator_logo, B.Cu at (15.5, -25.0)
- added G***: LOGO, Octanis3:VogelwarteLogo3, B.Cu at (15.5, -43.0)
- added G***: LOGO, Octanis3:octanis_open_incubator_logo, B.Cu at (15.5, -55.5)
- added J1: CONN_01X05, Pin_Headers:Pin_Header_Straight_1x05_Pitch2.54mm, F.Cu at (11.4, -8.00)
- added J1: CONN_01X05, Pin_Headers:Pin_Header_Straight_1x05_Pitch2.54mm, F.Cu at (11.4, -38.5)
- added J2: CONN_01X01, Measurement_Points:Measurement_Point_Square-SMD-Pad_Small, F.Cu at (19.0, -32.0)
- added J2: CONN_01X01, Measurement_Points:Measurement_Point_Square-SMD-Pad_Small, F.Cu at (19.0, -62.5)
- added J3: CONN_01X01, Measurement_Points:Measurement_Point_Square-SMD-Pad_Small, F.Cu at (11.9, -32.0)
- added J3: CONN_01X01, Measurement_Points:Measurement_Point_Square-SMD-Pad_Small, F.Cu at (11.9, -62.5)
- added R3: 0R, Resistors_SMD:R_0603, F.Cu at (16.5, -13.0)
- added R3: 0R, Resistors_SMD:R_0603, F.Cu at (16.5, -43.5)
- added U1: EM4095, Housings_SOIC:SOIC-16_3.9x9.9mm_Pitch1.27mm, F.Cu at (16.5, -19.1)
- added U1: EM4095, Housings_SOIC:SOIC-16_3.9x9.9mm_Pitch1.27mm, F.Cu at (16.5, -49.6)
- added mouse-bite-2mm-slot: VAL**, Panelization:mouse-bite-2mm-slot, F.Cu at (15.5, -34.5)
- added mouse-bite-2mm-slot: VAL**, Panelization:mouse-bite-2mm-slot, F.Cu at (15.5, -65.0)
- moved C1 188.7 mm to (83.0, -26.2)
- moved C1 188.7 mm to (17.0, -87.2)
- moved C1 188.7 mm to (83.0, -56.7)
- moved C1 188.7 mm to (83.0, -87.2)
- moved C1 188.7 mm to (61.0, -26.2)
- moved C1 188.7 mm to (61.0, -56.7)
- moved C1 188.7 mm to (61.0, -87.2)
- moved C1 188.7 mm to (39.0, -87.2)
- moved C1 188.7 mm to (39.0, -56.7)
- moved C1 188.7 mm to (39.0, -26.2)
- moved C11 188.7 mm to (83.0, -24.5)
- moved C11 188.7 mm to (17.0, -85.5)
- moved C11 188.7 mm to (83.0, -55.0)
- moved C11 188.7 mm to (83.0, -85.5)
- moved C11 188.7 mm to (61.0, -24.5)
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