File: RFID_BOARD_V3_EM4095/RFID_BOARD_V3_EM4095.sch (KiCad schematic (older format))
At the start: 18 parts, among them J1 CONN_01X05, J2 CONN_01X01, J3 CONN_01X01, U1 EM4095

Commit message: various changes & updates, production state
Other:
- moved on the sheet: J2, J3
Changed lines of the file:
@@
 LIBS:valves
 LIBS:cmut_lib
+LIBS:RFID_BOARD_V3_EM4095-cache
 EELAYER 25 0
 EELAYER END
@@
 U 1 1 5AFA1B9F
 P 5700 4050
-F 0 "C5" H 5725 4150 50  0000 L CNN
+F 0 "C5" V 5650 3850 50  0000 L CNN
 F 1 "10n  (22n max)" V 5500 3850 50  0000 L CNN
 F 2 "Capacitors_SMD:C_0603" H 5738 3900 50  0001 C CNN
@@
 U 1 1 5AFA1EF5
 P 5700 4150
-F 0 "C6" H 5725 4250 50  0000 L CNN
+F 0 "C6" V 5750 3950 50  0000 L CNN
 F 1 "10n" V 5850 4050 50  0000 L CNN
 F 2 "Capacitors_SMD:C_0603" H 5738 4000 50  0001 C CNN
@@
 U 1 1 5AFA0C2C
 P 4850 4600
-F 0 "U1" H 4850 5578 50  0000 C CNN
-F 1 "EM4095" H 4850 5487 50  0000 C CNN
+F 0 "U1" H 5250 5300 50  0000 C CNN
+F 1 "EM4095" H 4550 5300 50  0000 C CNN
 F 2 "Housings_SOIC:SOIC-16_3.9x9.9mm_Pitch1.27mm" H 4850 4600 50  0001 C CIN
 F 3 "" H 4850 4600 50  0001 C CNN
@@
 Connection ~ 8400 4850
 Wire Wire Line
-	2700 3450 2700 3650
-Wire Wire Line
-	2700 3650 2750 3650
-Wire Wire Line
-	2600 3450 2600 3650
-Wire Wire Line
-	2600 3650 2550 3650
-Text Label 2550 3650 2    60   ~ 0
+	3100 3550 3100 3750
+Wire Wire Line
+	3100 3750 3150 3750
+Wire Wire Line
+	3000 3550 3000 3750
+Wire Wire Line
+	3000 3750 2950 3750
+Text Label 2950 3750 2    60   ~ 0
 ant1
-Text Label 2750 3650 0    60   ~ 0
+Text Label 3150 3750 0    60   ~ 0
 ant2
 $Comp
@@
 L CONN_01X01 J2
 U 1 1 5B1D646B
-P 2600 3250
-F 0 "J2" H 2600 3350 50  0000 C CNN
-F 1 "CONN_01X01" V 2700 3250 50  0000 C CNN
-F 2 "Measurement_Points:Measurement_Point_Square-SMD-Pad_Small" H 2600 3250 50  0001 C CNN
-F 3 "" H 2600 3250 50  0001 C CNN
-	1    2600 3250
+P 3000 3350
+F 0 "J2" H 3000 3450 50  0000 C CNN
+F 1 "CONN_01X01" V 3100 3350 50  0000 C CNN
+F 2 "Measurement_Points:Measurement_Point_Square-SMD-Pad_Small" H 3000 3350 50  0001 C CNN
+F 3 "" H 3000 3350 50  0001 C CNN
+	1    3000 3350
 	0    -1   -1   0
 $EndComp
@@
 L CONN_01X01 J3
 U 1 1 5B1D64DD
-P 2700 3250
-F 0 "J3" H 2700 3350 50  0000 C CNN
-F 1 "CONN_01X01" V 2800 3250 50  0000 C CNN
-F 2 "Measurement_Points:Measurement_Point_Square-SMD-Pad_Small" H 2700 3250 50  0001 C CNN
-F 3 "" H 2700 3250 50  0001 C CNN
-	1    2700 3250
-	0    -1   -1   0
-$EndComp
+P 3100 3350
+F 0 "J3" H 3100 3450 50  0000 C CNN
+F 1 "CONN_01X01" V 3200 3350 50  0000 C CNN
+F 2 "Measurement_Points:Measurement_Point_Square-SMD-Pad_Small" H 3100 3350 50  0001 C CNN
+F 3 "" H 3100 3350 50  0001 C CNN
+	1    3100 3350
+	0    -1   -1   0
+$EndComp
